Commit message: Update scene

File: catkin_ws/src/o2ac_scene_description/urdf/components/screw_tools.xacro (robot description, xacro)
@@ -1,3 +1,3 @@
-<!-- This has a size of about 155 mm x 40 mm x 26 mm -->
+<!-- This holder has a size of about 155 mm x 40 mm x 26 mm -->
 <!-- The Bit cushion has a height of 30.5 mm, starts about 24 mm from the top-->
 <!-- The gripper center would be about 44 mm from the top, so the tip might be 111 mm further down -->
@@ -5,8 +5,7 @@
 <robot xmlns:xacro="http://www.ros.org/wiki/xacro">
   <joint name="screw_holder_to_environment_joint" type="fixed">
-    <parent link="cross_column_2" />
+    <parent link="horizontal_column_for_tools" />
     <child link="screw_tool_holder" />
     <origin xyz=".04 .0 .04" rpy="0.0 0.0 ${-pi/2}" />
-    <!-- +.005 is a MAGIC NUMBER added on Sep 17 to put the tool roughly between c_bot and b_bot's physical position. -->
   </joint>
   <link name="screw_tool_holder">
@@ -22,4 +21,7 @@
         <box size=".3 .066 .004"/>
       </geometry>
+      <material name="grey">
+        <color rgba=".5 .5 .5 1"/>
+      </material>
     </visual>
     <collision>
@@ -35,4 +37,7 @@
         <box size=".3 .004 .035"/>
       </geometry>
+      <material name="grey">
+        <color rgba=".5 .5 .5 1"/>
+      </material>
     </visual>
     <collision>
@@ -47,29 +52,29 @@
   <xacro:property name="tool_offset" value="${-.005 + bit_cushion_to_axis}" />
   <!-- The collision boxes of the tools only include the top part (not what is hanging underneath the holder) -->
-  <link name="screw_tool_m6_link">
-    <inertial>
-      <origin rpy="0 0 0" xyz="0 0 0"/>
-      <mass value="1.0"/>
-      <inertia ixx="1" ixy="0" ixz="0" iyy="1" iyz="0" izz="1"/>
-    </inertial>
-    <visual>
-      <origin rpy="0 0 0" xyz="0 0 0"/>
-      <geometry>
-        <mesh filename="package://o2ac_scene_description/meshes/screw_tool_m6_BC5-XL320-LG20-R_v2.stl" scale="0.001 0.001 0.001"/>
-      </geometry>
-      <material name="white">
-        <color rgba=".9 .9 .9 1"/>
-      </material>
-    </visual>
-    <collision>
-      <origin rpy="0 0 0" xyz="0 ${bit_cushion_to_axis - .02} .0275"/>
-      <geometry>
-        <box size=".026 .04 .055"/>
-      </geometry>
-    </collision>
-  </link>
-  <joint name="screw_tool_m6_to_holder" type="fixed">
-    <parent link="screw_tool_holder" />
-    <child link="screw_tool_m6_link" />
+  <link name="belt_tool_link">
+    <inertial>
+      <origin rpy="0 0 0" xyz="0 0 0"/>
+      <mass value="1.0"/>
+      <inertia ixx="1" ixy="0" ixz="0" iyy="1" iyz="0" izz="1"/>
+    </inertial>
+    <visual>
+      <origin rpy="0 0 ${pi}" xyz="0 0 0"/>
+      <geometry>
+        <mesh filename="package://o2ac_scene_description/meshes/belt_hook_tool.stl" scale="0.001 0.001 0.001"/>
+      </geometry>
+      <material name="white">
+        <color rgba=".9 .9 .9 1"/>
+      </material>
+    </visual>
+    <collision>
+      <origin rpy="0 0 0" xyz="0 ${bit_cushion_to_axis - .02} .0275"/>
+      <geometry>
+        <box size=".026 .04 .055"/>
+      </geometry>
+    </collision>
+  </link>
+  <joint name="belt_tool_to_holder" type="fixed">
+    <parent link="screw_tool_holder" />
+    <child link="belt_tool_link" />
     <origin xyz="-0.05 ${tool_offset} 0.004" rpy="0.0 0.0 0.0" />
   </joint>
@@ -101,31 +106,4 @@
     <origin xyz="-0.35 ${tool_offset} 0.004" rpy="0.0 0.0 0.0" />
   </joint>
-  <link name="suction_tool_link">
-    <inertial>
-      <origin rpy="0 0 0" xyz="0 0 0"/>
-      <mass value="1.0"/>
-      <inertia ixx="1" ixy="0" ixz="0" iyy="1" iyz="0" izz="1"/>
-    </inertial>
-    <visual>
-      <origin rpy="${pi/2} 0 ${-pi/2}" xyz="0 0.009 0.047"/>
-      <geometry>
-        <mesh filename="package://o2ac_scene_description/meshes/suction_tool_phi10.stl" scale="0.001 0.001 0.001"/>
-      </geometry>
-      <material name="white">
-        <color rgba=".9 .9 .9 1"/>
-      </material>
-    </visual>
-    <collision>
-      <origin rpy="0 0 0" xyz="0 ${bit_cushion_to_axis - .02} .0275"/>
-      <geometry>
-        <box size=".026 .04 .055"/>
-      </geometry>
-    </collision>
-  </link>
-  <joint name="suction_tool_to_holder" type="fixed">
-    <parent link="screw_tool_holder" />
-    <child link="suction_tool_link" />
-    <origin xyz="-0.355 ${tool_offset - .015} 0.004" rpy="0.0 0.0 0.0" />
-  </joint>
   <link name="set_screw_tool_link">
     <inertial>
@@ -195,38 +173,32 @@
   </joint>
   <!-- Extra links to position the gripper more easily -->
-  <link name="screw_tool_m3_helper_link"/>
-  <joint name="screw_tool_m3_helper_joint" type="fixed">
+  <link name="screw_tool_m3_pickup_link"/>
+  <joint name="screw_tool_m3_pickup_joint" type="fixed">
     <parent link="screw_tool_m3_link" />
-    <child link="screw_tool_m3_helper_link" />
-    <origin xyz="0.0 0.0 0.0" rpy="0.0 0.0 ${-pi/2}" />
-  </joint>
-  <link name="screw_tool_m4_helper_link"/>
-  <joint name="screw_tool_m4_helper_joint" type="fixed">
+    <child link="screw_tool_m3_pickup_link" />
+    <origin xyz="0.0 0.0 0.0" rpy="0.0 0.0 ${-pi/2}" />
+  </joint>
+  <link name="screw_tool_m4_pickup_link"/>
+  <joint name="screw_tool_m4_pickup_joint" type="fixed">
     <parent link="screw_tool_m4_link" />
-    <child link="screw_tool_m4_helper_link" />
-    <origin xyz="0.0 0.0 0.0" rpy="0.0 0.0 ${-pi/2}" />
-  </joint>
-  <link name="screw_tool_m6_helper_link"/>
-  <joint name="screw_tool_m6_helper_joint" type="fixed">
-    <parent link="screw_tool_m6_link" />
-    <child link="screw_tool_m6_helper_link" />
-    <origin xyz="0.0 0.0 0.0" rpy="0.0 0.0 ${-pi/2}" />
-  </joint>
-  <link name="nut_tool_m6_helper_link"/>
-  <joint name="nut_tool_m6_helper_joint" type="fixed">
+    <child link="screw_tool_m4_pickup_link" />
+    <origin xyz="0.0 0.0 0.0" rpy="0.0 0.0 ${-pi/2}" />
+  </joint>
+  <link name="belt_tool_pickup_link"/>
+  <joint name="belt_tool_pickup_joint" type="fixed">
+    <parent link="belt_tool_link" />
+    <child link="belt_tool_pickup_link" />
+    <origin xyz="0.0 0.0 0.0" rpy="0.0 0.0 ${-pi/2}" />
+  </joint>
+  <link name="nut_tool_m6_pickup_link"/>
+  <joint name="nut_tool_m6_pickup_joint" type="fixed">
     <parent link="nut_tool_m6_link" />
-    <child link="nut_tool_m6_helper_link" />
-    <origin xyz="0.0 0.0 0.0" rpy="0.0 0.0 ${-pi/2}" />
-  </joint>
-  <link name="suction_tool_helper_link"/>
-  <joint name="suction_tool_helper_joint" type="fixed">
-    <parent link="suction_tool_link" />
-    <child link="suction_tool_helper_link" />
-    <origin xyz="0.0 0.0 0.0" rpy="0.0 0.0 ${-pi/2}" />
-  </joint>
-  <link name="set_screw_tool_helper_link"/>
-  <joint name="set_screw_tool_helper_joint" type="fixed">
+    <child link="nut_tool_m6_pickup_link" />
+    <origin xyz="0.0 0.0 0.0" rpy="0.0 0.0 ${-pi/2}" />
+  </joint>
+  <link name="set_screw_tool_pickup_link"/>
+  <joint name="set_screw_tool_pickup_joint" type="fixed">
     <parent link="set_screw_tool_link" />
-    <child link="set_screw_tool_helper_link" />
+    <child link="set_screw_tool_pickup_link" />
     <origin xyz="0.0 0.0 0.0" rpy="0.0 0.0 ${-pi/2}" />
   </joint>

File: catkin_ws/src/o2ac_scene_description/urdf/components/taskboard.xacro (robot description, xacro)
@@ -15,6 +15,6 @@
         <mesh filename="${mesh_file_base}" scale=".001 .001 .001"/>
       </geometry>
-      <material name="white">
-        <color rgba="1 1 1 1"/>
+      <material name="gray">
+        <color rgba=".5 .5 .5 1"/>
       </material>
     </visual>
@@ -32,9 +32,4 @@
   </joint>
   <link name="${boardname}_plate">
-    <inertial>
-      <origin rpy="${pi/2} 0 ${pi/2}" xyz="0 0 0"/>
-      <mass value="1.0"/>
-      <inertia ixx="1.0" ixy="0" ixz="0" iyy="1.0" iyz="0" izz="1.0"/>
-    </inertial>
     <visual>
       <origin rpy="${pi/2} 0 ${pi/2}" xyz="0 0 0"/>
@@ -42,6 +37,6 @@
         <mesh filename="${mesh_file_plate}" scale=".001 .001 .001"/>
       </geometry>
-      <material name="white">
-        <color rgba="1 1 1 1"/>
+      <material name="gray">
+        <color rgba=".5 .5 .5 1"/>
       </material>
     </visual>
@@ -58,32 +53,140 @@
     <origin rpy="0 0 0" xyz="-0.06 0.0 0.0"/>
   </joint>
+  <!-- ========== Shaft, pulleys, bearing -->
+  <joint name="${boardname}_small_shaft" type="fixed">
+    <parent link="${boardname}_plate" />
+    <child link = "${boardname}_small_shaft" />
+    <origin rpy="0 0 ${pi}" xyz="${.025+.025} 0.099 0.085"/>
+  </joint>
+  <link name="${boardname}_small_shaft">
+    <visual>
+      <origin rpy="0 ${pi/2} 0" xyz="0.0125 0 0"/>
+      <geometry>
+        <cylinder length="0.025" radius="0.003"/>
+      </geometry>
+      <material name="gray">
+        <color rgba=".5 .5 .5 1"/>
+      </material>
+    </visual>
+    <collision>
+      <origin rpy="0 ${pi/2} 0" xyz="0.0125 0 0"/>
+      <geometry>
+        <cylinder length="0.025" radius="0.003"/>
+      </geometry>
+    </collision>
+  </link>
+  <!-- The bearing -->
+  <xacro:include filename="$(find o2ac_parts_description)/urdf/generated/07_SBARB6200ZZ_30_macro.urdf.xacro" />
+  <xacro:assy_part_07 prefix="${boardname}_" parent="${boardname}_plate" spawn_attached="true">
+    <origin rpy="0 0 0" xyz="${0.025+.008} 0.165 0.12"/>
+  </xacro:assy_part_07>
+  <joint name="${boardname}_small_pulley" type="fixed">
+    <parent link="${boardname}_plate" />
+    <child link = "${boardname}_small_pulley" />
+    <origin rpy="0 0 ${pi}" xyz="${.025+.013} 0.0275 0.033"/>
+  </joint>
+  <link name="${boardname}_small_pulley">
+    <visual>
+      <origin rpy="0 0 0" xyz="0 0 0"/>
+      <geometry>
+        <mesh filename="package://o2ac_parts_description/meshes/50_MBGNA30-2.stl" scale="0.001 0.001 0.001"/>
+      </geometry>
+      <material name="gray">
+        <color rgba=".5 .5 .5 1"/>
+      </material>
+    </visual>
+    <collision>
+      <origin rpy="0 0 0" xyz="0 0 0"/>
+      <geometry>
+        <mesh filename="package://o2ac_parts_description/meshes/50_MBGNA30-2.stl" scale="0.001 0.001 0.001"/>
+      </geometry>
+    </collision>
+  </link>
+  <!-- 16.5 -->
+  <joint name="${boardname}_large_pulley" type="fixed">
+    <parent link="${boardname}_plate" />
+    <child link = "${boardname}_large_pulley" />
+    <origin rpy="0 0 ${pi}" xyz="${.025+.0165} 0.1575 0.04"/>
+  </joint>
+  <link name="${boardname}_large_pulley">
+    <visual>
+      <origin rpy="0 0 0" xyz="0 0 0"/>
+      <geometry>
+        <mesh filename="package://o2ac_parts_description/meshes/51_MBGNA60-2.stl" scale="0.001 0.001 0.001"/>
+      </geometry>
+      <material name="gray">
+        <color rgba=".5 .5 .5 1"/>
+      </material>
+    </visual>
+    <collision>
+      <origin rpy="0 0 0" xyz="0 0 0"/>
+      <geometry>
+        <mesh filename="package://o2ac_parts_description/meshes/51_MBGNA60-2.stl" scale="0.001 0.001 0.001"/>
+      </geometry>
+    </collision>
+  </link>
+  <!-- ========== Helper frames -->
   <joint name="${boardname}_surface_joint" type="fixed">
     <parent link="${boardname}_plate"/>
     <child link="${boardname}_surface"/>
-    <origin rpy="0.0 ${pi} 0" xyz="0.025 0.1 0.05"/>
+    <origin rpy="0 0 ${pi}" xyz="0.025 0.1 0.05"/>
   </joint>
   <link name="${boardname}_surface"/>
-  <joint name="${boardname}_set_screw_tool_joint" type="fixed">
+  <joint name="${boardname}_set_screw_joint" type="fixed">
     <parent link="${boardname}_plate"/>
-    <child link="${boardname}_set_screw_tool_link"/>
-    <origin rpy="0.0 ${pi/2} ${pi/2}" xyz="-0.08 0.3 0"/>
+    <child link="${boardname}_set_screw_link"/>
+    <origin rpy="0 0 ${pi}" xyz=".025 0.054 0.075"/>
   </joint>
-  <link name="${boardname}_set_screw_tool_link"/>
-  <!-- <joint name="${boardname}_part7_2" type="fixed">
-    <parent link="${boardname}_part7_1"/>
-    <child link="${boardname}_part7_2"/>
-    <origin rpy="0.0 0.0 ${pi*1.0}" xyz="0.003 0.0 0.0"/>
+  <link name="${boardname}_set_screw_link"/>
+  <joint name="${boardname}_m3_screw_joint" type="fixed">
+    <parent link="${boardname}_plate"/>
+    <child link="${boardname}_m3_screw_link"/>
+    <origin rpy="0 0 ${pi}" xyz=".025 0.072 0.035"/>
   </joint>
-  <link name="${boardname}_part7_2">
-    <visual>
-      <origin xyz="0.0015 0 -0.0125" rpy="0 0 ${pi/2}"/>
-      <geometry>
-        <box size=".025 0.003 .076"/>
-      </geometry>
-      <material name="grey">
-        <color rgba=".3 .3 .3 1"/>
-      </material>
-    </visual>
-  </link> -->
+  <link name="${boardname}_m3_screw_link"/>
+  <joint name="${boardname}_m4_screw_joint" type="fixed">
+    <parent link="${boardname}_plate"/>
+    <child link="${boardname}_m4_screw_link"/>
+    <origin rpy="0 0 ${pi}" xyz=".025 0.105 0.036"/>
+  </joint>
+  <link name="${boardname}_m4_screw_link"/>
+  <joint name="${boardname}_long_hole_middle_joint" type="fixed">
+    <parent link="${boardname}_plate"/>
+    <child link="${boardname}_long_hole_middle_link"/>
+    <origin rpy="0 0 ${pi}" xyz=".025 0.1 0.125"/>
+  </joint>
+  <link name="${boardname}_long_hole_middle_link"/>
+  <joint name="${boardname}_bearing_target_joint" type="fixed">
+    <parent link="${boardname}_plate"/>
+    <child link="${boardname}_bearing_target_link"/>
+    <origin rpy="0 0 ${pi}" xyz=".025 0.034 0.12"/>
+  </joint>
+  <link name="${boardname}_bearing_target_link"/>
+  <!-- I wrote these bearing screw frames out, but actually they should
+      come from the subframes of the bearing that will be placed there. If they are used at all. -->
+  <!-- <joint name="${boardname}_bearing_screw_1_joint" type="fixed">
+    <parent link="${boardname}_plate"/>
+    <child link="${boardname}_bearing_screw_1_link"/>
+    <origin rpy="0 0 ${pi}" xyz="${.025+.008} ${0.034} ${0.12+.022}"/>
+  </joint>
+  <link name="${boardname}_bearing_screw_1_link"/>
+  <joint name="${boardname}_bearing_screw_2_joint" type="fixed">
+    <parent link="${boardname}_plate"/>
+    <child link="${boardname}_bearing_screw_2_link"/>
+    <origin rpy="0 0 ${pi}" xyz="${.025+.008} ${0.034} ${0.12-.022}"/>
+  </joint>
+  <link name="${boardname}_bearing_screw_2_link"/>
+  <joint name="${boardname}_bearing_screw_3_joint" type="fixed">
+    <parent link="${boardname}_plate"/>
+    <child link="${boardname}_bearing_screw_3_link"/>
+    <origin rpy="0 0 ${pi}" xyz="${.025+.008} ${0.034+.022} ${0.12}"/>
+  </joint>
+  <link name="${boardname}_bearing_screw_3_link"/>
+  <joint name="${boardname}_bearing_screw_4_joint" type="fixed">
+    <parent link="${boardname}_plate"/>
+    <child link="${boardname}_bearing_screw_4_link"/>
+    <origin rpy="0 0 ${pi}" xyz="${.025+.008} ${0.034-.022} ${0.12}"/>
+  </joint>
+  <link name="${boardname}_bearing_screw_4_link"/> -->
   </xacro:macro>
   <!-- Add additional links for us to plan with.-->

File: catkin_ws/src/o2ac_scene_description/urdf/o2ac_environment.xacro (robot description, xacro)
@@ -4,6 +4,5 @@
   <xacro:include filename="$(find o2ac_scene_description)/urdf/components/o2ac_box.xacro" />
   <!-- This file defines the frames surrounding the robots, used to fix the tools, multi-jig etc. -->
-  <xacro:property name="vert_column_x_back" value="${-.325-.15}"/>
-  <xacro:property name="vert_column_x_front" value="${.325-.04}"/>
+  <xacro:property name="vert_column_x_back" value="${-.325-.15-.04}"/>
   <xacro:o2ac_box boxname="vertical_column_right" box_w=".04" box_l=".04" box_h="2.0" parent="o2ac_ground">
     <origin xyz="${vert_column_x_back} .2 0" rpy="0 0 0" />
@@ -12,12 +11,9 @@
     <origin xyz="${vert_column_x_back} -.24 0" rpy="0 0 0" />
   </xacro:o2ac_box>
-  <xacro:o2ac_box boxname="cross_column_top" box_w=".04" box_l=".4" box_h=".04" parent="o2ac_ground">
+  <xacro:o2ac_box boxname="horizontal_column_top" box_w=".04" box_l=".4" box_h=".04" parent="o2ac_ground">
     <origin xyz="${vert_column_x_back} -.2 1.96" rpy="0 0 0" />
   </xacro:o2ac_box>
-  <xacro:o2ac_box boxname="cross_column_1" box_w=".04" box_l=".4" box_h=".04" parent="o2ac_ground">
-    <origin xyz="${vert_column_x_back} -.2 1.0" rpy="0 0 0" />
-  </xacro:o2ac_box>
-  <xacro:o2ac_box boxname="cross_column_2" box_w=".04" box_l=".4" box_h=".04" parent="o2ac_ground">
-    <origin xyz="${vert_column_x_back} -.2 1.3" rpy="0 0 0" />
+  <xacro:o2ac_box boxname="horizontal_column_for_tools" box_w=".04" box_l=".4" box_h=".04" parent="o2ac_ground">
+    <origin xyz="${vert_column_x_back} -.2 1.05" rpy="0 0 0" />
   </xacro:o2ac_box>
   <!-- Screw holder & screw tool visual -->
@@ -26,16 +22,16 @@
   <xacro:include filename="$(find o2ac_scene_description)/urdf/components/screw_feeder.xacro" />
   <xacro:screw_feeder feedername="m4_feeder" parent="workspace_center">
-    <origin xyz="${vert_column_x_back} .3 0" rpy="0 0 0" />
+    <origin xyz="-.55 .05 -0.043" rpy="0 0 0" />
   </xacro:screw_feeder>
   <xacro:screw_feeder feedername="m3_feeder" parent="workspace_center">
-    <origin xyz="${vert_column_x_back} .45 0" rpy="0 0 0" />
+    <origin xyz="-.55 -.15 -0.043" rpy="0 0 0" />
   </xacro:screw_feeder>
   <!-- Add the jigs -->
-  <xacro:include filename="$(find o2ac_scene_description)/urdf/components/jig_flat_slope.xacro" />
-  <xacro:jig_flat_slope jigname="jig_flat_slope" parent="cross_column_1">
+  <!-- <xacro:include filename="$(find o2ac_scene_description)/urdf/components/jig_flat_slope.xacro" />
+  <xacro:jig_flat_slope jigname="jig_flat_slope" parent="horizontal_column_1">
     <origin xyz="0.04 0.15 0" rpy="0 0 0" />
-  </xacro:jig_flat_slope>
+  </xacro:jig_flat_slope>  -->
   <xacro:include filename="$(find o2ac_scene_description)/urdf/components/jig_v_slope.xacro" />
-  <!-- <xacro:jig_v_slope jigname="jig_v_slope" parent="cross_column_1">
+  <!-- <xacro:jig_v_slope jigname="jig_v_slope" parent="horizontal_column_1">
     <origin xyz="0 0 0" rpy="0 0 0" />
   </xacro:jig_v_slope>  -->
