Commit message: Add holders, update tools, models etc.

File: catkin_ws/src/o2ac_scene_description/urdf/components/wrist_cameras.xacro (robot description, xacro)
@@ -25,5 +25,5 @@
         <origin rpy="0 0 0" xyz="-.01 0.0 .035"/>
         <geometry>
-          <box size=".03 .12 .08"/>
+          <box size=".03 .15 .08"/>
         </geometry>
       </collision>

Commit message: Add camera cables to robot model

File: catkin_ws/src/o2ac_scene_description/urdf/components/wrist_cameras.xacro (robot description, xacro)
@@ -34,4 +34,32 @@
       <origin xyz="0.035 0.0 0.025" rpy="0 0 0"/>
     </joint>
+    <!-- A collision box to represent the USB 3.1 cable connectors on the side of the cameras -->
+    <link name="${prefix}cam_cables_link">
+      <inertial>
+        <origin rpy="0 0 0" xyz="0 0 0.0"/>
+        <mass value="0.1"/>
+        <inertia ixx="1.0" ixy="0" ixz="0" iyy="1.0" iyz="0" izz="1.0"/>
+      </inertial>
+      <visual>
+        <origin rpy="0 0 0" xyz="0 0 0"/>
+        <geometry>
+          <box size=".05 .03 .055"/>
+        </geometry>
+        <material name="black">
+          <color rgba=".2 .2 .2 1"/>
+        </material>
+      </visual>
+      <collision>
+        <origin rpy="0 0 0" xyz="0 0 0"/>
+        <geometry>
+          <box size=".05 .03 .055"/>
+        </geometry>
+      </collision>
+    </link>
+    <joint name="${prefix}cam_cables_joint" type="fixed">
+      <parent link="${parent}" />
+      <child link ="${prefix}cam_cables_link" />
+      <origin xyz=".014 -.085 0.07" rpy="0 0 0"/>
+    </joint>
     <link name="${prefix}inside_cam_link" />
     <joint name="${prefix}inside_cam_joint" type="fixed">

Commit message: Fix cable collision box size (was too large)

File: catkin_ws/src/o2ac_scene_description/urdf/components/wrist_cameras.xacro (robot description, xacro)
@@ -44,5 +44,5 @@
         <origin rpy="0 0 0" xyz="0 0 0"/>
         <geometry>
-          <box size=".05 .03 .055"/>
+          <box size=".03 .03 .055"/>
         </geometry>
         <material name="black">
@@ -53,5 +53,5 @@
         <origin rpy="0 0 0" xyz="0 0 0"/>
         <geometry>
-          <box size=".05 .03 .055"/>
+          <box size=".03 .03 .055"/>
         </geometry>
       </collision>
@@ -60,5 +60,5 @@
       <parent link="${parent}" />
       <child link ="${prefix}cam_cables_link" />
-      <origin xyz=".014 -.085 0.07" rpy="0 0 0"/>
+      <origin xyz=".034 -.085 0.07" rpy="0 0 0"/>
     </joint>
     <link name="${prefix}inside_cam_link" />
