Commit message: Add bearing fastening to taskboard task

File: catkin_ws/src/o2ac_scene_description/urdf/components/taskboard.xacro (robot description, xacro)
@@ -164,4 +164,29 @@
   </joint>
   <link name="${boardname}_bearing_target_link"/>
+  <!-- The screw holes of the bearing -->
+  <joint name="${boardname}_bearing_target_screw_1_joint" type="fixed">
+    <parent link="${boardname}_bearing_target_link"/>
+    <child link="${boardname}_bearing_target_screw_1_link"/>
+    <origin rpy="${pi} 0 0" xyz="-.004 .022 0"/>
+  </joint>
+  <link name="${boardname}_bearing_target_screw_1_link"/>
+  <joint name="${boardname}_bearing_target_screw_2_joint" type="fixed">
+    <parent link="${boardname}_bearing_target_link"/>
+    <child link="${boardname}_bearing_target_screw_2_link"/>
+    <origin rpy="${pi} 0 0" xyz="-.004 0 .022"/>
+  </joint>
+  <link name="${boardname}_bearing_target_screw_2_link"/>
+  <joint name="${boardname}_bearing_target_screw_3_joint" type="fixed">
+    <parent link="${boardname}_bearing_target_link"/>
+    <child link="${boardname}_bearing_target_screw_3_link"/>
+    <origin rpy="${pi} 0 0" xyz="-.004 -0.022 0"/>
+  </joint>
+  <link name="${boardname}_bearing_target_screw_3_link"/>
+  <joint name="${boardname}_bearing_target_screw_4_joint" type="fixed">
+    <parent link="${boardname}_bearing_target_link"/>
+    <child link="${boardname}_bearing_target_screw_4_link"/>
+    <origin rpy="${pi} 0 0" xyz="-.004 0 -0.022"/>
+  </joint>
+  <link name="${boardname}_bearing_target_screw_4_link"/>
   <!-- Screw positions of the base plate -->
   <xacro:property name="base_l" value="0.2" />

Commit message: Insert and keep pulley at top of ridge

File: catkin_ws/src/o2ac_scene_description/urdf/components/taskboard.xacro (robot description, xacro)
@@ -158,4 +158,10 @@
   </joint>
   <link name="${boardname}_long_hole_middle_link"/>
+  <joint name="${boardname}_long_hole_top_joint" type="fixed">
+    <parent link="${boardname}_long_hole_middle_link"/>
+    <child link="${boardname}_long_hole_top_link"/>
+    <origin rpy="0 0 0" xyz="0 0 -0.015"/>
+  </joint>
+  <link name="${boardname}_long_hole_top_link"/>
   <joint name="${boardname}_bearing_target_joint" type="fixed">
     <parent link="${boardname}_plate"/>
