Commit message: Fix collision geometry and taskboard

File: catkin_ws/src/o2ac_scene_description/urdf/components/base_fixture.xacro (robot description, xacro)
@@ -6,5 +6,5 @@
   <xacro:property name="long_bar_mesh" value="package://o2ac_scene_description/meshes/HFSP5-2080-320.stl" />
   <xacro:property name="length" value=".32" />
-  <xacro:property name="width" value=".2" />
+  <xacro:property name="width" value=".24" />
   <link name="base_fixture_top">
     <visual>
@@ -18,8 +18,21 @@
     </visual>
     <collision>
-      <origin rpy="0 0 0" xyz="${width/2} ${length/2} 0.095"/>
+      <origin rpy="0 0 0" xyz="${width/2} ${length/2} ${.08+.01/2}"/>
       <geometry>
-        <box size="${width} ${length} 0.03"/>
-        <!-- <mesh filename="${top_mesh}" scale=".001 .001 .001"/> -->
+        <box size="${width} ${length} 0.01"/>
+      </geometry>
+    </collision>
+    <!-- The long stopper bar -->
+    <collision>
+      <origin rpy="0 0 0" xyz="${width-.02/2} ${length-.20/2} ${.08+.03/2}"/>
+      <geometry>
+        <box size="${.02} ${.20} 0.03"/>
+      </geometry>
+    </collision>
+    <!-- The short stopper bar -->
+    <collision>
+      <origin rpy="0 0 0" xyz="${width-.16/2} ${length-.02/2} ${.08+.03/2}"/>
+      <geometry>
+        <box size="${.16} ${.02} 0.03"/>
       </geometry>
     </collision>
@@ -35,5 +48,4 @@
       <geometry>
         <box size=".02 ${length} .08"/>
-        <!-- <mesh filename="${long_bar_mesh}" scale=".001 .001 .001"/> -->
       </geometry>
       <material name="grey">

File: catkin_ws/src/o2ac_scene_description/urdf/components/nut_holder.xacro (robot description, xacro)
@@ -21,7 +21,13 @@
     </visual>
     <collision>
-      <origin rpy="${pi/2} 0 ${-pi/2}" xyz="0 0 0.0"/>
+      <origin rpy="0 0 0" xyz="${-.02/2} ${-.06/2} ${.01/2}"/>
       <geometry>
-        <mesh filename="${mesh_file}" scale=".001 .001 .001"/>
+        <box size=".02 .06 .01"/>
+      </geometry>
+    </collision>
+    <collision>
+      <origin rpy="0 0 0" xyz="${-.02/2} ${-.06/2} ${.05/2}"/>
+      <geometry>
+        <cylinder length="0.05" radius="0.005"/>
       </geometry>
     </collision>

File: catkin_ws/src/o2ac_scene_description/urdf/components/taskboard.xacro (robot description, xacro)
@@ -6,10 +6,10 @@
   <link name="${boardname}_base">
     <inertial>
-      <origin rpy="${-pi/2} 0 ${pi/2}" xyz="0 0 0.0"/>
+      <origin rpy="${-pi/2} 0 ${pi/2}" xyz="0 0 0.01"/>
       <mass value="1.0"/>
       <inertia ixx="1.0" ixy="0" ixz="0" iyy="1.0" iyz="0" izz="1.0"/>
     </inertial>
     <visual>
-      <origin rpy="${-pi/2} 0 ${pi/2}" xyz="0 0 0.0"/>
+      <origin rpy="${-pi/2} 0 ${pi/2}" xyz=".12 0 0.01"/>
       <geometry>
         <mesh filename="${mesh_file_base}" scale=".001 .001 .001"/>
@@ -20,5 +20,5 @@
     </visual>
     <collision>
-      <origin rpy="${-pi/2} 0 ${pi/2}" xyz="0 0 0.0"/>
+      <origin rpy="${-pi/2} 0 ${pi/2}" xyz=".12 0 0.01"/>
       <geometry>
         <mesh filename="${mesh_file_base}" scale=".001 .001 .001"/>
@@ -51,5 +51,5 @@
     <parent link="${boardname}_base" />
     <child link = "${boardname}_plate" />
-    <origin rpy="0 0 0" xyz="-0.06 0.0 0.0"/>
+    <origin rpy="0 0 0" xyz="0.058 0.0 0.01"/>
   </joint>
   <!-- ========== Shaft, pulleys, bearing -->
@@ -81,4 +81,5 @@
     <origin rpy="0 0 0" xyz="${0.025+.008} 0.165 0.12"/>
   </xacro:assy_part_07>
+  <!-- The large pulley -->
   <joint name="${boardname}_small_pulley" type="fixed">
     <parent link="${boardname}_plate" />
@@ -103,5 +104,5 @@
     </collision>
   </link>
-  <!-- 16.5 -->
+  <!-- The large pulley -->
   <joint name="${boardname}_large_pulley" type="fixed">
     <parent link="${boardname}_plate" />
@@ -163,30 +164,32 @@
   </joint>
   <link name="${boardname}_bearing_target_link"/>
-  <!-- I wrote these bearing screw frames out, but actually they should
-      come from the subframes of the bearing that will be placed there. If they are used at all. -->
-  <!-- <joint name="${boardname}_bearing_screw_1_joint" type="fixed">
-    <parent link="${boardname}_plate"/>
-    <child link="${boardname}_bearing_screw_1_link"/>
-    <origin rpy="0 0 ${pi}" xyz="${.025+.008} ${0.034} ${0.12+.022}"/>
+  <!-- Screw positions of the base plate -->
+  <xacro:property name="base_l" value="0.2" />
+  <xacro:property name="base_w" value="0.12" />
+  <xacro:property name="d0" value="0.01" />
+  <joint name="${boardname}_base_screw_1_joint" type="fixed">
+    <parent link="${boardname}_base"/>
+    <child link="${boardname}_base_screw_1_link"/>
+    <origin rpy="0 ${pi/2} 0" xyz="${base_w-d0} ${base_l-d0} .01"/>
   </joint>
-  <link name="${boardname}_bearing_screw_1_link"/>
-  <joint name="${boardname}_bearing_screw_2_joint" type="fixed">
-    <parent link="${boardname}_plate"/>
-    <child link="${boardname}_bearing_screw_2_link"/>
-    <origin rpy="0 0 ${pi}" xyz="${.025+.008} ${0.034} ${0.12-.022}"/>
+  <link name="${boardname}_base_screw_1_link"/>
+  <joint name="${boardname}_base_screw_2_joint" type="fixed">
+    <parent link="${boardname}_base"/>
+    <child link="${boardname}_base_screw_2_link"/>
+    <origin rpy="0 ${pi/2} 0" xyz="${d0} ${base_l-d0} .01"/>
   </joint>
-  <link name="${boardname}_bearing_screw_2_link"/>
-  <joint name="${boardname}_bearing_screw_3_joint" type="fixed">
-    <parent link="${boardname}_plate"/>
-    <child link="${boardname}_bearing_screw_3_link"/>
-    <origin rpy="0 0 ${pi}" xyz="${.025+.008} ${0.034+.022} ${0.12}"/>
+  <link name="${boardname}_base_screw_2_link"/>
+  <joint name="${boardname}_base_screw_3_joint" type="fixed">
+    <parent link="${boardname}_base"/>
+    <child link="${boardname}_base_screw_3_link"/>
+    <origin rpy="0 ${pi/2} 0" xyz="${base_w-d0} ${d0} .01"/>
   </joint>
-  <link name="${boardname}_bearing_screw_3_link"/>
-  <joint name="${boardname}_bearing_screw_4_joint" type="fixed">
-    <parent link="${boardname}_plate"/>
-    <child link="${boardname}_bearing_screw_4_link"/>
-    <origin rpy="0 0 ${pi}" xyz="${.025+.008} ${0.034-.022} ${0.12}"/>
+  <link name="${boardname}_base_screw_3_link"/>
+  <joint name="${boardname}_base_screw_4_joint" type="fixed">
+    <parent link="${boardname}_base"/>
+    <child link="${boardname}_base_screw_4_link"/>
+    <origin rpy="0 ${pi/2} 0" xyz="${d0} ${d0} .01"/>
   </joint>
-  <link name="${boardname}_bearing_screw_4_link"/> -->
+  <link name="${boardname}_base_screw_4_link"/>
   </xacro:macro>
   <!-- Add additional links for us to plan with.-->

File: catkin_ws/src/o2ac_scene_description/urdf/components/tools.xacro (robot description, xacro)
@@ -175,7 +175,13 @@
     </visual>
     <collision>
-      <origin rpy="0 0 0" xyz="0 ${bit_cushion_to_axis - .02} .0275"/>
+      <origin rpy="0 0 0" xyz="0 ${-bit_cushion_to_axis + .02} .0275"/>
       <geometry>
         <box size=".026 .04 .055"/>
+      </geometry>
+    </collision>
+    <collision>
+      <origin rpy="0 0 0" xyz="0 0 ${-.12/2}"/>
+      <geometry>
+        <cylinder length=".12" radius=".01"/>
       </geometry>
     </collision>
@@ -202,7 +208,13 @@
     </visual>
     <collision>
-      <origin rpy="0 0 0" xyz="0 ${bit_cushion_to_axis - .02} .0275"/>
+      <origin rpy="0 0 0" xyz="0 ${-bit_cushion_to_axis + .02} .0275"/>
       <geometry>
         <box size=".026 .04 .055"/>
+      </geometry>
+    </collision>
+    <collision>
+      <origin rpy="0 0 0" xyz="0 0 ${-.1/2}"/>
+      <geometry>
+        <cylinder length=".1" radius=".01"/>
       </geometry>
     </collision>
@@ -226,10 +238,4 @@
     <origin xyz="0.0 0.0 0.0" rpy="0.0 ${pi} ${pi/2}" />
   </joint>
-  <link name="belt_tool_pickup_link"/>
-  <joint name="belt_tool_pickup_joint" type="fixed">
-    <parent link="belt_tool_link" />
-    <child link="belt_tool_pickup_link" />
-    <origin xyz="0.0 0.0 0.0" rpy="0.0 ${pi} ${pi/2}" />
-  </joint>
   <link name="nut_tool_m6_pickup_link"/>
   <joint name="nut_tool_m6_pickup_joint" type="fixed">
@@ -258,7 +264,7 @@
     </visual>
     <collision>
-      <origin rpy="0 0 0" xyz="0 0 0"/>
-      <geometry>
-        <box size=".001 .001 .001"/>
+      <origin rpy="0 0 0" xyz="${.05/2} 0 ${-.045/2}"/>
+      <geometry>
+        <box size=".05 .05 .045"/>
       </geometry>
     </collision>
@@ -284,16 +290,30 @@
       </material>
     </visual>
-    <collision>
-      <origin rpy="0 0 0" xyz="0 0 0"/>
-      <geometry>
-        <box size=".026 .04 .055"/>
-      </geometry>
-    </collision>
-  </link>
-  <joint name="belt_tool_to_holder" type="fixed">
+    <!-- The graspable part -->
+    <collision>
+      <origin rpy="0 0 0" xyz="${.04/2} 0 ${-.01}"/>
+      <geometry>
+        <box size=".04 .03 .055"/>
+      </geometry>
+    </collision>
+    <!-- The bottom part -->
+    <collision>
+      <origin rpy="0 0 0" xyz="${.02} 0 ${-.03-.1/2}"/>
+      <geometry>
+        <box size=".01 .035 .1"/>
+      </geometry>
+    </collision>
+  </link>
+  <joint name="belt_tool_to_holder_joint" type="fixed">
     <parent link="belt_tool_holder" />
     <child link="belt_tool_link" />
     <origin xyz="0 0 0" rpy="0 0 0" />
   </joint>
+  <link name="belt_tool_pickup_link"/>
+  <joint name="belt_holder_to_pickup_link_joint" type="fixed">
+    <parent link="belt_tool_link" />
+    <child link="belt_tool_pickup_link" />
+    <origin xyz=".02 0 -.01" rpy="0 ${pi/2} 0" />
+  </joint>
   <!-- Plunger tool -->
   <link name="plunger_tool_holder">
@@ -308,7 +328,7 @@
     </visual>
     <collision>
-      <origin rpy="0 0 0" xyz="0 0 0"/>
-      <geometry>
-        <box size=".001 .001 .001"/>
+      <origin rpy="0 0 0" xyz="${.05/2} 0 ${-.045/2}"/>
+      <geometry>
+        <box size=".05 .05 .045"/>
       </geometry>
     </collision>
@@ -335,14 +355,26 @@
     </visual>
     <collision>
-      <origin rpy="0 0 0" xyz="0 0 0"/>
-      <geometry>
-        <box size=".026 .04 .055"/>
-      </geometry>
-    </collision>
-  </link>
-  <joint name="plunger_tool_to_holder" type="fixed">
+      <origin rpy="0 0 0" xyz="${.04/2} 0 ${-.01}"/>
+      <geometry>
+        <box size=".04 .03 .055"/>
+      </geometry>
+    </collision>
+    <collision>
+      <origin rpy="0 0 0" xyz="${.02} 0 ${-.03-.08/2}"/>
+      <geometry>
+        <cylinder length=".08" radius=".01"/>
+      </geometry>
+    </collision>
+  </link>
+  <joint name="plunger_tool_to_holder_joint" type="fixed">
     <parent link="plunger_tool_holder" />
     <child link="plunger_tool_link" />
     <origin xyz="0 0 0" rpy="0 0 0" />
   </joint>
+  <link name="plunger_tool_pickup_link"/>
+  <joint name="plunger_holder_to_pickup_link_joint" type="fixed">
+    <parent link="plunger_tool_link" />
+    <child link="plunger_tool_pickup_link" />
+    <origin xyz=".02 0 -.01" rpy="0 ${pi/2} 0" />
+  </joint>
 </robot>

File: catkin_ws/src/o2ac_scene_description/urdf/components/washer_holder.xacro (robot description, xacro)
@@ -21,7 +21,13 @@
     </visual>
     <collision>
-      <origin rpy="${pi/2} 0 ${-pi/2}" xyz="0 0 0.0"/>
+      <origin rpy="0 0 0" xyz="${-.02/2} ${-.06/2} ${.01/2}"/>
       <geometry>
-        <mesh filename="${mesh_file}" scale=".001 .001 .001"/>
+        <box size=".02 .06 .01"/>
+      </geometry>
+    </collision>
+    <collision>
+      <origin rpy="0 0 0" xyz="${-.02/2} ${-.06/2} ${.05/2}"/>
+      <geometry>
+        <cylinder length="0.05" radius="0.005"/>
       </geometry>
     </collision>
@@ -35,7 +41,13 @@
     <parent link="${partname}"/>
     <child link="${partname}_collar_link"/>
-    <origin rpy="0 0 0" xyz="-0.01 -.03 0.04"/>
+    <origin rpy="0 ${pi/2} 0" xyz="-0.01 -.03 0.04"/>
   </joint>
   <link name="${partname}_collar_link"/>
+  <joint name="${partname}_tip_joint" type="fixed">
+    <parent link="${partname}_collar_link"/>
+    <child link="${partname}_tip_link"/>
+    <origin rpy="0 0 0" xyz="-0.01 0 0"/>
+  </joint>
+  <link name="${partname}_tip_link"/>
   </xacro:macro>
 </robot>

File: catkin_ws/src/o2ac_scene_description/urdf/components/wrist_cameras.xacro (robot description, xacro)
@@ -25,5 +25,5 @@
         <origin rpy="0 0 0" xyz="-.01 0.0 .035"/>
         <geometry>
-          <box size=".03 .12 .08"/>
+          <box size=".03 .15 .08"/>
         </geometry>
       </collision>

File: catkin_ws/src/o2ac_scene_description/urdf/taskboard_scene.xacro (robot description, xacro)
@@ -3,5 +3,5 @@
   <xacro:include filename="$(find o2ac_scene_description)/urdf/components/taskboard.xacro" />
   <xacro:taskboard boardname="taskboard" parent="attached_base_origin_link">
-    <origin xyz=".12 0 0" rpy="0 0 0" />
+    <origin xyz="0 0 0" rpy="0 0 0" />
   </xacro:taskboard>
 </robot>

Commit message: Update camera launch file, scene

File: catkin_ws/src/o2ac_scene_description/urdf/components/base_fixture.xacro (robot description, xacro)
@@ -25,14 +25,14 @@
     <!-- The long stopper bar -->
     <collision>
-      <origin rpy="0 0 0" xyz="${width-.02/2} ${length-.20/2} ${.08+.03/2}"/>
+      <origin rpy="0 0 0" xyz="${width-.02/2} ${length-.22/2} ${.08+.02/2}"/>
       <geometry>
-        <box size="${.02} ${.20} 0.03"/>
+        <box size="${.02} ${.22} ${0.02}"/>
       </geometry>
     </collision>
     <!-- The short stopper bar -->
     <collision>
-      <origin rpy="0 0 0" xyz="${width-.16/2} ${length-.02/2} ${.08+.03/2}"/>
+      <origin rpy="0 0 0" xyz="${width-.18/2} ${length-.02/2} ${.08+.02/2}"/>
       <geometry>
-        <box size="${.16} ${.02} 0.03"/>
+        <box size="${.18} ${.02} ${0.02}"/>
       </geometry>
     </collision>

Commit message: Fix assembly position in fixture

File: catkin_ws/src/o2ac_scene_description/urdf/components/base_fixture.xacro (robot description, xacro)
@@ -138,7 +138,13 @@
     <parent link="base_fixture_top"/>
     <child link="attached_base_origin_link"/>
+    <origin rpy="${pi/2} 0 ${-pi/2}" xyz=".22 .3 0.085"/>
+  </joint>
+  <link name="attached_base_origin_link"/>
+  <!-- <joint name="attached_base_origin_joint" type="fixed">
+    <parent link="base_fixture_top"/>
+    <child link="attached_base_origin_link"/>
     <origin rpy="0.0 0 0" xyz=".1 .1 0.085"/>
   </joint>
-  <link name="attached_base_origin_link"/>
+  <link name="attached_base_origin_link"/> -->
 <!--
   <joint name="base_fixture_corner_2_joint" type="fixed">

Commit message: Repair taskboard position

File: catkin_ws/src/o2ac_scene_description/urdf/components/base_fixture.xacro (robot description, xacro)
@@ -141,10 +141,10 @@
   </joint>
   <link name="attached_base_origin_link"/>
-  <!-- <joint name="attached_base_origin_joint" type="fixed">
+  <joint name="attached_base_origin_back_joint" type="fixed">
     <parent link="base_fixture_top"/>
-    <child link="attached_base_origin_link"/>
+    <child link="attached_base_origin_back_link"/>
     <origin rpy="0.0 0 0" xyz=".1 .1 0.085"/>
   </joint>
-  <link name="attached_base_origin_link"/> -->
+  <link name="attached_base_origin_back_link"/>
 <!--
   <joint name="base_fixture_corner_2_joint" type="fixed">

File: catkin_ws/src/o2ac_scene_description/urdf/taskboard_scene.xacro (robot description, xacro)
@@ -2,5 +2,5 @@
 <robot xmlns:xacro="http://www.ros.org/wiki/xacro" name="taskboard_scene">
   <xacro:include filename="$(find o2ac_scene_description)/urdf/components/taskboard.xacro" />
-  <xacro:taskboard boardname="taskboard" parent="attached_base_origin_link">
+  <xacro:taskboard boardname="taskboard" parent="attached_base_origin_back_link">
     <origin xyz="0 0 0" rpy="0 0 0" />
   </xacro:taskboard>
