Commit message: Prepare screw picking (switch M4/M3 tool, set robot poses etc)

File: catkin_ws/src/o2ac_scene_description/urdf/components/screw_feeder.xacro (robot description, xacro)
@@ -72,5 +72,5 @@
     <parent link="${feedername}_link"/>
     <child link="${feedername}_outlet_link"/>
-    <origin rpy="0.0 ${pi/2} 0.0" xyz="${length-.01} ${width/2} ${height/2}"/>
+    <origin rpy="0.0 ${pi/2} ${pi}" xyz="${length-.01} ${width/2} ${height/2}"/>
   </joint>
   <link name="${feedername}_outlet_link"/>

File: catkin_ws/src/o2ac_scene_description/urdf/components/tools.xacro (robot description, xacro)
@@ -196,5 +196,5 @@
     <parent link="screw_tool_holder_long" />
     <child link="screw_tool_m4_link" />
-    <origin xyz="-0.15 ${tool_offset} 0.004" rpy="0.0 0.0 0.0" />
+    <origin xyz="-0.25 ${tool_offset} 0.004" rpy="0.0 0.0 0.0" />
   </joint>
   <link name="screw_tool_m3_link">
@@ -235,5 +235,5 @@
     <parent link="screw_tool_holder_long" />
     <child link="screw_tool_m3_link" />
-    <origin xyz="-0.25 ${tool_offset} 0.004" rpy="0.0 0.0 0.0" />
+    <origin xyz="-0.15 ${tool_offset} 0.004" rpy="0.0 0.0 0.0" />
   </joint>
   <!-- Extra links to position the gripper more easily -->

File: catkin_ws/src/o2ac_scene_description/urdf/o2ac_environment.xacro (robot description, xacro)
@@ -22,9 +22,13 @@
   <xacro:include filename="$(find o2ac_scene_description)/urdf/components/screw_feeder.xacro" />
   <xacro:screw_feeder feedername="m4_feeder" parent="workspace_center">
-    <origin xyz="-.55 .05 -0.043" rpy="0 0 0" />
+    <origin xyz="-.511 -.13 -0.043" rpy="0 0 0" />
+    <!-- <origin xyz="-.55 .05 -0.043" rpy="0 0 0" />    -->
   </xacro:screw_feeder>
+  <!-- -0.016241; 0.18032; -0.039283 -->
   <xacro:screw_feeder feedername="m3_feeder" parent="workspace_center">
-    <origin xyz="-.55 -.15 -0.043" rpy="0 0 0" />
+    <origin xyz="-.512 0 -0.043" rpy="0 0 0" />
+    <!-- <origin xyz="-.55 -.15 -0.043" rpy="0 0 0" />    -->
   </xacro:screw_feeder>
+  <!-- -0.018032; -0.15035; -0.038212 -->
   <!-- Base fixture -->
   <xacro:include filename="$(find o2ac_scene_description)/urdf/components/base_fixture.xacro" />

Commit message: Remove collision geometry from screw feeders

File: catkin_ws/src/o2ac_scene_description/urdf/components/screw_feeder.xacro (robot description, xacro)
@@ -1,5 +1,5 @@
 <?xml version="1.0" ?>
 <robot xmlns:xacro="http://www.ros.org/wiki/xacro" name="screw_feeder">
-  <xacro:macro name="screw_feeder" params="feedername parent *origin">
+  <xacro:macro name="screw_feeder" params="feedername parent with_collision_geometry:=true *origin">
   <!-- This creates a screw feeder (roughly) with the origin in the back right corner. -->
   <!-- This is the feeder: https://www.monotaro.com/g/02001466/ -->
@@ -25,10 +25,12 @@
       </material>
     </visual>
-    <collision>
-      <origin rpy="0 0 0" xyz="${(length-.05)/2} ${width/2} ${height/2}"/>
-      <geometry>
-        <box size="${length-.05} ${width} ${height}"/>
-      </geometry>
-    </collision>
+    <xacro:if value="${with_collision_geometry}">
+      <collision>
+        <origin rpy="0 0 0" xyz="${(length-.05)/2} ${width/2} ${height/2}"/>
+        <geometry>
+          <box size="${length-.05} ${width} ${height}"/>
+        </geometry>
+      </collision>
+    </xacro:if>
     <!-- Front side -->
     <visual>
@@ -41,10 +43,12 @@
       </material>
     </visual>
-    <collision>
-      <origin rpy="0 0 0" xyz="${(length-.025)} ${width/2} ${height/4}"/>
-      <geometry>
-        <box size="${.05} ${width} ${height/2}"/>
-      </geometry>
-    </collision>
+    <xacro:if value="${with_collision_geometry}">
+      <collision>
+        <origin rpy="0 0 0" xyz="${(length-.025)} ${width/2} ${height/4}"/>
+        <geometry>
+          <box size="${.05} ${width} ${height/2}"/>
+        </geometry>
+      </collision>
+    </xacro:if>
     <!-- The screw output area -->
     <visual>
@@ -57,10 +61,12 @@
       </material>
     </visual>
-    <collision>
-      <origin rpy="0 0 0" xyz="${(length-.025)} ${width/2} ${height/2}"/>
-      <geometry>
-        <box size="${.05} ${.02} ${.005}"/>
-      </geometry>
-    </collision>
+    <xacro:if value="${with_collision_geometry}">
+      <collision>
+        <origin rpy="0 0 0" xyz="${(length-.025)} ${width/2} ${height/2}"/>
+        <geometry>
+          <box size="${.05} ${.02} ${.005}"/>
+        </geometry>
+      </collision>
+    </xacro:if>
   </link>
   <joint name="${feedername}_joint" type="fixed">

File: catkin_ws/src/o2ac_scene_description/urdf/o2ac_environment.xacro (robot description, xacro)
@@ -21,8 +21,8 @@
   <!-- Add screw feeders -->
   <xacro:include filename="$(find o2ac_scene_description)/urdf/components/screw_feeder.xacro" />
-  <xacro:screw_feeder feedername="m3_feeder" parent="workspace_center">
+  <xacro:screw_feeder feedername="m3_feeder" parent="workspace_center" with_collision_geometry="false">
     <origin xyz="-.512 -.1525 -0.023" rpy="0 0 0" />
   </xacro:screw_feeder>
-  <xacro:screw_feeder feedername="m4_feeder" parent="workspace_center">
+  <xacro:screw_feeder feedername="m4_feeder" parent="workspace_center" with_collision_geometry="false">
     <origin xyz="-.514 .004 -0.023" rpy="0 0 0" />
   </xacro:screw_feeder>
