Commit message: Update vgroove aid meshes and collision

File: catkin_ws/src/o2ac_scene_description/urdf/components/vgroove_aid.xacro (robot description, xacro)
@@ -19,16 +19,7 @@
     </visual>
     <collision>
-      <origin rpy="0 0 0" xyz="0 0.02 0.025"/>
-      <!-- <geometry>
-        <box size=".04 .04 .02"/>
-      </geometry> -->
+      <origin rpy="${pi/2} 0 ${pi/2}" xyz="0 0 0.0"/>
       <geometry>
-        <box size=".04 .005 .05"/>
-      </geometry>
-    </collision>
-    <collision>
-      <origin rpy="0 0 0" xyz="0 -.02 0.025"/>
-      <geometry>
-        <box size=".04 .005 .05"/>
+        <mesh filename="${mesh_file}" scale=".001 .001 .001"/>
       </geometry>
     </collision>

Commit message: Update vgroove aid meshes and links

File: catkin_ws/src/o2ac_scene_description/urdf/components/vgroove_aid.xacro (robot description, xacro)
@@ -33,5 +33,5 @@
     <parent link="${jigname}_link"/>
     <child link="${jigname}_drop_point_link"/>
-    <origin rpy="0 ${pi/2} ${-pi/2}" xyz="0 0 0.04"/>
+    <origin rpy="0 ${pi/2} ${-pi/2}" xyz="0 0 0.05"/>
   </joint>
   <link name="${jigname}_drop_point_link"/>

File: catkin_ws/src/o2ac_scene_description/urdf/o2ac_environment.xacro (robot description, xacro)
@@ -48,10 +48,10 @@
   <xacro:include filename="$(find o2ac_scene_description)/urdf/components/vgroove_aid.xacro" />
   <xacro:vgroove_aid jigname="vgroove_aid" parent="b_bot_base_link">
-    <origin xyz="-0.2927 0.17214 0.0" rpy="0 0 0" />
+    <origin xyz="-0.2927 0.17214 0.0" rpy="0 0 ${pi/2}" />
   </xacro:vgroove_aid>
   <!-- The second vgroove at the back (for the motor)-->
-  <xacro:vgroove_aid jigname="vgroove_aid_motor" parent="b_bot_base_link">
-    <origin xyz="-0.225 -0.210 0.001" rpy="0 0 0" />
-  </xacro:vgroove_aid>
+  <!-- <xacro:vgroove_aid jigname="vgroove_aid_motor" parent="b_bot_base_link">
+    <origin xyz="-0.26 -0.28 0.001" rpy="0 0 0" />
+  </xacro:vgroove_aid>  -->
   <xacro:include filename="$(find o2ac_scene_description)/urdf/components/simple_holder.xacro" />
   <xacro:simple_holder partname="simple_holder" parent="workspace_center">
