Commit message: Use SubscriberFilter for aist_aruco_ros and cleanup launch files

File: catkin_ws/src/o2ac_scene_description/urdf/components/ft300.urdf.xacro (robot description, xacro)
@@ -4,13 +4,14 @@
   <xacro:property name="ft300_length" value="0.0360"/>
   <xacro:macro name="ft300" params="prefix parent *origin">
-    <link name="${prefix}ft300_link">
+    <link name="${prefix}base_link">
       <visual>
         <origin xyz="${ft300_length} 0 0" rpy="${pi} ${pi/2} 0"/>
-	<geometry>
-          <mesh filename="package://o2ac_scene_description/meshes/ft300.stl" scale="0.001 0.001 0.001"/>
-	</geometry>
-	<material name="Black">
-	  <color rgba="0.2 0.2 0.2 1"/>
-	</material>
+      	<geometry>
+          <mesh filename="package://o2ac_scene_description/meshes/ft300.stl"
+		scale="0.001 0.001 0.001"/>
+      	</geometry>
+      	<material name="Black">
+      	  <color rgba="0.2 0.2 0.2 1"/>
+      	</material>
       </visual>
       <!-- <visual> -->
@@ -33,17 +34,17 @@
     <joint name="${prefix}ft300_joint" type="fixed">
       <parent link="${parent}"/>
-      <child  link="${prefix}ft300_link"/>
+      <child  link="${prefix}base_link"/>
       <xacro:insert_block name="origin"/>
     </joint>
-    <link name="${prefix}ft300_flange_link"/>
-    <joint name="${prefix}ft300_flange_joint" type="fixed">
-      <parent link="${prefix}ft300_link"/>
-      <child  link="${prefix}ft300_flange_link"/>
+    <link name="${prefix}flange_link"/>
+    <joint name="${prefix}flange_joint" type="fixed">
+      <parent link="${prefix}base_link"/>
+      <child  link="${prefix}flange_link"/>
       <origin xyz="${ft300_length} 0 0" rpy="0 0 0"/>
     </joint>
-    <link name="${prefix}ft300_wrench_link"/>
-    <joint name="${prefix}ft300_wrench_joint" type="fixed">
-      <parent link="${prefix}ft300_flange_link"/>
-      <child  link="${prefix}ft300_wrench_link"/>
+    <link name="${prefix}wrench_link"/>
+    <joint name="${prefix}wrench_joint" type="fixed">
+      <parent link="${prefix}flange_link"/>
+      <child  link="${prefix}wrench_link"/>
       <origin xyz="0 0 0" rpy="${-pi/2} 0 ${-pi/2}"/>
     </joint>
