Commit message: Screw bearing to taskboard

File: catkin_ws/src/o2ac_scene_description/urdf/components/o2ac_end_effector.urdf.xacro (robot description, xacro)
@@ -19,43 +19,48 @@
     <!-- Screw tool tip frames. X-axis points along the screw into the hole. -->
     <!-- Offset of the gripper tooltips -->
-    <xacro:property name="dx" value="-.03"/>
+    <joint name="${prefix}tool_intermediate_joint" type="fixed">
+      <parent link="${prefix}robotiq_85_tip_link"/>
+      <child link="${prefix}tool_intermediate_link"/>
+      <origin rpy="${pi} 0.0 0.0" xyz="-.03 0.0 0.0"/>
+    </joint>
+    <link name="${prefix}tool_intermediate_link"/>
     <joint name="${prefix}robotiq_85_screw_tool_m6_tip_joint" type="fixed">
-      <parent link="${prefix}robotiq_85_tip_link"/>
+      <parent link="${prefix}tool_intermediate_link"/>
       <child link="${prefix}screw_tool_m6_tip_link"/>
-      <origin rpy="0.0 ${pi/2} 0.0" xyz="${dx} 0.0 -0.135 "/>
+      <origin rpy="0.0 ${pi/2} 0.0" xyz="0.0 0.0 -0.135 "/>
     </joint>
     <link name="${prefix}screw_tool_m6_tip_link"/>
     <joint name="${prefix}robotiq_85_nut_tool_m6_tip_joint" type="fixed">
-      <parent link="${prefix}robotiq_85_tip_link"/>
+      <parent link="${prefix}tool_intermediate_link"/>
       <child link="${prefix}nut_tool_m6_tip_link"/>
-      <origin rpy="0.0 ${pi/4} 0.0" xyz="${dx} 0.0 -0.12 "/>
+      <origin rpy="0.0 ${pi/4} 0.0" xyz="0.0 0.0 -0.12 "/>
     </joint>
     <link name="${prefix}nut_tool_m6_tip_link"/>
     <joint name="${prefix}robotiq_85_screw_tool_m4_tip_joint" type="fixed">
-      <parent link="${prefix}robotiq_85_tip_link"/>
+      <parent link="${prefix}tool_intermediate_link"/>
       <child link="${prefix}screw_tool_m4_tip_link"/>
-      <origin rpy="0.0 ${pi/2} 0.0" xyz="${dx-.002} 0.0 -0.146 "/>
+      <origin rpy="0.0 ${pi/2} 0.0" xyz="-.002 0.0 -0.146 "/>
     </joint>
     <link name="${prefix}screw_tool_m4_tip_link"/>
     <joint name="${prefix}robotiq_85_screw_tool_m3_tip_joint" type="fixed">
-      <parent link="${prefix}robotiq_85_tip_link"/>
+      <parent link="${prefix}tool_intermediate_link"/>
       <child link="${prefix}screw_tool_m3_tip_link"/>
-      <origin rpy="0.0 ${pi/2} 0.0" xyz="${dx-.004} 0.0 -0.125 "/>
+      <origin rpy="0.0 ${pi/2} 0.0" xyz=".015 0.0 -0.14 "/>
     </joint>
     <link name="${prefix}screw_tool_m3_tip_link"/>
     <joint name="${prefix}robotiq_85_set_screw_tool_tip_joint" type="fixed">
-      <parent link="${prefix}robotiq_85_tip_link"/>
+      <parent link="${prefix}tool_intermediate_link"/>
       <child link="${prefix}set_screw_tool_tip_link"/>
-      <origin rpy="0.0 ${pi/2} 0.0" xyz="${dx+.01} 0.0 -0.085 "/>
+      <origin rpy="0.0 ${pi/2} 0.0" xyz=".01 0.0 -0.085 "/>
     </joint>
     <link name="${prefix}set_screw_tool_tip_link"/>
     <joint name="${prefix}robotiq_85_suction_tool_tip_joint" type="fixed">
-      <parent link="${prefix}robotiq_85_tip_link"/>
+      <parent link="${prefix}tool_intermediate_link"/>
       <child link="${prefix}suction_tool_tip_link"/>
-      <origin rpy="0.0 ${pi/2} 0.0" xyz="${dx+.02} 0.0 -0.131 "/>
+      <origin rpy="0.0 ${pi/2} 0.0" xyz=".02 0.0 -0.131 "/>
     </joint>
     <link name="${prefix}suction_tool_tip_link"/>
     <joint name="${prefix}dual_suction_gripper_pad_joint" type="fixed">
-      <parent link="${prefix}suction_tool_tip_link"/>
+      <parent link="${prefix}tool_intermediate_link"/>
       <child link="${prefix}dual_suction_gripper_pad_link"/>
       <origin rpy="0.0 0 0.0" xyz="0 0 0 "/>

Commit message: Fix set screw tool frame

File: catkin_ws/src/o2ac_scene_description/urdf/components/o2ac_end_effector.urdf.xacro (robot description, xacro)
@@ -69,15 +69,9 @@
     <link name="${prefix}screw_tool_m3_tip_link"/>
     <joint name="${prefix}robotiq_85_set_screw_tool_tip_joint" type="fixed">
-      <parent link="${prefix}robotiq_85_tip_link"/>
+      <parent link="${prefix}tool_intermediate_link"/>
       <child link="${prefix}set_screw_tool_tip_link"/>
-      <origin rpy="0 0 0" xyz=".0049 0 0.01"/>
+      <origin rpy="0 0 0" xyz="0.0725 0 0.009"/>
     </joint>
     <link name="${prefix}set_screw_tool_tip_link"/>
-    <joint name="${prefix}dual_suction_gripper_pad_joint" type="fixed">
-      <parent link="${prefix}tool_intermediate_link"/>
-      <child link="${prefix}dual_suction_gripper_pad_link"/>
-      <origin rpy="0 0 0" xyz="0 0 0 "/>
-    </joint>
-    <link name="${prefix}dual_suction_gripper_pad_link"/>
   </xacro:macro>
 </robot>

Commit message: Fix end effector tool frames

File: catkin_ws/src/o2ac_scene_description/urdf/components/o2ac_end_effector.urdf.xacro (robot description, xacro)
@@ -53,5 +53,5 @@
       <parent link="${prefix}tool_intermediate_link"/>
       <child link="${prefix}nut_tool_m6_tip_link"/>
-      <origin rpy="0 0 0" xyz="0.12 0 0 "/>
+      <origin rpy="0 0 0" xyz="0.107 0 -0.0075 "/>
     </joint>
     <link name="${prefix}nut_tool_m6_tip_link"/>
@@ -71,5 +71,5 @@
       <parent link="${prefix}tool_intermediate_link"/>
       <child link="${prefix}set_screw_tool_tip_link"/>
-      <origin rpy="0 0 0" xyz="0.0725 0 0.009"/>
+      <origin rpy="0 0 0" xyz="0.058 0 0.006"/>
     </joint>
     <link name="${prefix}set_screw_tool_tip_link"/>

File: catkin_ws/src/o2ac_scene_description/urdf/components/o2ac_end_effector_2F-140.urdf.xacro (robot description, xacro)
@@ -31,5 +31,5 @@
       <parent link="${prefix}tool_intermediate_link"/>
       <child link="${prefix}nut_tool_m6_tip_link"/>
-      <origin rpy="0 0 0" xyz="0.12 0 0 "/>
+      <origin rpy="0 0 0" xyz="0.107 0 -0.0075 "/>
     </joint>
     <link name="${prefix}nut_tool_m6_tip_link"/>
@@ -49,5 +49,5 @@
       <parent link="${prefix}tool_intermediate_link"/>
       <child link="${prefix}set_screw_tool_tip_link"/>
-      <origin rpy="0 0 0" xyz="0.0725 0 0.009"/>
+      <origin rpy="0 0 0" xyz="0.058 0 0.006"/>
     </joint>
     <link name="${prefix}set_screw_tool_tip_link"/>

Commit message: WIP: Add UR service to close popup, minor fixes

File: catkin_ws/src/o2ac_scene_description/urdf/components/o2ac_end_effector.urdf.xacro (robot description, xacro)
@@ -71,5 +71,5 @@
       <parent link="${prefix}tool_intermediate_link"/>
       <child link="${prefix}set_screw_tool_tip_link"/>
-      <origin rpy="0 0 0" xyz="0.058 0 0.006"/>
+      <origin rpy="0 0 0" xyz="0.068 0 0.0014"/>
     </joint>
     <link name="${prefix}set_screw_tool_tip_link"/>

Commit message: Housekeeping, clean up

File: catkin_ws/src/o2ac_scene_description/urdf/components/o2ac_end_effector.urdf.xacro (robot description, xacro)
@@ -8,5 +8,5 @@
         <origin rpy="0.0 0.0 0.0" xyz="0.01 0 0"/> <!-- This 0.01 offset is the Robotiq/UR coupling -->
     </xacro:robotiq_85_gripper>
-    <link name="${prefix}_coupling">
+    <link name="${prefix}coupling">
       <visual>
         <origin rpy="0 ${pi/2} 0" xyz=".005 0 0"/>
@@ -25,7 +25,7 @@
       </collision>
     </link>
-    <joint name="${prefix}_coupling_joint" type="fixed">
+    <joint name="${prefix}coupling_joint" type="fixed">
       <parent link="${parent}" />
-      <child link = "${prefix}_coupling" />
+      <child link = "${prefix}coupling" />
       <origin rpy="0 0 0" xyz="0 0 0"/>
     </joint>

Commit message: Improve bearing hole alignment

File: catkin_ws/src/o2ac_scene_description/urdf/components/o2ac_end_effector.urdf.xacro (robot description, xacro)
@@ -74,4 +74,12 @@
     </joint>
     <link name="${prefix}set_screw_tool_tip_link"/>
+    <!-- ========= -->
+    <!-- Add helper frames, e.g. for rotating bearing. -->
+    <joint name="${prefix}bearing_rotate_helper_joint" type="fixed">
+      <parent link="${prefix}robotiq_85_tip_link"/>
+      <child link="${prefix}bearing_rotate_helper_link"/>
+      <origin rpy="${radians(180)} ${radians(30)} 0" xyz="-.003 0 -0.011"/>
+    </joint>
+    <link name="${prefix}bearing_rotate_helper_link"/>
   </xacro:macro>
 </robot>

Commit message: Unify bearing & screw frame orientations

File: catkin_ws/src/o2ac_scene_description/urdf/components/o2ac_end_effector.urdf.xacro (robot description, xacro)
@@ -79,5 +79,5 @@
       <parent link="${prefix}gripper_tip_link"/>
       <child link="${prefix}bearing_rotate_helper_link"/>
-      <origin rpy="${radians(180)} ${radians(30)} 0" xyz="-.003 0 -0.011"/>
+      <origin rpy="0 ${radians(30)} 0" xyz="-.003 0 -0.011"/>
     </joint>
     <link name="${prefix}bearing_rotate_helper_link"/>

File: catkin_ws/src/o2ac_scene_description/urdf/components/taskboard.xacro (robot description, xacro)
@@ -167,5 +167,5 @@
     <parent link="${boardname}_plate"/>
     <child link="${boardname}_bearing_target_link"/>
-    <origin rpy="0 0 ${pi}" xyz=".025 0.034 0.12"/>
+    <origin rpy="${pi} 0 ${pi}" xyz=".025 0.034 0.12"/>
   </joint>
   <link name="${boardname}_bearing_target_link"/>
@@ -174,5 +174,5 @@
     <parent link="${boardname}_bearing_target_link"/>
     <child link="${boardname}_bearing_target_screw_1_link"/>
-    <origin rpy="${pi} 0 0" xyz="-.004 .022 0"/>
+    <origin rpy="0 0 0" xyz="-.004 .022 0"/>
   </joint>
   <link name="${boardname}_bearing_target_screw_1_link"/>
@@ -180,5 +180,5 @@
     <parent link="${boardname}_bearing_target_link"/>
     <child link="${boardname}_bearing_target_screw_2_link"/>
-    <origin rpy="${pi} 0 0" xyz="-.004 0 .022"/>
+    <origin rpy="0 0 0" xyz="-.004 0 .022"/>
   </joint>
   <link name="${boardname}_bearing_target_screw_2_link"/>
@@ -186,5 +186,5 @@
     <parent link="${boardname}_bearing_target_link"/>
     <child link="${boardname}_bearing_target_screw_3_link"/>
-    <origin rpy="${pi} 0 0" xyz="-.004 -0.022 0"/>
+    <origin rpy="0 0 0" xyz="-.004 -0.022 0"/>
   </joint>
   <link name="${boardname}_bearing_target_screw_3_link"/>
@@ -192,5 +192,5 @@
     <parent link="${boardname}_bearing_target_link"/>
     <child link="${boardname}_bearing_target_screw_4_link"/>
-    <origin rpy="${pi} 0 0" xyz="-.004 0 -0.022"/>
+    <origin rpy="0 0 0" xyz="-.004 0 -0.022"/>
   </joint>
   <link name="${boardname}_bearing_target_screw_4_link"/>

Commit message: Finetune pull from border with tool

File: catkin_ws/src/o2ac_scene_description/urdf/components/o2ac_end_effector.urdf.xacro (robot description, xacro)
@@ -41,4 +41,10 @@
     </joint>
     <link name="${prefix}gripper_tip_link"/>
+    <joint name="${prefix}plunger_tip_link_joint" type="fixed">
+      <parent link="${prefix}gripper_tip_link"/>
+      <child link="${prefix}plunger_tip_link"/>
+      <origin rpy="0 0 0" xyz=".10 0 0"/>
+    </joint>
+    <link name="${prefix}plunger_tip_link"/>
     <!-- ========= -->
     <!-- Add screw tool tip frames. X-axis points along the screw into the hole. -->

Commit message: Finetune tools

File: catkin_ws/src/o2ac_scene_description/urdf/components/o2ac_end_effector.urdf.xacro (robot description, xacro)
@@ -65,5 +65,5 @@
       <parent link="${prefix}tool_intermediate_link"/>
       <child link="${prefix}screw_tool_m4_tip_link"/>
-      <origin rpy="0 0 0" xyz=".141 0 0.005 "/>
+      <origin rpy="0 0 0" xyz=".146 0 0.005 "/>
     </joint>
     <link name="${prefix}screw_tool_m4_tip_link"/>
@@ -71,5 +71,5 @@
       <parent link="${prefix}tool_intermediate_link"/>
       <child link="${prefix}screw_tool_m3_tip_link"/>
-      <origin rpy="0 0 0" xyz=".14 0 .015 "/>
+      <origin rpy="0 0 0" xyz=".145 0 .015 "/>
     </joint>
     <link name="${prefix}screw_tool_m3_tip_link"/>

File: catkin_ws/src/o2ac_scene_description/urdf/components/o2ac_end_effector_2F-140.urdf.xacro (robot description, xacro)
@@ -57,5 +57,5 @@
       <parent link="${prefix}tool_intermediate_link"/>
       <child link="${prefix}screw_tool_m4_tip_link"/>
-      <origin rpy="0 0 0" xyz=".141 0 -0.005 "/>
+      <origin rpy="0 0 0" xyz=".146 0 -0.005 "/>
     </joint>
     <link name="${prefix}screw_tool_m4_tip_link"/>
@@ -63,5 +63,5 @@
       <parent link="${prefix}tool_intermediate_link"/>
       <child link="${prefix}screw_tool_m3_tip_link"/>
-      <origin rpy="0 0 0" xyz=".121 0 -.0045 "/>
+      <origin rpy="0 0 0" xyz=".128 0 -.0045 "/>
     </joint>
     <link name="${prefix}screw_tool_m3_tip_link"/>

File: catkin_ws/src/o2ac_scene_description/urdf/o2ac_environment.xacro (robot description, xacro)
@@ -39,8 +39,8 @@
   <xacro:include filename="$(find o2ac_scene_description)/urdf/components/screw_feeder.xacro" />
   <xacro:screw_feeder feedername="m3_feeder" parent="workspace_center" with_collision_geometry="false">
-    <origin xyz="-.511 -.154 0.028" rpy="0 0 0" />
+    <origin xyz="-.512 -.155 0.015" rpy="0 0 0" />
   </xacro:screw_feeder>
   <xacro:screw_feeder feedername="m4_feeder" parent="workspace_center" with_collision_geometry="false">
-    <origin xyz="-.514 .0035 0.03" rpy="0 0 0" />
+    <origin xyz="-.512 .0037 0.018" rpy="0 0 0" />
   </xacro:screw_feeder>
   <!-- Base fixture -->

Commit message: Finetuning taskboard

File: catkin_ws/src/o2ac_scene_description/urdf/components/o2ac_end_effector.urdf.xacro (robot description, xacro)
@@ -77,5 +77,5 @@
       <parent link="${prefix}tool_intermediate_link"/>
       <child link="${prefix}set_screw_tool_tip_link"/>
-      <origin rpy="0 0 0" xyz="0.068 0 0.0014"/>
+      <origin rpy="0 0 0" xyz="0.078 0 0.0014"/>
     </joint>
     <link name="${prefix}set_screw_tool_tip_link"/>

Commit message: Fix set screw procedure, adjust tool
This is still using the old tool, not the new one with rails.

File: catkin_ws/src/o2ac_scene_description/urdf/components/o2ac_end_effector.urdf.xacro (robot description, xacro)
@@ -77,5 +77,5 @@
       <parent link="${prefix}tool_intermediate_link"/>
       <child link="${prefix}set_screw_tool_tip_link"/>
-      <origin rpy="0 0 0" xyz="0.078 0 0.0014"/>
+      <origin rpy="0 0 0" xyz="0.076 0 0.0014"/>
     </joint>
     <link name="${prefix}set_screw_tool_tip_link"/>

Commit message: Calibrate m4 tool and motor panel 2021

File: catkin_ws/src/o2ac_scene_description/urdf/components/o2ac_end_effector.urdf.xacro (robot description, xacro)
@@ -65,5 +65,5 @@
       <parent link="${prefix}tool_intermediate_link"/>
       <child link="${prefix}screw_tool_m4_tip_link"/>
-      <origin rpy="0 0 0" xyz=".146 0 0.005 "/>
+      <origin rpy="0 0 0" xyz=".14689 0.0 0.003 "/>
     </joint>
     <link name="${prefix}screw_tool_m4_tip_link"/>

Commit message: WIP: insert motor cables
- Add cable tool equip/unequip
- Add insert cables w/wo tool
- TODO: check success or retry

File: catkin_ws/src/o2ac_scene_description/urdf/components/o2ac_end_effector.urdf.xacro (robot description, xacro)
@@ -41,4 +41,10 @@
     </joint>
     <link name="${prefix}gripper_tip_link"/>
+    <link name="${prefix}cable_tool_tip_link"/>
+    <joint name="${prefix}cable_tool_tip_link_joint" type="fixed">
+      <parent link="${prefix}gripper_tip_link"/>
+      <child link="${prefix}cable_tool_tip_link"/>
+      <origin rpy="0.0 0.0 0.0" xyz="${.03} 0.0 0.0"/>
+    </joint>
     <joint name="${prefix}plunger_tip_link_joint" type="fixed">
       <parent link="${prefix}gripper_tip_link"/>

File: catkin_ws/src/o2ac_scene_description/urdf/components/o2ac_end_effector_2F-140.urdf.xacro (robot description, xacro)
@@ -39,4 +39,10 @@
     </joint>
     <link name="${prefix}gripper_tip_link"/>
+    <link name="${prefix}cable_tool_tip_link"/>
+    <joint name="${prefix}cable_tool_tip_link_joint" type="fixed">
+      <parent link="${prefix}gripper_tip_link"/>
+      <child link="${prefix}cable_tool_tip_link"/>
+      <origin rpy="0.0 0.0 0.0" xyz="${.03} 0.0 0.0"/>
+    </joint>
     <!-- ========= -->
     <!-- Add screw tool tip frames. X-axis points along the screw into the hole. -->

File: catkin_ws/src/o2ac_scene_description/urdf/components/tools.xacro (robot description, xacro)
@@ -368,4 +368,31 @@
     <origin xyz="-0.11 -0.2 -0.015" rpy="0 0 0" />
   </joint>
+  <link name="cable_holder_link">
+      <inertial>
+      <origin rpy="0 0 0" xyz="0 0 0"/>
+      <mass value="1.0"/>
+      <inertia ixx="1" ixy="0" ixz="0" iyy="1" iyz="0" izz="1"/>
+    </inertial>
+    <visual>
+      <origin rpy="${-pi/2} 0 0" xyz="0.13 0.043 0.0225"/>
+      <geometry>
+        <mesh filename="package://o2ac_scene_description/meshes/cable_tool_holder_vertical.stl" scale="0.001 0.001 0.001"/>
+      </geometry>
+      <material name="white">
+        <color rgba=".9 .9 .9 1"/>
+      </material>
+    </visual>
+  </link>
+  <joint name="cable_holder_joint" type="fixed">
+    <parent link="workspace_center" />
+    <child link="cable_holder_link" />
+    <origin xyz="-0.49 -0.225 0.2" rpy="0 0 0" />
+  </joint>
+  <link name="cable_holder_pickup_link"/>
+  <joint name="cable_holder_pickup_joint" type="fixed">
+    <parent link="cable_holder_link" />
+    <child link="cable_holder_pickup_link" />
+    <origin xyz="0.1 0.0 0.015" rpy="0 ${pi/2} 0" />
+  </joint>
   <link name="nut_holder2_link"/>
   <joint name="nut_holder2_joint" type="fixed">

Commit message: Stub: Add belt threading parametrization

File: catkin_ws/src/o2ac_scene_description/urdf/components/o2ac_end_effector.urdf.xacro (robot description, xacro)
@@ -53,4 +53,10 @@
     </joint>
     <link name="${prefix}plunger_tip_link"/>
+    <joint name="${prefix}belt_hook_curve_link_joint" type="fixed">
+      <parent link="${prefix}gripper_tip_link"/>
+      <child link="${prefix}belt_hook_curve_link"/>
+      <origin rpy="0 0 ${-radians(10)}" xyz=".04 0 0"/>
+    </joint>
+    <link name="${prefix}belt_hook_curve_link"/>
     <!-- ========= -->
     <!-- Add screw tool tip frames. X-axis points along the screw into the hole. -->

Commit message: WIP: Calibrate b_bot M4 screw tool

File: catkin_ws/src/o2ac_scene_description/urdf/components/o2ac_end_effector.urdf.xacro (robot description, xacro)
@@ -77,5 +77,5 @@
       <parent link="${prefix}tool_intermediate_link"/>
       <child link="${prefix}screw_tool_m4_tip_link"/>
-      <origin rpy="0 0 0" xyz=".148 0.0 0.005 "/>
+      <origin rpy="0 0 0" xyz=".148 -0.002 0.003 "/>
     </joint>
     <link name="${prefix}screw_tool_m4_tip_link"/>
