Commit message: Fix tray height

File: catkin_ws/src/o2ac_scene_description/urdf/components/tray.xacro (robot description, xacro)
@@ -29,5 +29,5 @@
   <link name="${trayname}_center">
     <visual>
-      <origin rpy="0 0 0" xyz="0 0 -0.001"/>
+      <origin rpy="0 0 0" xyz="0 0 -0.0001"/>
       <geometry>
         <box size="${tray_w-0.01} ${tray_l-0.01} 0.001"/>
@@ -47,5 +47,5 @@
     <parent link="${trayname}" />
     <child link = "${trayname}_center" />
-    <origin rpy="0 0 0" xyz="${tray_w/2} ${tray_l/2} 0.02"/>
+    <origin rpy="0 0 0" xyz="${tray_w/2} ${tray_l/2} 0.013"/>
   </joint>
   <!-- Frames on top of corners -->

Commit message: Add tray stoppers to base scene
Visuals only

File: catkin_ws/src/o2ac_scene_description/urdf/components/tray.xacro (robot description, xacro)
@@ -49,4 +49,48 @@
     <origin rpy="0 0 0" xyz="${tray_w/2} ${tray_l/2} 0.013"/>
   </joint>
+  <link name="${trayname}_left_stopper">
+    <visual>
+      <origin rpy="0 0 0" xyz="0.0 -0.01 0.01"/>
+      <geometry>
+        <box size="0.06 0.02 0.05"/>
+      </geometry>
+      <material name="white">
+        <color rgba="0 0 0 1"/>
+      </material>
+    </visual>
+    <!-- <collision>
+      <origin rpy="0 0 0" xyz="0.0 -0.01 0.01"/>
+      <geometry>
+        <box size="0.06 0.02 0.05"/>
+      </geometry>
+    </collision> -->
+  </link>
+  <joint name="${trayname}_left_stopper_joint" type="fixed">
+    <parent link="${trayname}" />
+    <child link = "${trayname}_left_stopper" />
+    <origin rpy="0 0 0" xyz="0.08 ${tray_l+0.02} 0.0"/>
+  </joint>
+  <link name="${trayname}_right_stopper">
+    <visual>
+      <origin rpy="0 0 0" xyz="0.0 -0.01 0.01"/>
+      <geometry>
+        <box size="0.06 0.02 0.05"/>
+      </geometry>
+      <material name="white">
+        <color rgba="0 0 0 1"/>
+      </material>
+    </visual>
+    <!-- <collision>
+      <origin rpy="0 0 0" xyz="0.0 -0.01 0.01"/>
+      <geometry>
+        <box size="0.06 0.02 0.05"/>
+      </geometry>
+    </collision> -->
+  </link>
+  <joint name="${trayname}_right_stopper_joint" type="fixed">
+    <parent link="${trayname}" />
+    <child link = "${trayname}_right_stopper" />
+    <origin rpy="0 0 0" xyz="0.08 0.0 0.0"/>
+  </joint>
   <!-- Frames on top of corners -->
   <joint name="${trayname}corner_1_joint" type="fixed">

Commit message: Add AGV tray to scene

File: catkin_ws/src/o2ac_scene_description/urdf/components/tray.xacro (robot description, xacro)
@@ -1,24 +1,28 @@
 <?xml version="1.0"?>
 <robot xmlns:xacro="http://www.ros.org/wiki/xacro" name="task_board">
-  <xacro:macro name="tray" params="trayname parent *origin">
+  <xacro:macro name="tray" params="trayname parent with_visual:=true with_collision_geometry:=true with_stoppers:=true *origin">
   <xacro:property name="mesh_file" value="package://o2ac_scene_description/meshes/tray.stl" />
   <xacro:property name="tray_l" value=".4" />
   <xacro:property name="tray_w" value=".28" />
   <link name="${trayname}">
-    <visual>
-      <origin rpy="${pi/2} 0 ${pi/2}" xyz="0 0 0.0"/>
-      <geometry>
-        <mesh filename="${mesh_file}" scale=".001 .001 .001"/>
-      </geometry>
-      <material name="blue">
-        <color rgba=".2 .2 1 1"/>
-      </material>
-    </visual>
-    <collision>
-      <origin rpy="${pi/2} 0 ${pi/2}" xyz="0 0 0.0"/>
-      <geometry>
-        <mesh filename="${mesh_file}" scale=".001 .001 .001"/>
-      </geometry>
-    </collision>
+    <xacro:if value="${with_visual}">
+      <visual>
+        <origin rpy="${pi/2} 0 ${pi/2}" xyz="0 0 0.0"/>
+        <geometry>
+          <mesh filename="${mesh_file}" scale=".001 .001 .001"/>
+        </geometry>
+        <material name="blue">
+          <color rgba=".2 .2 1 1"/>
+        </material>
+      </visual>
+    </xacro:if>
+    <xacro:if value="${with_collision_geometry}">
+      <collision>
+        <origin rpy="${pi/2} 0 ${pi/2}" xyz="0 0 0.0"/>
+        <geometry>
+          <mesh filename="${mesh_file}" scale=".001 .001 .001"/>
+        </geometry>
+      </collision>
+    </xacro:if>
   </link>
   <joint name="${trayname}_joint" type="fixed" >
@@ -28,19 +32,23 @@
   </joint>
   <link name="${trayname}_center">
-    <visual>
-      <origin rpy="0 0 0" xyz="0 0 -0.0001"/>
-      <geometry>
-        <box size="${tray_w-0.01} ${tray_l-0.01} 0.001"/>
-      </geometry>
-      <material name="black">
-        <color rgba="1 1 1 1"/>
-      </material>
-    </visual>
-    <collision>
-      <origin rpy="0 0 0" xyz="0 0 -0.001"/>
-      <geometry>
-        <box size="${tray_w-0.01} ${tray_l-0.01} 0.001"/>
-      </geometry>
-    </collision>
+    <xacro:if value="${with_visual}">
+      <visual>
+        <origin rpy="0 0 0" xyz="0 0 -0.0001"/>
+        <geometry>
+          <box size="${tray_w-0.01} ${tray_l-0.01} 0.001"/>
+        </geometry>
+        <material name="black">
+          <color rgba="1 1 1 1"/>
+        </material>
+      </visual>
+    </xacro:if>
+    <xacro:if value="${with_collision_geometry}">
+      <collision>
+        <origin rpy="0 0 0" xyz="0 0 -0.001"/>
+        <geometry>
+          <box size="${tray_w-0.01} ${tray_l-0.01} 0.001"/>
+        </geometry>
+      </collision>
+    </xacro:if>
   </link>
   <joint name="${trayname}_center_joint" type="fixed">
@@ -49,48 +57,50 @@
     <origin rpy="0 0 0" xyz="${tray_w/2} ${tray_l/2} 0.013"/>
   </joint>
-  <link name="${trayname}_left_stopper">
-    <visual>
-      <origin rpy="0 0 0" xyz="0.0 -0.01 0.01"/>
-      <geometry>
-        <box size="0.06 0.02 0.05"/>
-      </geometry>
-      <material name="white">
-        <color rgba="0 0 0 1"/>
-      </material>
-    </visual>
-    <!-- <collision>
-      <origin rpy="0 0 0" xyz="0.0 -0.01 0.01"/>
-      <geometry>
-        <box size="0.06 0.02 0.05"/>
-      </geometry>
-    </collision> -->
-  </link>
-  <joint name="${trayname}_left_stopper_joint" type="fixed">
-    <parent link="${trayname}" />
-    <child link = "${trayname}_left_stopper" />
-    <origin rpy="0 0 0" xyz="0.08 ${tray_l+0.02} 0.0"/>
-  </joint>
-  <link name="${trayname}_right_stopper">
-    <visual>
-      <origin rpy="0 0 0" xyz="0.0 -0.01 0.01"/>
-      <geometry>
-        <box size="0.06 0.02 0.05"/>
-      </geometry>
-      <material name="white">
-        <color rgba="0 0 0 1"/>
-      </material>
-    </visual>
-    <!-- <collision>
-      <origin rpy="0 0 0" xyz="0.0 -0.01 0.01"/>
-      <geometry>
-        <box size="0.06 0.02 0.05"/>
-      </geometry>
-    </collision> -->
-  </link>
-  <joint name="${trayname}_right_stopper_joint" type="fixed">
-    <parent link="${trayname}" />
-    <child link = "${trayname}_right_stopper" />
-    <origin rpy="0 0 0" xyz="0.08 0.0 0.0"/>
-  </joint>
+  <xacro:if value="${with_stoppers}">
+    <link name="${trayname}_left_stopper">
+      <visual>
+        <origin rpy="0 0 0" xyz="0.0 -0.01 0.01"/>
+        <geometry>
+          <box size="0.06 0.02 0.05"/>
+        </geometry>
+        <material name="white">
+          <color rgba="0 0 0 1"/>
+        </material>
+      </visual>
+      <!-- <collision>
+        <origin rpy="0 0 0" xyz="0.0 -0.01 0.01"/>
+        <geometry>
+          <box size="0.06 0.02 0.05"/>
+        </geometry>
+      </collision> -->
+    </link>
+    <joint name="${trayname}_left_stopper_joint" type="fixed">
+      <parent link="${trayname}" />
+      <child link = "${trayname}_left_stopper" />
+      <origin rpy="0 0 0" xyz="0.08 ${tray_l+0.02} 0.0"/>
+    </joint>
+    <link name="${trayname}_right_stopper">
+      <visual>
+        <origin rpy="0 0 0" xyz="0.0 -0.01 0.01"/>
+        <geometry>
+          <box size="0.06 0.02 0.05"/>
+        </geometry>
+        <material name="white">
+          <color rgba="0 0 0 1"/>
+        </material>
+      </visual>
+      <!-- <collision>
+        <origin rpy="0 0 0" xyz="0.0 -0.01 0.01"/>
+        <geometry>
+          <box size="0.06 0.02 0.05"/>
+        </geometry>
+      </collision> -->
+    </link>
+    <joint name="${trayname}_right_stopper_joint" type="fixed">
+      <parent link="${trayname}" />
+      <child link = "${trayname}_right_stopper" />
+      <origin rpy="0 0 0" xyz="0.08 0.0 0.0"/>
+    </joint>
+  </xacro:if>
   <!-- Frames on top of corners -->
   <joint name="${trayname}corner_1_joint" type="fixed">

File: catkin_ws/src/o2ac_scene_description/urdf/o2ac_environment.xacro (robot description, xacro)
@@ -36,4 +36,8 @@
   <xacro:tray trayname="tray" parent="workspace_center">
     <origin xyz="0.05 -0.2 0.001" rpy="0 0 0" />
+  </xacro:tray>
+  <xacro:include filename="$(find o2ac_scene_description)/urdf/components/tray.xacro" />
+  <xacro:tray trayname="agv_tray" parent="workspace_center" with_visual="false" with_collision_geometry="false" with_stoppers="false">
+    <origin xyz="0.37 -0.2 0.001" rpy="0 0 0" />
   </xacro:tray>
   <!-- Add the jigs -->

Commit message: Adjust tray geometry

File: catkin_ws/src/o2ac_scene_description/urdf/components/tray.xacro (robot description, xacro)
@@ -34,5 +34,5 @@
     <xacro:if value="${with_visual}">
       <visual>
-        <origin rpy="0 0 0" xyz="0 0 -0.0001"/>
+        <origin rpy="0 0 0" xyz="0 0 -0.001"/>
         <geometry>
           <box size="${tray_w-0.01} ${tray_l-0.01} 0.001"/>
@@ -45,5 +45,5 @@
     <xacro:if value="${with_collision_geometry}">
       <collision>
-        <origin rpy="0 0 0" xyz="0 0 -0.001"/>
+        <origin rpy="0 0 0" xyz="0 0 -0.002"/>
         <geometry>
           <box size="${tray_w-0.01} ${tray_l-0.01} 0.001"/>

File: catkin_ws/src/o2ac_scene_description/urdf/o2ac_environment.xacro (robot description, xacro)
@@ -35,5 +35,5 @@
   <xacro:include filename="$(find o2ac_scene_description)/urdf/components/tray.xacro" />
   <xacro:tray trayname="tray" parent="workspace_center">
-    <origin xyz="0.05 -0.2 0.001" rpy="0 0 0" />
+    <origin xyz="0.05 -0.2 0.0001" rpy="0 0 0" />
   </xacro:tray>
   <xacro:include filename="$(find o2ac_scene_description)/urdf/components/tray.xacro" />

Commit message: WIP: update L-plates assembly

File: catkin_ws/src/o2ac_scene_description/urdf/components/tray.xacro (robot description, xacro)
@@ -80,4 +80,26 @@
       <origin rpy="0 0 0" xyz="0.08 ${tray_l+0.02} 0.0"/>
     </joint>
+    <link name="${trayname}_left_stopper2">
+      <visual>
+        <origin rpy="0 0 0" xyz="0.0 -0.01 0.01"/>
+        <geometry>
+          <box size="0.06 0.02 0.05"/>
+        </geometry>
+        <material name="white">
+          <color rgba="0 0 0 1"/>
+        </material>
+      </visual>
+      <!-- <collision>
+        <origin rpy="0 0 0" xyz="0.0 -0.01 0.01"/>
+        <geometry>
+          <box size="0.06 0.02 0.05"/>
+        </geometry>
+      </collision> -->
+    </link>
+    <joint name="${trayname}_left_stopper2_joint" type="fixed">
+      <parent link="${trayname}" />
+      <child link = "${trayname}_left_stopper2" />
+      <origin rpy="0 0 0" xyz="0.21 ${tray_l+0.02} 0.0"/>
+    </joint>
     <link name="${trayname}_right_stopper">
       <visual>
@@ -101,4 +123,26 @@
       <child link = "${trayname}_right_stopper" />
       <origin rpy="0 0 0" xyz="0.08 0.0 0.0"/>
+    </joint>
+    <link name="${trayname}_right_stopper2">
+      <visual>
+        <origin rpy="0 0 0" xyz="0.0 -0.01 0.01"/>
+        <geometry>
+          <box size="0.06 0.02 0.05"/>
+        </geometry>
+        <material name="white">
+          <color rgba="0 0 0 1"/>
+        </material>
+      </visual>
+      <!-- <collision>
+        <origin rpy="0 0 0" xyz="0.0 -0.01 0.01"/>
+        <geometry>
+          <box size="0.06 0.02 0.05"/>
+        </geometry>
+      </collision> -->
+    </link>
+    <joint name="${trayname}_right_stopper2_joint" type="fixed">
+      <parent link="${trayname}" />
+      <child link = "${trayname}_right_stopper2" />
+      <origin rpy="0 0 0" xyz="0.21 0.0 0.0"/>
     </joint>
   </xacro:if>

Commit message: Lots of calibrations for assembly

File: catkin_ws/src/o2ac_scene_description/urdf/components/tray.xacro (robot description, xacro)
@@ -55,5 +55,5 @@
     <parent link="${trayname}" />
     <child link = "${trayname}_center" />
-    <origin rpy="0 0 0" xyz="${tray_w/2} ${tray_l/2} 0.013"/>
+    <origin rpy="0 0 0" xyz="${tray_w/2} ${tray_l/2} 0.010"/>
   </joint>
   <xacro:if value="${with_stoppers}">
