Commit message: WIP: Remove screw tools from fixed scene, simplify Subtask B MTC plan

File: catkin_ws/src/o2ac_scene_description/urdf/components/tools.xacro (robot description, xacro)
@@ -28,10 +28,10 @@
       </material>
     </visual>
-    <collision>
+    <!-- <collision>
       <origin rpy="0 0 0" xyz="-0.15 .0033 0.002"/>
       <geometry>
         <box size=".3 .066 .004"/>
       </geometry>
-    </collision>
+    </collision> -->
     <!-- The vertical plate -->
     <visual>
@@ -44,10 +44,10 @@
       </material>
     </visual>
-    <collision>
+    <!-- <collision>
       <origin rpy="0 0 0" xyz="-0.15 -.011 0.0179"/>
       <geometry>
         <box size=".3 .004 .035"/>
       </geometry>
-    </collision>
+    </collision> -->
   </link>
   <!-- ==== -->
@@ -110,5 +110,5 @@
       <inertia ixx="1" ixy="0" ixz="0" iyy="1" iyz="0" izz="1"/>
     </inertial>
-    <visual>
+    <!-- <visual>
       <origin rpy="0 0 0" xyz="0 0 ${.052/2}"/>
       <geometry>
@@ -118,11 +118,11 @@
         <color rgba=".9 .9 .7 1"/>
       </material>
-    </visual>
-    <collision>
+    </visual> -->
+    <!-- <collision>
       <origin rpy="0 0 0" xyz="0 0 ${.052/2}"/>
       <geometry>
         <box size=".026 .059 .052"/>
       </geometry>
-    </collision>
+    </collision> -->
   </link>
   <joint name="nut_tool_m6_to_holder" type="fixed">
@@ -138,5 +138,5 @@
       <inertia ixx="1" ixy="0" ixz="0" iyy="1" iyz="0" izz="1"/>
     </inertial>
-    <visual>
+    <!-- <visual>
       <origin rpy="0 0 0" xyz="0 0 ${.052/2}"/>
       <geometry>
@@ -146,11 +146,11 @@
         <color rgba=".9 .9 .7 1"/>
       </material>
-    </visual>
-    <collision>
+    </visual> -->
+    <!-- <collision>
       <origin rpy="0 0 0" xyz="0 0 ${.052/2}"/>
       <geometry>
         <box size=".026 .059 .052"/>
       </geometry>
-    </collision>
+    </collision> -->
   </link>
   <joint name="set_screw_tool_to_holder" type="fixed">
@@ -165,5 +165,5 @@
       <inertia ixx="1" ixy="0" ixz="0" iyy="1" iyz="0" izz="1"/>
     </inertial>
-    <visual>
+    <!-- <visual>
       <origin rpy="0 0 0" xyz="0 0 0"/>
       <geometry>
@@ -174,10 +174,4 @@
       </material>
     </visual>
-    <!-- <collision>
-      <origin rpy="0 0 0" xyz="0 ${-bit_cushion_to_axis + .02} .0275"/>
-      <geometry>
-        <box size=".026 .04 .055"/>
-      </geometry>
-    </collision> -->
     <collision>
       <origin rpy="0 0 0" xyz="0 0 ${-.12/2}"/>
@@ -191,5 +185,5 @@
         <cylinder length=".12" radius=".01"/>
       </geometry>
-    </collision>
+    </collision> -->
   </link>
   <joint name="screw_tool_m4_to_holder" type="fixed">
@@ -204,5 +198,5 @@
       <inertia ixx="1" ixy="0" ixz="0" iyy="1" iyz="0" izz="1"/>
     </inertial>
-    <visual>
+    <!-- <visual>
       <origin rpy="0 0 0" xyz="0 0 0"/>
       <geometry>
@@ -213,10 +207,4 @@
       </material>
     </visual>
-    <!-- <collision>
-      <origin rpy="0 0 0" xyz="0 ${-bit_cushion_to_axis + .02} .0275"/>
-      <geometry>
-        <box size=".026 .04 .055"/>
-      </geometry>
-    </collision> -->
     <collision>
       <origin rpy="0 0 0" xyz="0 0 ${-.1/2}"/>
@@ -230,5 +218,5 @@
         <cylinder length=".1" radius=".01"/>
       </geometry>
-    </collision>
+    </collision> -->
   </link>
   <joint name="screw_tool_m3_to_holder" type="fixed">

Commit message: Add padless m4 tool, move m3 tool

File: catkin_ws/src/o2ac_scene_description/urdf/components/tools.xacro (robot description, xacro)
@@ -104,32 +104,4 @@
   <xacro:property name="tool_offset" value="${-.005 + bit_cushion_to_axis}" />
   <!-- The collision boxes of the tools only include the top part (not what is hanging underneath the holder) -->
-  <link name="nut_tool_m6_link">
-    <inertial>
-      <origin rpy="0 0 0" xyz="0 0 0"/>
-      <mass value="1.0"/>
-      <inertia ixx="1" ixy="0" ixz="0" iyy="1" iyz="0" izz="1"/>
-    </inertial>
-    <!-- <visual>
-      <origin rpy="0 0 0" xyz="0 0 ${.052/2}"/>
-      <geometry>
-        <box size=".026 .059 .052"/>
-      </geometry>
-      <material name="yellowish">
-        <color rgba=".9 .9 .7 1"/>
-      </material>
-    </visual> -->
-    <!-- <collision>
-      <origin rpy="0 0 0" xyz="0 0 ${.052/2}"/>
-      <geometry>
-        <box size=".026 .059 .052"/>
-      </geometry>
-    </collision> -->
-  </link>
-  <joint name="nut_tool_m6_to_holder" type="fixed">
-    <parent link="screw_tool_holder_long" />
-    <child link="nut_tool_m6_link" />
-    <origin xyz="-0.05 ${-back_plate_offset_long + .059/2 + .0155} 0.004" rpy="0.0 0.0 0.0" />
-    <!-- .0155 is the distance from the center of the box to the axis of the tool -->
-  </joint>
   <link name="set_screw_tool_link">
     <inertial>
@@ -223,4 +195,16 @@
     <parent link="screw_tool_holder_long" />
     <child link="screw_tool_m3_link" />
+    <origin xyz="-0.05 ${tool_offset} 0.004" rpy="0.0 0.0 0.0" />
+  </joint>
+  <link name="padless_tool_m4_link">
+    <inertial>
+      <origin rpy="0 0 0" xyz="0 0 0"/>
+      <mass value="1.0"/>
+      <inertia ixx="1" ixy="0" ixz="0" iyy="1" iyz="0" izz="1"/>
+    </inertial>
+  </link>
+  <joint name="padless_tool_m4_to_holder" type="fixed">
+    <parent link="screw_tool_holder_long" />
+    <child link="padless_tool_m4_link" />
     <origin xyz="-0.15 ${tool_offset} 0.004" rpy="0.0 0.0 0.0" />
   </joint>
@@ -238,8 +222,8 @@
     <origin xyz="0.0 0.0 0.0" rpy="0.0 ${pi} ${pi/2}" />
   </joint>
-  <link name="nut_tool_m6_pickup_link"/>
-  <joint name="nut_tool_m6_pickup_joint" type="fixed">
-    <parent link="nut_tool_m6_link" />
-    <child link="nut_tool_m6_pickup_link" />
+  <link name="padless_tool_m4_pickup_link"/>
+  <joint name="padless_tool_m4_pickup_joint" type="fixed">
+    <parent link="padless_tool_m4_link" />
+    <child link="padless_tool_m4_pickup_link" />
     <origin xyz="0.0 0.0 0.0" rpy="0.0 ${pi} ${pi/2}" />
   </joint>

Commit message: WIP: motor cables insertion

File: catkin_ws/src/o2ac_scene_description/urdf/components/tools.xacro (robot description, xacro)
@@ -390,5 +390,5 @@
     <parent link="workspace_center" />
     <child link="cable_holder_link" />
-    <origin xyz="-0.49 -0.225 0.2" rpy="0 0 0" />
+    <origin xyz="-0.503 -0.225 0.19" rpy="0 0 0" />
   </joint>
   <link name="cable_holder_pickup_link"/>
@@ -396,5 +396,5 @@
     <parent link="cable_holder_link" />
     <child link="cable_holder_pickup_link" />
-    <origin xyz="0.1 0.0 0.015" rpy="0 ${pi/2} 0" />
+    <origin xyz="0.1 0.004 0.015" rpy="0 ${pi/2} 0" />
   </joint>
   <link name="nut_holder2_link"/>

File: catkin_ws/src/o2ac_scene_description/urdf/o2ac_environment.xacro (robot description, xacro)
@@ -101,5 +101,5 @@
     <origin xyz="0 -0.05 0.001" rpy="0 0 0" />
   </xacro:washer_holder>
-  <xacro:include filename="$(find o2ac_scene_description)/urdf/components/washer_holder.xacro" />
+  <!-- <xacro:include filename="$(find o2ac_scene_description)/urdf/components/washer_holder.xacro" />
   <xacro:washer_holder partname="washer_holder3" parent="workspace_center">
     <origin xyz="0.325 -0.6 -0.045" rpy="0 ${pi/2} 0" />
@@ -108,5 +108,5 @@
   <xacro:washer_holder partname="washer_holder4" parent="workspace_center">
     <origin xyz="0.325 -0.5 -0.045" rpy="0 ${pi/2} 0" />
-  </xacro:washer_holder>
+  </xacro:washer_holder>  -->
   <!-- ======== -->
   <!-- <xacro:include filename="$(find o2ac_scene_description)/urdf/components/nut_holder.xacro" />
