Commit message: Change a_bot gripper to robotiq_140

File: catkin_ws/src/o2ac_scene_description/urdf/components/o2ac_end_effector_2F-140.urdf.xacro (robot description, xacro)
@@ -4,15 +4,15 @@
 <robot name="robotiq_85_gripper_o2ac" xmlns:xacro="http://www.ros.org/wiki/xacro">
   <xacro:macro name="o2ac_end_effector" params="prefix use_soft_wrist:=false use_cameras:=false parent">
-    <xacro:include filename="$(find robotiq_description)/urdf/robotiq_85_gripper.urdf.xacro"/>
-    <xacro:robotiq_85_gripper prefix="${prefix}" parent="${parent}">
+    <xacro:include filename="$(find robotiq_description)/urdf/robotiq_140_gripper.urdf.xacro"/>
+    <xacro:robotiq_140_gripper prefix="${prefix}" parent="${parent}">
         <origin rpy="0.0 0.0 0.0" xyz="0 0 0"/>
-    </xacro:robotiq_85_gripper>
+    </xacro:robotiq_140_gripper>
     <xacro:if value="${use_cameras}">
       <xacro:include filename="$(find o2ac_scene_description)/urdf/components/wrist_cameras.xacro" />
-      <xacro:wrist_cameras prefix="${prefix}" parent="${prefix}robotiq_85_base_link"/>
+      <xacro:wrist_cameras prefix="${prefix}" parent="${prefix}robotiq_140_base_link"/>
     </xacro:if>
     <!-- Add an additional link to plan with. Oriented like the UR ee_link frame. -->
     <joint name="${prefix}robotiq_85_tip_link_joint" type="fixed">
-      <parent link="${prefix}robotiq_85_base_link"/>
+      <parent link="${prefix}robotiq_140_base_link"/>
       <child link="${prefix}robotiq_85_tip_link"/>
       <origin rpy="0.0 0.0 0.0" xyz="${.163+.083} 0.0 0.0"/>

Commit message: Fix tool frames in robotiq 140 gripper

File: catkin_ws/src/o2ac_scene_description/urdf/components/o2ac_end_effector_2F-140.urdf.xacro (robot description, xacro)
@@ -25,17 +25,11 @@
       <parent link="${prefix}robotiq_85_tip_link"/>
       <child link="${prefix}tool_intermediate_link"/>
-      <origin rpy="${pi} 0.0 0.0" xyz="-.03 0.0 0.0"/>
+      <origin rpy="${pi} ${-pi/3} 0" xyz="-.03 0 0"/>
     </joint>
     <link name="${prefix}tool_intermediate_link"/>
-    <joint name="${prefix}robotiq_85_screw_tool_m6_tip_joint" type="fixed">
-      <parent link="${prefix}tool_intermediate_link"/>
-      <child link="${prefix}screw_tool_m6_tip_link"/>
-      <origin rpy="0.0 ${pi/2} 0.0" xyz="0.0 0.0 -0.135 "/>
-    </joint>
-    <link name="${prefix}screw_tool_m6_tip_link"/>
     <joint name="${prefix}robotiq_85_nut_tool_m6_tip_joint" type="fixed">
       <parent link="${prefix}tool_intermediate_link"/>
       <child link="${prefix}nut_tool_m6_tip_link"/>
-      <origin rpy="0.0 ${pi/4} 0.0" xyz="0.0 0.0 -0.12 "/>
+      <origin rpy="0 0 0" xyz="0.12 0 0 "/>
     </joint>
     <link name="${prefix}nut_tool_m6_tip_link"/>
@@ -43,5 +37,5 @@
       <parent link="${prefix}tool_intermediate_link"/>
       <child link="${prefix}screw_tool_m4_tip_link"/>
-      <origin rpy="0.0 ${pi/2} 0.0" xyz="-.002 0.0 -0.146 "/>
+      <origin rpy="0 0 0" xyz=".141 0 0.005 "/>
     </joint>
     <link name="${prefix}screw_tool_m4_tip_link"/>
@@ -49,5 +43,5 @@
       <parent link="${prefix}tool_intermediate_link"/>
       <child link="${prefix}screw_tool_m3_tip_link"/>
-      <origin rpy="0.0 ${pi/2} 0.0" xyz=".015 0.0 -0.14 "/>
+      <origin rpy="0 0 0" xyz=".14 0 .015 "/>
     </joint>
     <link name="${prefix}screw_tool_m3_tip_link"/>
@@ -55,19 +49,7 @@
       <parent link="${prefix}tool_intermediate_link"/>
       <child link="${prefix}set_screw_tool_tip_link"/>
-      <origin rpy="0.0 ${pi/2} 0.0" xyz=".01 0.0 -0.085 "/>
+      <origin rpy="0 0 0" xyz="0.0725 0 0.009"/>
     </joint>
     <link name="${prefix}set_screw_tool_tip_link"/>
-    <joint name="${prefix}robotiq_85_suction_tool_tip_joint" type="fixed">
-      <parent link="${prefix}tool_intermediate_link"/>
-      <child link="${prefix}suction_tool_tip_link"/>
-      <origin rpy="0.0 ${pi/2} 0.0" xyz=".02 0.0 -0.131 "/>
-    </joint>
-    <link name="${prefix}suction_tool_tip_link"/>
-    <joint name="${prefix}dual_suction_gripper_pad_joint" type="fixed">
-      <parent link="${prefix}tool_intermediate_link"/>
-      <child link="${prefix}dual_suction_gripper_pad_link"/>
-      <origin rpy="0.0 0 0.0" xyz="0 0 0 "/>
-    </joint>
-    <link name="${prefix}dual_suction_gripper_pad_link"/>
   </xacro:macro>
 </robot>

Commit message: Add nut tool tip link to a_bot

File: catkin_ws/src/o2ac_scene_description/urdf/components/o2ac_end_effector_2F-140.urdf.xacro (robot description, xacro)
@@ -52,4 +52,12 @@
     </joint>
     <link name="${prefix}set_screw_tool_tip_link"/>
+    <!-- ========= -->
+    <!-- Nut tool frame. X-axis points into the nut. -->
+    <joint name="${prefix}_nut_tool_m4_joint" type="fixed">
+      <parent link="${prefix}gripper_tip_link"/>
+      <child link="${prefix}nut_tool_m4_hole_link"/>
+      <origin rpy="0.923 1.571 0.923" xyz="${-.018+.020} 0.0 .017"/>
+    </joint>
+    <link name="${prefix}nut_tool_m4_hole_link"/>
   </xacro:macro>
 </robot>

Commit message: Fix position of a_bot cameras, fix tray view poses

File: catkin_ws/src/o2ac_scene_description/urdf/components/o2ac_end_effector_2F-140.urdf.xacro (robot description, xacro)
@@ -1,11 +1,31 @@
 <?xml version="1.0"?>
-<!-- This file is a safety measure because a_bot is temporarily using a 2F-140 gripper
-     instead of a 2F-85 gripper. The tip link is set to the . -->
-<robot name="robotiq_85_gripper_o2ac" xmlns:xacro="http://www.ros.org/wiki/xacro">
+<robot name="robotiq_140_gripper_o2ac" xmlns:xacro="http://www.ros.org/wiki/xacro">
   <xacro:macro name="o2ac_end_effector" params="prefix use_soft_wrist:=false use_cameras:=false parent">
     <xacro:include filename="$(find robotiq_description)/urdf/robotiq_140_gripper.urdf.xacro"/>
     <xacro:robotiq_140_gripper prefix="${prefix}" parent="${parent}">
-        <origin rpy="0.0 0.0 0.0" xyz="0 0 0"/>
+        <origin rpy="0.0 0.0 0.0" xyz="0.01 0 0"/> <!-- This 0.01 offset is the Robotiq/UR coupling -->
     </xacro:robotiq_140_gripper>
+    <link name="${prefix}coupling">
+      <visual>
+        <origin rpy="0 ${pi/2} 0" xyz=".005 0 0"/>
+        <geometry>
+          <cylinder length="0.01" radius="0.0375"/>
+        </geometry>
+        <material name="black">
+        <color rgba=".1 .1 .1 1"/>
+      </material>
+      </visual>
+      <collision>
+        <origin rpy="0 ${pi/2} 0" xyz=".005 0 0"/>
+        <geometry>
+          <cylinder length="0.01" radius="0.0375"/>
+        </geometry>
+      </collision>
+    </link>
+    <joint name="${prefix}coupling_joint" type="fixed">
+      <parent link="${parent}" />
+      <child link = "${prefix}coupling" />
+      <origin rpy="0 0 0" xyz="0 0 0"/>
+    </joint>
     <xacro:if value="${use_cameras}">
       <xacro:include filename="$(find o2ac_scene_description)/urdf/components/wrist_cameras.xacro" />
@@ -16,5 +36,5 @@
       <parent link="${prefix}robotiq_140_base_link"/>
       <child link="${prefix}gripper_tip_link"/>
-      <origin rpy="0.0 0.0 0.0" xyz="${.163+.083} 0.0 0.0"/>
+      <origin rpy="0.0 0.0 0.0" xyz="${.163+.073} 0.0 0.0"/>
     </joint>
     <link name="${prefix}gripper_tip_link"/>

Commit message: Change a_bot tool grasp to increase stability
Moves the gripper deeper into the tool. This seems to increase the grasp strength/stability

File: catkin_ws/src/o2ac_scene_description/urdf/components/o2ac_end_effector_2F-140.urdf.xacro (robot description, xacro)
@@ -51,5 +51,5 @@
       <parent link="${prefix}tool_intermediate_link"/>
       <child link="${prefix}nut_tool_m6_tip_link"/>
-      <origin rpy="0 0 0" xyz="0.107 0 -0.0075 "/>
+      <origin rpy="0 0 0" xyz="0.107 0 -0.0175 "/>
     </joint>
     <link name="${prefix}nut_tool_m6_tip_link"/>
@@ -57,5 +57,5 @@
       <parent link="${prefix}tool_intermediate_link"/>
       <child link="${prefix}screw_tool_m4_tip_link"/>
-      <origin rpy="0 0 0" xyz=".141 0 0.005 "/>
+      <origin rpy="0 0 0" xyz=".141 0 -0.005 "/>
     </joint>
     <link name="${prefix}screw_tool_m4_tip_link"/>
@@ -63,5 +63,5 @@
       <parent link="${prefix}tool_intermediate_link"/>
       <child link="${prefix}screw_tool_m3_tip_link"/>
-      <origin rpy="0 0 0" xyz=".121 0 .0055 "/>
+      <origin rpy="0 0 0" xyz=".121 0 -.0045 "/>
     </joint>
     <link name="${prefix}screw_tool_m3_tip_link"/>
@@ -69,5 +69,5 @@
       <parent link="${prefix}tool_intermediate_link"/>
       <child link="${prefix}set_screw_tool_tip_link"/>
-      <origin rpy="0 0 0" xyz="0.058 0 0.006"/>
+      <origin rpy="0 0 0" xyz="0.058 0 -0.004"/>
     </joint>
     <link name="${prefix}set_screw_tool_tip_link"/>

Commit message: Add horizontal tooltip offset to a_bot (?!)
Today the tool was crazy. This might have to be changed back.

File: catkin_ws/src/o2ac_scene_description/urdf/components/o2ac_end_effector_2F-140.urdf.xacro (robot description, xacro)
@@ -57,5 +57,5 @@
       <parent link="${prefix}tool_intermediate_link"/>
       <child link="${prefix}screw_tool_m4_tip_link"/>
-      <origin rpy="0 0 0" xyz=".146 0 -0.005 "/>
+      <origin rpy="0 0 0" xyz=".146 -.001 -0.005 "/>
     </joint>
     <link name="${prefix}screw_tool_m4_tip_link"/>
@@ -63,5 +63,5 @@
       <parent link="${prefix}tool_intermediate_link"/>
       <child link="${prefix}screw_tool_m3_tip_link"/>
-      <origin rpy="0 0 0" xyz=".128 0 -.0045 "/>
+      <origin rpy="0 0 0" xyz=".128 -.001 -.0045 "/>
     </joint>
     <link name="${prefix}screw_tool_m3_tip_link"/>

Commit message: Add flexbe states for cooking

File: catkin_ws/src/o2ac_scene_description/urdf/components/o2ac_end_effector_2F-140.urdf.xacro (robot description, xacro)
@@ -39,34 +39,32 @@
     </joint>
     <link name="${prefix}gripper_tip_link"/>
-    <link name="${prefix}cable_tool_tip_link"/>
+    <joint name="${prefix}tool_intermediate_joint" type="fixed">
+      <parent link="${prefix}gripper_tip_link"/>
+      <child link="${prefix}tool_intermediate_link"/>
+      <origin rpy="0 ${-pi/3} 0" xyz="0 0 0"/>
+    </joint>
+    <link name="${prefix}tool_intermediate_link"/>
+    <link name="${prefix}knife_tool_tip_link"/>
+    <joint name="${prefix}knife_tool_tip_link_joint" type="fixed">
+      <parent link="${prefix}tool_intermediate_link"/>
+      <child link="${prefix}knife_tool_tip_link"/>
+      <origin rpy="0.0 0.0 0.0" xyz="${.15} 0.0 0.0"/>
+    </joint>
+    <!-- <link name="${prefix}cable_tool_tip_link"/>
     <joint name="${prefix}cable_tool_tip_link_joint" type="fixed">
       <parent link="${prefix}gripper_tip_link"/>
       <child link="${prefix}cable_tool_tip_link"/>
       <origin rpy="0.0 0.0 0.0" xyz="${.03} 0.0 0.0"/>
-    </joint>
+    </joint> -->
     <!-- ========= -->
     <!-- Add screw tool tip frames. X-axis points along the screw into the hole. -->
     <!-- Offset of the gripper tooltips -->
-    <joint name="${prefix}tool_intermediate_joint" type="fixed">
+    <!-- <joint name="${prefix}tool_intermediate_joint" type="fixed">
       <parent link="${prefix}gripper_tip_link"/>
       <child link="${prefix}tool_intermediate_link"/>
       <origin rpy="${pi} ${-pi/3} 0" xyz="-.03 0 0"/>
     </joint>
-    <link name="${prefix}tool_intermediate_link"/>
-    <joint name="${prefix}robotiq_85_nut_tool_m6_tip_joint" type="fixed">
-      <parent link="${prefix}tool_intermediate_link"/>
-      <child link="${prefix}nut_tool_m6_tip_link"/>
-      <origin rpy="0 0 0" xyz="0.107 0 -0.0175 "/>
-    </joint>
-    <link name="${prefix}nut_tool_m6_tip_link"/>
-    <joint name="${prefix}robotiq_85_screw_tool_m4_tip_joint" type="fixed">
-      <parent link="${prefix}tool_intermediate_link"/>
-      <child link="${prefix}screw_tool_m4_tip_link"/>
-      <!-- y: points towards back -->
-      <!-- z: points towards left -->
-      <origin rpy="0 0 0" xyz=".145 -.001 0.0 "/>
-    </joint>
-    <link name="${prefix}screw_tool_m4_tip_link"/>
-    <joint name="${prefix}robotiq_85_screw_tool_m3_tip_joint" type="fixed">
+    <link name="${prefix}tool_intermediate_link"/> -->
+    <!-- <joint name="${prefix}robotiq_85_screw_tool_m3_tip_joint" type="fixed">
       <parent link="${prefix}tool_intermediate_link"/>
       <child link="${prefix}screw_tool_m3_tip_link"/>
@@ -79,5 +77,5 @@
       <origin rpy="0 0 0" xyz="0.058 0 -0.004"/>
     </joint>
-    <link name="${prefix}set_screw_tool_tip_link"/>
+    <link name="${prefix}set_screw_tool_tip_link"/> -->
     <!-- ========= -->
     <!-- Nut tool frame. X-axis points into the nut. -->
