Commit message: Add support for calibration in o2ac environment

File: catkin_ws/src/o2ac_scene_description/urdf/calibration_scene.xacro (robot description, xacro)
@@ -3,10 +3,10 @@
   <!-- Add AR markers -->
   <xacro:include filename="$(find o2ac_gazebo)/urdf/ar_markers.urdf.xacro"/>
-  <xacro:ar_marker_70_5 prefix="b_bot_"
-  			parent="b_bot_robotiq_85_tip_link"
-  			marker_id="26"
-  			thickness="0.005">
-    <origin xyz="0.0 0.0 0.0185" rpy="0 0 0"/>
-  </xacro:ar_marker_70_5>
+  <!-- <xacro:ar_marker_70_5 prefix="b_bot_" -->
+  <!-- 			parent="b_bot_robotiq_85_tip_link" -->
+  <!-- 			marker_id="26" -->
+  <!-- 			thickness="0.005"> -->
+  <!--   <origin xyz="0.0 0.0 0.0185" rpy="0 0 0"/> -->
+  <!-- </xacro:ar_marker_70_5> -->
   <xacro:ar_marker_80_10 prefix="base_"
 			parent="attached_base_origin_link"
