Commit message: Add base fixture, update belt tool and holder

File: catkin_ws/src/o2ac_scene_description/urdf/assembly_scene.xacro (robot description, xacro)
@@ -4,10 +4,7 @@
   <xacro:include filename="$(find o2ac_parts_description)/urdf/assembly_parts_macros.urdf.xacro"/>
   <!-- <xacro:include filename="$(find o2ac_parts_description)/urdf/display_all_parts.urdf.xacro"/> -->
-  <!-- The holes in the new table are spaced 10 cm apart. (.65/2) is the width of the robot base. 15 mm is the bracket. -->
-  <!-- -.415+.65/2 = -.415+.325 = -.09 -->
-  <xacro:property name="assy_dx" value="-.09" />
   <xacro:include filename="$(find o2ac_parts_description)/urdf/generated/full_assembly.urdf.xacro"/>
-  <xacro:full_assembly prefix="assembled_" parent="workspace_center">
-    <origin xyz="${assy_dx} 0.11 .08" rpy="0 0 ${-pi/2}" />
+  <xacro:full_assembly prefix="assembled_" parent="attached_base_origin_link">
+    <origin xyz=".12 .2 0" rpy="0 0 ${-pi/2}" />
   </xacro:full_assembly>
   <!-- <xacro:include filename="$(find o2ac_parts_description)/urdf/generated/full_assembly_frames_only.urdf.xacro"/>

File: catkin_ws/src/o2ac_scene_description/urdf/base_scene.urdf.xacro (robot description, xacro)
@@ -22,6 +22,6 @@
   <xacro:include filename="$(find o2ac_scene_description)/urdf/o2ac_environment.xacro" />
   <!-- <xacro:include filename="$(find flexwrist_experiment)/urdf/2020-01-experiment-scene.xacro" /> -->
-  <!-- <xacro:include filename="$(find o2ac_scene_description)/urdf/taskboard_scene.xacro" /> -->
-  <xacro:include filename="$(find o2ac_scene_description)/urdf/assembly_scene.xacro" />
+  <xacro:include filename="$(find o2ac_scene_description)/urdf/taskboard_scene.xacro" />
+  <!-- <xacro:include filename="$(find o2ac_scene_description)/urdf/assembly_scene.xacro" /> -->
   <!-- Robot bases -->
   <!-- Putting these at height 0.0 makes them intersect with the ground, so they are elevated. -->

File: catkin_ws/src/o2ac_scene_description/urdf/o2ac_environment.xacro (robot description, xacro)
@@ -18,5 +18,5 @@
   </xacro:o2ac_box>
   <!-- Screw holder & screw tool visual -->
-  <xacro:include filename="$(find o2ac_scene_description)/urdf/components/screw_tools.xacro" />
+  <xacro:include filename="$(find o2ac_scene_description)/urdf/components/tools.xacro" />
   <!-- Add screw feeders -->
   <xacro:include filename="$(find o2ac_scene_description)/urdf/components/screw_feeder.xacro" />
@@ -27,4 +27,14 @@
     <origin xyz="-.55 -.15 -0.043" rpy="0 0 0" />
   </xacro:screw_feeder>
+  <!-- Base fixture -->
+  <xacro:include filename="$(find o2ac_scene_description)/urdf/components/base_fixture.xacro" />
+  <xacro:base_fixture parent="workspace_center">
+    <origin xyz="-0.27 -.18 0" rpy="0 0 0" />
+  </xacro:base_fixture>
+  <!-- Tray -->
+  <xacro:include filename="$(find o2ac_scene_description)/urdf/components/tray.xacro" />
+  <xacro:tray trayname="tray" parent="workspace_center">
+    <origin xyz="0.05 -0.2 0" rpy="0 0 0" />
+  </xacro:tray>
   <!-- Add the jigs -->
   <!-- <xacro:include filename="$(find o2ac_scene_description)/urdf/components/jig_flat_slope.xacro" />
@@ -36,9 +46,4 @@
     <origin xyz="0 0 0" rpy="0 0 0" />
   </xacro:jig_v_slope>  -->
-  <!-- Tray -->
-  <xacro:include filename="$(find o2ac_scene_description)/urdf/components/tray.xacro" />
-  <xacro:tray trayname="tray" parent="workspace_center">
-    <origin xyz="0.05 -0.2 0" rpy="0 0 0" />
-  </xacro:tray>
   <!-- <link name="scene_cam_holder_link" />
   <joint name="scene_cam_holder_joint" type="fixed">

File: catkin_ws/src/o2ac_scene_description/urdf/taskboard_scene.xacro (robot description, xacro)
@@ -2,6 +2,6 @@
 <robot xmlns:xacro="http://www.ros.org/wiki/xacro" name="taskboard_scene">
   <xacro:include filename="$(find o2ac_scene_description)/urdf/components/taskboard.xacro" />
-  <xacro:taskboard boardname="taskboard" parent="workspace_center">
-    <origin xyz="0 -.1 .08" rpy="0 0 0" />
+  <xacro:taskboard boardname="taskboard" parent="attached_base_origin_link">
+    <origin xyz=".12 0 0" rpy="0 0 0" />
   </xacro:taskboard>
 </robot>

Commit message: Fix assembly scene

File: catkin_ws/src/o2ac_scene_description/urdf/assembly_scene.xacro (robot description, xacro)
@@ -7,10 +7,10 @@
   <xacro:full_assembly prefix="assembled_" parent="attached_base_origin_link">
     <origin xyz=".12 .2 0" rpy="0 0 ${-pi/2}" />
-  </xacro:full_assembly>
+  </xacro:full_assembly> -->
   <!-- ====== Uncomment this block to add the frames of the complete assembly, but not the objects -->
-  <!-- <xacro:include filename="$(find o2ac_parts_description)/urdf/generated/full_assembly_frames_only.urdf.xacro"/>
+  <xacro:include filename="$(find o2ac_parts_description)/urdf/generated/full_assembly_frames_only.urdf.xacro"/>
   <xacro:full_assembly_frames_only prefix="assembled_" parent="workspace_center">
-    <origin xyz="${assy_dx} 0.1 .08" rpy="0 0 ${-pi/2}" />
-  </xacro:full_assembly_frames_only> -->
+    <origin xyz=".12 .2 0" rpy="0 0 ${-pi/2}" />
+  </xacro:full_assembly_frames_only>
   <!-- The base plate -->
   <!-- <xacro:assy_part_01 prefix="dummy" parent="assembled_assy_part_01" spawn_attached="true">
