Commit message: WIP: Tool/scene position updates

File: catkin_ws/src/o2ac_scene_description/urdf/assembly_scene.xacro (robot description, xacro)
@@ -1,11 +1,12 @@
 <?xml version="1.0"?>
 <robot xmlns:xacro="http://www.ros.org/wiki/xacro" name="assembly_scene">
-  <!-- Trays -->
   <xacro:include filename="$(find o2ac_parts_description)/urdf/assembly_parts_macros.urdf.xacro"/>
   <!-- <xacro:include filename="$(find o2ac_parts_description)/urdf/display_all_parts.urdf.xacro"/> -->
+  <!-- ====== Uncomment this block to show the completed assembly -->
   <xacro:include filename="$(find o2ac_parts_description)/urdf/generated/full_assembly.urdf.xacro"/>
   <xacro:full_assembly prefix="assembled_" parent="attached_base_origin_link">
     <origin xyz=".12 .2 0" rpy="0 0 ${-pi/2}" />
   </xacro:full_assembly>
+  <!-- ====== Uncomment this block to add the frames of the complete assembly, but not the objects -->
   <!-- <xacro:include filename="$(find o2ac_parts_description)/urdf/generated/full_assembly_frames_only.urdf.xacro"/>
   <xacro:full_assembly_frames_only prefix="assembled_" parent="workspace_center">

File: catkin_ws/src/o2ac_scene_description/urdf/base_scene.urdf.xacro (robot description, xacro)
@@ -51,5 +51,5 @@
     elbow_joint_lower_limit="0.0" elbow_joint_upper_limit="${pi}"
     wrist_1_lower_limit="${-pi}" wrist_1_upper_limit="${pi}"
-    wrist_2_lower_limit="${-pi}" wrist_2_upper_limit="${pi}"
+    wrist_2_lower_limit="${-pi*1.5}" wrist_2_upper_limit="${pi*1.5}"
     wrist_3_lower_limit="${-pi}" wrist_3_upper_limit="${pi}"
     transmission_hw_interface="hardware_interface/PositionJointInterface"
@@ -63,5 +63,5 @@
     elbow_joint_lower_limit="0.0" elbow_joint_upper_limit="${pi}"
     wrist_1_lower_limit="${-pi}" wrist_1_upper_limit="${pi}"
-    wrist_2_lower_limit="${-pi}" wrist_2_upper_limit="${pi}"
+    wrist_2_lower_limit="${-pi*1.5}" wrist_2_upper_limit="${pi*1.5}"
     wrist_3_lower_limit="${-pi}" wrist_3_upper_limit="${pi}"
     transmission_hw_interface="hardware_interface/PositionJointInterface"

File: catkin_ws/src/o2ac_scene_description/urdf/components/nut_holder.xacro (robot description, xacro)
@@ -1,4 +1,6 @@
 <?xml version="1.0"?>
 <robot xmlns:xacro="http://www.ros.org/wiki/xacro" name="task_board">
+  <!-- To use the tip of the holder to place the macro, use these offsets: -->
+  <!-- <origin xyz="${+0.01} ${+.03} ${-0.0465}" rpy="0 0 0" />   -->
   <xacro:macro name="nut_holder" params="partname parent *origin">
   <xacro:property name="mesh_file" value="package://o2ac_scene_description/meshes/nut_holder.stl" />
@@ -33,7 +35,13 @@
     <parent link="${partname}"/>
     <child link="${partname}_collar_link"/>
-    <origin rpy="0 0 0" xyz="-0.01 -.03 0.04"/>
+    <origin rpy="0 ${pi/2} 0" xyz="-0.01 -.03 0.04"/>
   </joint>
   <link name="${partname}_collar_link"/>
+  <joint name="${partname}_tip_joint" type="fixed">
+    <parent link="${partname}_collar_link"/>
+    <child link="${partname}_tip_link"/>
+    <origin rpy="0 0 0" xyz="-0.01 0 0"/>
+  </joint>
+  <link name="${partname}_tip_link"/>
   </xacro:macro>
 </robot>

File: catkin_ws/src/o2ac_scene_description/urdf/components/tools.xacro (robot description, xacro)
@@ -5,112 +5,12 @@
 <!-- The gripper center would be about 44 mm from the top, so the tip might be 111 mm further down -->
 <!-- The tip\axis seems to be 11.5 mm from the "front" side. The front side looks into the gripper -->
-  <!-- Belt hook tool -->
-  <link name="belt_tool_holder">
-    <visual>
-      <origin rpy="${pi/2} 0 ${pi/2}" xyz="0 -.025 -.005"/>
-      <geometry>
-        <mesh filename="package://o2ac_scene_description/meshes/gravity_tool_holder.stl" scale="0.001 0.001 0.001"/>
-      </geometry>
-      <material name="grey">
-        <color rgba=".5 .5 .5 1"/>
-      </material>
-    </visual>
-    <collision>
-      <origin rpy="0 0 0" xyz="0 0 0"/>
-      <geometry>
-        <box size=".001 .001 .001"/>
-      </geometry>
-    </collision>
-  </link>
-  <joint name="belt_holder_to_environment_joint" type="fixed">
-    <parent link="b_bot_base" />
-    <child link="belt_tool_holder" />
-    <origin xyz=".325 -.2 .0" rpy="0 0 0" />
-  </joint>
-  <link name="belt_tool_link">
-    <inertial>
-      <origin rpy="0 0 0" xyz="0 0 0"/>
-      <mass value="1.0"/>
-      <inertia ixx="1" ixy="0" ixz="0" iyy="1" iyz="0" izz="1"/>
-    </inertial>
-    <visual>
-      <origin rpy="0 0 ${-pi/2}" xyz="0.02 0 -0.017"/>
-      <geometry>
-        <mesh filename="package://o2ac_scene_description/meshes/belt_hook_tool.stl" scale="0.001 0.001 0.001"/>
-      </geometry>
-      <material name="white">
-        <color rgba=".9 .9 .9 1"/>
-      </material>
-    </visual>
-    <collision>
-      <origin rpy="0 0 0" xyz="0 0 0"/>
-      <geometry>
-        <box size=".026 .04 .055"/>
-      </geometry>
-    </collision>
-  </link>
-  <joint name="belt_tool_to_holder" type="fixed">
-    <parent link="belt_tool_holder" />
-    <child link="belt_tool_link" />
-    <origin xyz="0 0 0" rpy="0 0 0" />
-  </joint>
-  <!-- Plunger tool -->
-  <link name="plunger_tool_holder">
-    <visual>
-      <origin rpy="${pi/2} 0 ${pi/2}" xyz="0 -.025 -.005"/>
-      <geometry>
-        <mesh filename="package://o2ac_scene_description/meshes/gravity_tool_holder.stl" scale="0.001 0.001 0.001"/>
-      </geometry>
-      <material name="grey">
-        <color rgba=".5 .5 .5 1"/>
-      </material>
-    </visual>
-    <collision>
-      <origin rpy="0 0 0" xyz="0 0 0"/>
-      <geometry>
-        <box size=".001 .001 .001"/>
-      </geometry>
-    </collision>
-  </link>
-  <joint name="plunger_holder_to_environment_joint" type="fixed">
-    <parent link="b_bot_base" />
-    <child link="plunger_tool_holder" />
-    <origin xyz=".325 -.1 .0" rpy="0 0 0" />
-  </joint>
-  <link name="plunger_tool_link">
-    <inertial>
-      <origin rpy="0 0 0" xyz="0 0 0"/>
-      <mass value="1.0"/>
-      <inertia ixx="1" ixy="0" ixz="0" iyy="1" iyz="0" izz="1"/>
-    </inertial>
-    <visual>
-      <origin rpy="0 ${pi/2} ${pi/2}" xyz="0.02 0 -0.017"/>
-      <geometry>
-        <mesh filename="package://o2ac_scene_description/meshes/plunger_tool.stl" scale="0.001 0.001 0.001"/>
-      </geometry>
-      <material name="white">
-        <color rgba=".9 .9 .9 1"/>
-      </material>
-    </visual>
-    <collision>
-      <origin rpy="0 0 0" xyz="0 0 0"/>
-      <geometry>
-        <box size=".026 .04 .055"/>
-      </geometry>
-    </collision>
-  </link>
-  <joint name="plunger_tool_to_holder" type="fixed">
-    <parent link="plunger_tool_holder" />
-    <child link="plunger_tool_link" />
-    <origin xyz="0 0 0" rpy="0 0 0" />
-  </joint>
-  <!-- +++++++++++++++++++ -->
-  <!-- Tools at the back of the robot system -->
-  <joint name="screw_holder_to_environment_joint" type="fixed">
+  <!-- Tool holders at the back of the robot system -->
+  <!-- The long tool holder with 3 tools -->
+  <joint name="screw_tool_holder_long_to_environment_joint" type="fixed">
     <parent link="horizontal_column_for_tools" />
-    <child link="screw_tool_holder" />
+    <child link="screw_tool_holder_long" />
     <origin xyz=".04 .0 .04" rpy="0.0 0.0 ${-pi/2}" />
   </joint>
-  <link name="screw_tool_holder">
+  <link name="screw_tool_holder_long">
     <inertial>
       <origin rpy="0 0 0" xyz="0 0 0"/>
@@ -151,7 +51,55 @@
     </collision>
   </link>
+  <!-- ==== -->
+  <!-- The short tool holder with a single tool -->
+  <joint name="screw_holder_short_to_environment_joint" type="fixed">
+    <parent link="horizontal_column_for_tools" />
+    <child link="screw_tool_holder_short" />
+    <origin xyz=".04 .3 .04" rpy="0.0 0.0 ${-pi/2}" />
+  </joint>
+  <link name="screw_tool_holder_short">
+    <inertial>
+      <origin rpy="0 0 0" xyz="0 0 0"/>
+      <mass value="1.0"/>
+      <inertia ixx="1" ixy="0" ixz="0" iyy="1" iyz="0" izz="1"/>
+    </inertial>
+    <!-- The horizontal plate -->
+    <visual>
+      <origin rpy="0 0 0" xyz="-0.05 .0013 0.002"/>
+      <geometry>
+        <box size=".1 .066 .004"/>
+      </geometry>
+      <material name="whitish">
+        <color rgba=".7 .7 .7 1"/>
+      </material>
+    </visual>
+    <collision>
+      <origin rpy="0 0 0" xyz="-0.05 .0013 0.002"/>
+      <geometry>
+        <box size=".1 .066 .004"/>
+      </geometry>
+    </collision>
+    <!-- The vertical plate -->
+    <visual>
+      <origin rpy="0 0 0" xyz="-0.05 -.014 0.0179"/>
+      <geometry>
+        <box size=".1 .004 .035"/>
+      </geometry>
+      <material name="grey">
+        <color rgba=".5 .5 .5 1"/>
+      </material>
+    </visual>
+    <collision>
+      <origin rpy="0 0 0" xyz="-0.05 -.014 0.0179"/>
+      <geometry>
+        <box size=".1 .004 .035"/>
+      </geometry>
+    </collision>
+  </link>
   <!-- ++++++++++++++++++++++++++++ -->
-  <!-- Screw tools -->
+  <!-- Screw tools on the holders in the back of the system -->
   <xacro:property name="bit_cushion_to_axis" value="0.0285"/>
+  <xacro:property name="back_plate_offset_long" value=".009"/>
+  <xacro:property name="back_plate_offset_short" value=".01"/>
   <xacro:property name="tool_offset" value="${-.005 + bit_cushion_to_axis}" />
   <!-- The collision boxes of the tools only include the top part (not what is hanging underneath the holder) -->
@@ -162,8 +110,63 @@
       <inertia ixx="1" ixy="0" ixz="0" iyy="1" iyz="0" izz="1"/>
     </inertial>
-    <!-- <visual>
-      <origin rpy="0 0 0" xyz="0 0 0"/>
-      <geometry>
-        <mesh filename="package://o2ac_scene_description/meshes/nut_tool_m6_BC5-XL320-LG20-R_v2.stl" scale="0.001 0.001 0.001"/>
+    <visual>
+      <origin rpy="0 0 0" xyz="0 0 ${.052/2}"/>
+      <geometry>
+        <box size=".026 .059 .052"/>
+      </geometry>
+      <material name="yellowish">
+        <color rgba=".9 .9 .7 1"/>
+      </material>
+    </visual>
+    <collision>
+      <origin rpy="0 0 0" xyz="0 0 ${.052/2}"/>
+      <geometry>
+        <box size=".026 .059 .052"/>
+      </geometry>
+    </collision>
+  </link>
+  <joint name="nut_tool_m6_to_holder" type="fixed">
+    <parent link="screw_tool_holder_long" />
+    <child link="nut_tool_m6_link" />
+    <origin xyz="-0.05 ${-back_plate_offset_long + .059/2 + .0155} 0.004" rpy="0.0 0.0 0.0" />
+    <!-- .0155 is the distance from the center of the box to the axis of the tool -->
+  </joint>
+  <link name="set_screw_tool_link">
+    <inertial>
+      <origin rpy="0 0 0" xyz="0 0 0"/>`
+      <mass value="1.0"/>
+      <inertia ixx="1" ixy="0" ixz="0" iyy="1" iyz="0" izz="1"/>
+    </inertial>
+    <visual>
+      <origin rpy="0 0 0" xyz="0 0 ${.052/2}"/>
+      <geometry>
+        <box size=".026 .059 .052"/>
+      </geometry>
+      <material name="yellowish">
+        <color rgba=".9 .9 .7 1"/>
+      </material>
+    </visual>
+    <collision>
+      <origin rpy="0 0 0" xyz="0 0 ${.052/2}"/>
+      <geometry>
+        <box size=".026 .059 .052"/>
+      </geometry>
+    </collision>
+  </link>
+  <joint name="set_screw_tool_to_holder" type="fixed">
+    <parent link="screw_tool_holder_short" />
+    <child link="set_screw_tool_link" />
+    <origin xyz="-0.05 ${-back_plate_offset_short + .059/2 + .0155} 0.004" rpy="0.0 0.0 0.0" />
+  </joint>
+  <link name="screw_tool_m4_link">
+    <inertial>
+      <origin rpy="0 0 0" xyz="0 0 0"/>
+      <mass value="1.0"/>
+      <inertia ixx="1" ixy="0" ixz="0" iyy="1" iyz="0" izz="1"/>
+    </inertial>
+    <visual>
+      <origin rpy="0 0 0" xyz="0 0 0"/>
+      <geometry>
+        <mesh filename="package://o2ac_scene_description/meshes/screw_tool_m4_BC5-XL320-AY3.5-EH3R4.stl" scale="0.001 0.001 0.001"/>
       </geometry>
       <material name="white">
@@ -176,33 +179,21 @@
         <box size=".026 .04 .055"/>
       </geometry>
-    </collision> -->
-  </link>
-  <joint name="nut_tool_m6_to_holder" type="fixed">
-    <parent link="screw_tool_holder" />
-    <child link="nut_tool_m6_link" />
-    <origin xyz="-0.35 ${tool_offset} 0.004" rpy="0.0 0.0 0.0" />
-  </joint>
-  <link name="set_screw_tool_link">
-    <inertial>
-      <origin rpy="0 0 0" xyz="0 0 0"/>
-      <mass value="1.0"/>
-      <inertia ixx="1" ixy="0" ixz="0" iyy="1" iyz="0" izz="1"/>
-    </inertial>
-  </link>
-  <joint name="set_screw_tool_to_holder" type="fixed">
-    <parent link="screw_tool_holder" />
-    <child link="set_screw_tool_link" />
-    <origin xyz="-0.355 ${tool_offset- .015} 0.004" rpy="0.0 0.0 0.0" />
-  </joint>
-  <link name="screw_tool_m4_link">
-    <inertial>
-      <origin rpy="0 0 0" xyz="0 0 0"/>
-      <mass value="1.0"/>
-      <inertia ixx="1" ixy="0" ixz="0" iyy="1" iyz="0" izz="1"/>
-    </inertial>
-    <visual>
-      <origin rpy="0 0 0" xyz="0 0 0"/>
-      <geometry>
-        <mesh filename="package://o2ac_scene_description/meshes/screw_tool_m4_BC5-XL320-AY3.5-EH3R4.stl" scale="0.001 0.001 0.001"/>
+    </collision>
+  </link>
+  <joint name="screw_tool_m4_to_holder" type="fixed">
+    <parent link="screw_tool_holder_long" />
+    <child link="screw_tool_m4_link" />
+    <origin xyz="-0.15 ${tool_offset} 0.004" rpy="0.0 0.0 0.0" />
+  </joint>
+  <link name="screw_tool_m3_link">
+    <inertial>
+      <origin rpy="0 0 0" xyz="0 0 0"/>
+      <mass value="1.0"/>
+      <inertia ixx="1" ixy="0" ixz="0" iyy="1" iyz="0" izz="1"/>
+    </inertial>
+    <visual>
+      <origin rpy="0 0 0" xyz="0 0 0"/>
+      <geometry>
+        <mesh filename="package://o2ac_scene_description/meshes/screw_tool_m3_BC5-XL320-R-AY2.6-EH2.stl" scale="0.001 0.001 0.001"/>
       </geometry>
       <material name="white">
@@ -217,33 +208,6 @@
     </collision>
   </link>
-  <joint name="screw_tool_m4_to_holder" type="fixed">
-    <parent link="screw_tool_holder" />
-    <child link="screw_tool_m4_link" />
-    <origin xyz="-0.15 ${tool_offset} 0.004" rpy="0.0 0.0 0.0" />
-  </joint>
-  <link name="screw_tool_m3_link">
-    <inertial>
-      <origin rpy="0 0 0" xyz="0 0 0"/>
-      <mass value="1.0"/>
-      <inertia ixx="1" ixy="0" ixz="0" iyy="1" iyz="0" izz="1"/>
-    </inertial>
-    <visual>
-      <origin rpy="0 0 0" xyz="0 0 0"/>
-      <geometry>
-        <mesh filename="package://o2ac_scene_description/meshes/screw_tool_m3_BC5-XL320-R-AY2.6-EH2.stl" scale="0.001 0.001 0.001"/>
-      </geometry>
-      <material name="white">
-        <color rgba=".9 .9 .9 1"/>
-      </material>
-    </visual>
-    <collision>
-      <origin rpy="0 0 0" xyz="0 ${bit_cushion_to_axis - .02} .0275"/>
-      <geometry>
-        <box size=".026 .04 .055"/>
-      </geometry>
-    </collision>
-  </link>
   <joint name="screw_tool_m3_to_holder" type="fixed">
-    <parent link="screw_tool_holder" />
+    <parent link="screw_tool_holder_long" />
     <child link="screw_tool_m3_link" />
     <origin xyz="-0.25 ${tool_offset} 0.004" rpy="0.0 0.0 0.0" />
@@ -254,5 +218,5 @@
     <parent link="screw_tool_m3_link" />
     <child link="screw_tool_m3_pickup_link" />
-    <origin xyz="0.0 0.0 0.0" rpy="0.0 0.0 ${-pi/2}" />
+    <origin xyz="0.0 0.0 0.0" rpy="0.0 ${pi} ${pi/2}" />
   </joint>
   <link name="screw_tool_m4_pickup_link"/>
@@ -260,5 +224,5 @@
     <parent link="screw_tool_m4_link" />
     <child link="screw_tool_m4_pickup_link" />
-    <origin xyz="0.0 0.0 0.0" rpy="0.0 0.0 ${-pi/2}" />
+    <origin xyz="0.0 0.0 0.0" rpy="0.0 ${pi} ${pi/2}" />
   </joint>
   <link name="belt_tool_pickup_link"/>
@@ -266,5 +230,5 @@
     <parent link="belt_tool_link" />
     <child link="belt_tool_pickup_link" />
-    <origin xyz="0.0 0.0 0.0" rpy="0.0 0.0 ${-pi/2}" />
+    <origin xyz="0.0 0.0 0.0" rpy="0.0 ${pi} ${pi/2}" />
   </joint>
   <link name="nut_tool_m6_pickup_link"/>
@@ -272,5 +236,5 @@
     <parent link="nut_tool_m6_link" />
     <child link="nut_tool_m6_pickup_link" />
-    <origin xyz="0.0 0.0 0.0" rpy="0.0 0.0 ${-pi/2}" />
+    <origin xyz="0.0 0.0 0.0" rpy="0.0 ${pi} ${pi/2}" />
   </joint>
   <link name="set_screw_tool_pickup_link"/>
@@ -278,5 +242,107 @@
     <parent link="set_screw_tool_link" />
     <child link="set_screw_tool_pickup_link" />
-    <origin xyz="0.0 0.0 0.0" rpy="0.0 0.0 ${-pi/2}" />
+    <origin xyz="0.0 0.0 0.0" rpy="0.0 ${pi} ${pi/2}" />
+  </joint>
+<!-- ================ -->
+<!-- Tools at the front of b_bot base -->
+<!-- Belt hook tool -->
+  <link name="belt_tool_holder">
+    <visual>
+      <origin rpy="${pi/2} 0 ${pi/2}" xyz="0 -.025 -.005"/>
+      <geometry>
+        <mesh filename="package://o2ac_scene_description/meshes/gravity_tool_holder.stl" scale="0.001 0.001 0.001"/>
+      </geometry>
+      <material name="grey">
+        <color rgba=".5 .5 .5 1"/>
+      </material>
+    </visual>
+    <collision>
+      <origin rpy="0 0 0" xyz="0 0 0"/>
+      <geometry>
+        <box size=".001 .001 .001"/>
+      </geometry>
+    </collision>
+  </link>
+  <joint name="belt_holder_to_environment_joint" type="fixed">
+    <parent link="b_bot_base" />
+    <child link="belt_tool_holder" />
+    <origin xyz=".325 -.2 .0" rpy="0 0 0" />
+  </joint>
+  <link name="belt_tool_link">
+    <inertial>
+      <origin rpy="0 0 0" xyz="0 0 0"/>
+      <mass value="1.0"/>
+      <inertia ixx="1" ixy="0" ixz="0" iyy="1" iyz="0" izz="1"/>
+    </inertial>
+    <visual>
+      <origin rpy="0 0 ${-pi/2}" xyz="0.02 0 -0.017"/>
+      <geometry>
+        <mesh filename="package://o2ac_scene_description/meshes/belt_hook_tool.stl" scale="0.001 0.001 0.001"/>
+      </geometry>
+      <material name="white">
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
File: catkin_ws/src/o2ac_scene_description/urdf/components/washer_holder.xacro (robot description, xacro)
@@ -1,4 +1,6 @@
 <?xml version="1.0"?>
 <robot xmlns:xacro="http://www.ros.org/wiki/xacro" name="task_board">
+  <!-- To use the tip of the holder to place the macro, use these offsets: -->
+  <!-- <origin xyz="${+0.01} ${+.03} ${-0.0465}" rpy="0 0 0" />   -->
   <xacro:macro name="washer_holder" params="partname parent *origin">
   <xacro:property name="mesh_file" value="package://o2ac_scene_description/meshes/washer_holder.stl" />

File: catkin_ws/src/o2ac_scene_description/urdf/o2ac_environment.xacro (robot description, xacro)
@@ -15,5 +15,5 @@
   </xacro:o2ac_box>
   <xacro:o2ac_box boxname="horizontal_column_for_tools" box_w=".04" box_l=".4" box_h=".04" parent="o2ac_ground">
-    <origin xyz="${vert_column_x_back} -.2 1.05" rpy="0 0 0" />
+    <origin xyz="${vert_column_x_back} -.2 1.058" rpy="0 0 0" />
   </xacro:o2ac_box>
   <!-- Screw holder & screw tool visual -->
