Commit message: Update scene, calibration and convenience scripts

File: catkin_ws/src/o2ac_scene_description/urdf/assembly_scene.xacro (robot description, xacro)
@@ -4,11 +4,11 @@
   <!-- <xacro:include filename="$(find o2ac_parts_description)/urdf/display_all_parts.urdf.xacro"/> -->
   <!-- ====== Uncomment this block to show the completed assembly -->
-  <xacro:include filename="$(find o2ac_parts_description)/urdf/generated/full_assembly.urdf.xacro"/>
+  <!-- <xacro:include filename="$(find o2ac_parts_description)/urdf/generated/full_assembly.urdf.xacro"/>
   <xacro:full_assembly prefix="assembled_" parent="attached_base_origin_link">
     <origin xyz=".12 .2 0" rpy="0 0 ${-pi/2}" />
   </xacro:full_assembly> -->
   <!-- ====== Uncomment this block to add the frames of the complete assembly, but not the objects -->
-  <!-- <xacro:include filename="$(find o2ac_parts_description)/urdf/generated/full_assembly_frames_only.urdf.xacro"/>
-  <xacro:full_assembly_frames_only prefix="assembled_" parent="workspace_center">
+  <xacro:include filename="$(find o2ac_parts_description)/urdf/generated/full_assembly_frames_only.urdf.xacro"/>
+  <xacro:full_assembly_frames_only prefix="assembled_" parent="attached_base_origin_link">
     <origin xyz=".12 .2 0" rpy="0 0 ${-pi/2}" />
   </xacro:full_assembly_frames_only>

File: catkin_ws/src/o2ac_scene_description/urdf/base_scene.urdf.xacro (robot description, xacro)
@@ -20,6 +20,6 @@
   <!-- <xacro:include filename="$(find flexwrist_experiment)/urdf/2020-01-experiment-scene.xacro" /> -->
   <!-- <xacro:include filename="$(find o2ac_scene_description)/urdf/taskboard_scene.xacro" /> -->
-  <!-- <xacro:include filename="$(find o2ac_scene_description)/urdf/assembly_scene.xacro" /> -->
-  <xacro:include filename="$(find o2ac_scene_description)/urdf/calibration_scene.xacro" />
+  <xacro:include filename="$(find o2ac_scene_description)/urdf/assembly_scene.xacro" />
+  <!-- <xacro:include filename="$(find o2ac_scene_description)/urdf/calibration_scene.xacro" /> -->
   <!-- Robot bases -->
   <!-- Putting these at height 0.0 makes them intersect with the ground, so they are elevated. -->
@@ -48,10 +48,10 @@
   </joint>
   <xacro:ur5e_robot prefix="a_bot_" joint_limited="true"
-    shoulder_pan_lower_limit="${-pi/1.5}" shoulder_pan_upper_limit="${pi/1.5}"
-    shoulder_lift_lower_limit="${-pi/1.5}" shoulder_lift_upper_limit="${pi/1.5}"
+    shoulder_pan_lower_limit="${-pi}" shoulder_pan_upper_limit="${pi}"
+    shoulder_lift_lower_limit="${-pi}" shoulder_lift_upper_limit="${pi}"
     elbow_joint_lower_limit="0.0" elbow_joint_upper_limit="${pi}"
     wrist_1_lower_limit="${-pi}" wrist_1_upper_limit="${pi}"
     wrist_2_lower_limit="${-pi*1.5}" wrist_2_upper_limit="${pi*1.5}"
-    wrist_3_lower_limit="${-pi}" wrist_3_upper_limit="${pi}"
+    wrist_3_lower_limit="${-2*pi}" wrist_3_upper_limit="${2*pi}"
     transmission_hw_interface="hardware_interface/PositionJointInterface"
     safety_limits="false" safety_pos_margin="0.15"
@@ -65,5 +65,5 @@
     wrist_1_lower_limit="${-pi}" wrist_1_upper_limit="${pi}"
     wrist_2_lower_limit="${-pi*1.5}" wrist_2_upper_limit="${pi*1.5}"
-    wrist_3_lower_limit="${-pi}" wrist_3_upper_limit="${pi}"
+    wrist_3_lower_limit="${-2*pi}" wrist_3_upper_limit="${2*pi}"
     transmission_hw_interface="hardware_interface/PositionJointInterface"
     safety_limits="false" safety_pos_margin="0.15"

File: catkin_ws/src/o2ac_scene_description/urdf/components/base_fixture.xacro (robot description, xacro)
@@ -1,4 +1,4 @@
 <?xml version="1.0"?>
-<robot xmlns:xacro="http://www.ros.org/wiki/xacro" name="task_board">
+<robot xmlns:xacro="http://www.ros.org/wiki/xacro" name="base_fixture">
   <xacro:macro name="base_fixture" params="parent *origin">
   <xacro:property name="top_mesh" value="package://o2ac_scene_description/meshes/base_fixture_reoriented.stl" />
@@ -90,7 +90,7 @@
   <link name="left_bar">
     <visual>
-      <origin rpy="0 0 0" xyz="${width/2} 0.01 .04"/>
+      <origin rpy="0 0 0" xyz="${width/2-.02} 0.01 .04"/>
       <geometry>
-        <box size="${width} .02 .08"/>
+        <box size="${width-.04} .02 .08"/>
         <!-- <mesh filename="${long_bar_mesh}" scale=".001 .001 .001"/> -->
       </geometry>
@@ -100,7 +100,7 @@
     </visual>
     <collision>
-      <origin rpy="0 0 0" xyz="${width/2} 0.01 .04"/>
+      <origin rpy="0 0 0" xyz="${width/2-.02} 0.01 .04"/>
       <geometry>
-        <box size="${width} .02 .08"/>
+        <box size="${width-.04} .02 .08"/>
       </geometry>
     </collision>
@@ -113,7 +113,7 @@
   <link name="right_bar">
     <visual>
-      <origin rpy="0 0 0" xyz="${width/2} 0.01 .04"/>
+      <origin rpy="0 0 0" xyz="${width/2-.02} 0.01 .04"/>
       <geometry>
-        <box size="${width} .02 .08"/>
+        <box size="${width-.04} .02 .08"/>
         <!-- <mesh filename="${long_bar_mesh}" scale=".001 .001 .001"/> -->
       </geometry>
@@ -123,7 +123,7 @@
     </visual>
     <collision>
-      <origin rpy="0 0 0" xyz="${width/2} 0.01 .04"/>
+      <origin rpy="0 0 0" xyz="${width/2-.02} 0.01 .04"/>
       <geometry>
-        <box size="${width} .02 .08"/>
+        <box size="${width-.04} .02 .08"/>
       </geometry>
     </collision>

File: catkin_ws/src/o2ac_scene_description/urdf/components/o2ac_end_effector.urdf.xacro (robot description, xacro)
@@ -38,5 +38,5 @@
       <parent link="${prefix}robotiq_85_base_link"/>
       <child link="${prefix}robotiq_85_tip_link"/>
-      <origin rpy="0.0 0.0 0.0" xyz=".163 0.0 0.0"/>
+      <origin rpy="0 0 0" xyz=".163 0 0"/>
     </joint>
     <link name="${prefix}robotiq_85_tip_link"/>
@@ -47,5 +47,5 @@
       <parent link="${prefix}robotiq_85_tip_link"/>
       <child link="${prefix}tool_intermediate_link"/>
-      <origin rpy="${pi} 0.0 0.0" xyz="-.03 0.0 0.0"/>
+      <origin rpy="${pi} ${-pi/3} 0" xyz="-.03 0 0"/>
     </joint>
     <link name="${prefix}tool_intermediate_link"/>
@@ -53,5 +53,5 @@
       <parent link="${prefix}tool_intermediate_link"/>
       <child link="${prefix}nut_tool_m6_tip_link"/>
-      <origin rpy="0.0 ${pi/4} 0.0" xyz="0.0 0.0 -0.12 "/>
+      <origin rpy="0 0 0" xyz="0.12 0 0 "/>
     </joint>
     <link name="${prefix}nut_tool_m6_tip_link"/>
@@ -59,5 +59,5 @@
       <parent link="${prefix}tool_intermediate_link"/>
       <child link="${prefix}screw_tool_m4_tip_link"/>
-      <origin rpy="0.0 ${pi/2} 0.0" xyz="-.002 0.0 -0.146 "/>
+      <origin rpy="0 0 0" xyz=".141 0 0.005 "/>
     </joint>
     <link name="${prefix}screw_tool_m4_tip_link"/>
@@ -65,5 +65,5 @@
       <parent link="${prefix}tool_intermediate_link"/>
       <child link="${prefix}screw_tool_m3_tip_link"/>
-      <origin rpy="0.0 ${pi/2} 0.0" xyz=".015 0.0 -0.14 "/>
+      <origin rpy="0 0 0" xyz=".14 0 .015 "/>
     </joint>
     <link name="${prefix}screw_tool_m3_tip_link"/>
@@ -71,5 +71,5 @@
       <parent link="${prefix}robotiq_85_tip_link"/>
       <child link="${prefix}set_screw_tool_tip_link"/>
-      <origin rpy="0.0 ${-pi/6} 0.0" xyz=".0045 0.0 0.047 "/>
+      <origin rpy="0 0 0" xyz=".0049 0 0.01"/>
     </joint>
     <link name="${prefix}set_screw_tool_tip_link"/>
@@ -77,5 +77,5 @@
       <parent link="${prefix}tool_intermediate_link"/>
       <child link="${prefix}dual_suction_gripper_pad_link"/>
-      <origin rpy="0.0 0 0.0" xyz="0 0 0 "/>
+      <origin rpy="0 0 0" xyz="0 0 0 "/>
     </joint>
     <link name="${prefix}dual_suction_gripper_pad_link"/>

File: catkin_ws/src/o2ac_scene_description/urdf/o2ac_environment.xacro (robot description, xacro)
@@ -30,5 +30,5 @@
   <xacro:include filename="$(find o2ac_scene_description)/urdf/components/base_fixture.xacro" />
   <xacro:base_fixture parent="workspace_center">
-    <origin xyz="-0.27 -.18 0" rpy="0 0 0" />
+    <origin xyz="-0.294 -.18 0" rpy="0 0 0" />
   </xacro:base_fixture>
   <!-- Tray -->
