Commit message: Fix gripper 85 simulation

File: catkin_ws/src/o2ac_scene_description/urdf/b_bot.urdf (robot description, URDF)
Before this commit: robot o2ac_base_scene, 53 links, 52 joints
Links:
- removed link b_bot_robotiq_140_base_link
- added link b_bot_coupling; collision cylinder length=0.01 radius=0.0375; visual cylinder length=0.01 radius=0.0375
- added link b_bot_robotiq_85_base_link
- link b_bot_left_inner_finger: geometry collision mesh filename=package://robotiq_2f_85_gripper_visualization/meshes/collis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 scale=0.001 0.001 0.001; visual mesh filename=package://robotiq_2f_85_gripper_visualization/meshes/visual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 scale=0.001 0.001 0.001
- link b_bot_left_inner_finger_pad: geometry collision box size=0.022 0.00635 0.0375; visual box size=0.022 0.00635 0.0375
- link b_bot_left_inner_knuckle: geometry collision mesh filename=package://robotiq_2f_85_gripper_visualization/meshes/collis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 scale=0.001 0.001 0.001; visual mesh filename=package://robotiq_2f_85_gripper_visualization/meshes/visual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 scale=0.001 0.001 0.001
- link b_bot_left_outer_finger: geometry collision mesh filename=package://robotiq_2f_85_gripper_visualization/meshes/collis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 scale=0.001 0.001 0.001; visual mesh filename=package://robotiq_2f_85_gripper_visualization/meshes/visual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 scale=0.001 0.001 0.001
- link b_bot_left_outer_knuckle: geometry collision mesh filename=package://robotiq_2f_85_gripper_visualization/meshes/collis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 scale=0.001 0.001 0.001; visual mesh filename=package://robotiq_2f_85_gripper_visualization/meshes/visual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 scale=0.001 0.001 0.001
- link b_bot_right_inner_finger: geometry collision mesh filename=package://robotiq_2f_85_gripper_visualization/meshes/collis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 scale=0.001 0.001 0.001; visual mesh filename=package://robotiq_2f_85_gripper_visualization/meshes/visual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 scale=0.001 0.001 0.001
- link b_bot_right_inner_finger_pad: geometry collision box size=0.022 0.00635 0.0375; visual box size=0.022 0.00635 0.0375
- link b_bot_right_inner_knuckle: geometry collision mesh filename=package://robotiq_2f_85_gripper_visualization/meshes/collis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 scale=0.001 0.001 0.001; visual mesh filename=package://robotiq_2f_85_gripper_visualization/meshes/visual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 scale=0.001 0.001 0.001
- link b_bot_right_outer_finger: geometry collision mesh filename=package://robotiq_2f_85_gripper_visualization/meshes/collis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 scale=0.001 0.001 0.001; visual mesh filename=package://robotiq_2f_85_gripper_visualization/meshes/visual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 scale=0.001 0.001 0.001
- link b_bot_right_outer_knuckle: geometry collision mesh filename=package://robotiq_2f_85_gripper_visualization/meshes/collis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 scale=0.001 0.001 0.001; visual mesh filename=package://robotiq_2f_85_gripper_visualization/meshes/visual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 scale=0.001 0.001 0.001
Joints:
- removed joint b_bot_robotiq_140_base_joint
- removed joint world_joint
- added joint b_bot_coupling_joint: type fixed, parent b_bot_ee_link, child b_bot_coupling, origin xyz=0 0 0 rpy=0 0 0
- added joint b_bot_robotiq_85_base_joint: type fixed, parent b_bot_ee_link, child b_bot_robotiq_85_base_link, origin xyz=0.01 0 0 rpy=0.0 0.0 0.0
- added joint world_b_bot_joint: type fixed, parent world, child b_bot_base_link, origin xyz=-0.0 0.525 0.75 rpy=0.0 0.0 -3.141
- added joint world_o2ac_joint: type fixed, parent world, child b_bot_base_link, origin xyz=0.0 0.0 0.0 rpy=0.0 0.0 0.0
- joint b_bot_cam_cables_joint: parent b_bot_robotiq_140_base_link -> b_bot_robotiq_85_base_link
- joint b_bot_cam_mount_joint: parent b_bot_robotiq_140_base_link -> b_bot_robotiq_85_base_link
- joint b_bot_finger_joint: axis -1 0 0 -> 1 0 0; limit lower=0 upper=0.7 effort=1000 velocity=2.0 -> lower=0 upper=0.9 effort=1000 velocity=2.0; origin xyz=0 -0.030601 0.054905 rpy=2.29579632679 0 0 -> xyz=0 -0.0306011 0.054904 rpy=0 0 3.14159265359
- joint b_bot_inside_cam_joint: parent b_bot_robotiq_140_base_link -> b_bot_robotiq_85_base_link
- joint b_bot_left_inner_finger_joint: mimic joint=b_bot_finger_joint multiplier=1 offset=0 -> joint=b_bot_finger_joint multiplier=-1 offset=0; origin xyz=0 0.0817554015893473 -0.0282203446692936 rpy=-0.725 0 0 -> xyz=0 0.0061 0.0471 rpy=0 0 0
- joint b_bot_left_inner_finger_pad_joint: origin xyz=0 0.0457554015893473 -0.0272203446692936 rpy=0 0 0 -> xyz=0 -0.0220203446692936 0.03242 rpy=0 0 0
- joint b_bot_left_inner_knuckle_joint: mimic joint=b_bot_finger_joint multiplier=-1 offset=0 -> joint=b_bot_finger_joint multiplier=1 offset=0; origin xyz=0 -0.0127 0.06142 rpy=2.29579632679 0 0.0 -> xyz=0 -0.0127 0.06142 rpy=0 0 3.14159265359
- joint b_bot_left_outer_finger_joint: origin xyz=0 0.01821998610742 0.0260018192872234 rpy=0 0 0 -> xyz=0 0.0315 -0.0041 rpy=0 0 0
- joint b_bot_outside_cam_joint: parent b_bot_robotiq_140_base_link -> b_bot_robotiq_85_base_link
- joint b_bot_right_inner_finger_joint: mimic joint=b_bot_finger_joint multiplier=1 offset=0 -> joint=b_bot_finger_joint multiplier=-1 offset=0; origin xyz=0 0.0817554015893473 -0.0282203446692936 rpy=-0.725 0 0 -> xyz=0 0.0061 0.0471 rpy=0 0 0
- joint b_bot_right_inner_finger_pad_joint: origin xyz=0 0.0457554015893473 -0.0272203446692936 rpy=0 0 0 -> xyz=0 -0.0220203446692936 0.03242 rpy=0 0 0
- joint b_bot_right_inner_knuckle_joint: mimic joint=b_bot_finger_joint multiplier=-1 offset=0 -> joint=b_bot_finger_joint multiplier=1 offset=0; origin xyz=0 0.0127 0.06142 rpy=2.29579632679 0 -3.14159265359 -> xyz=0 0.0127 0.06142 rpy=0 0 0.0
- joint b_bot_right_outer_finger_joint: origin xyz=0 0.01821998610742 0.0260018192872234 rpy=0 0 0 -> xyz=0 0.0315 -0.0041 rpy=0 0 0
- joint b_bot_right_outer_knuckle_joint: limit lower=-0.725 upper=0.725 effort=1000 velocity=2.0 -> lower=-0.81 upper=0.81 effort=1000 velocity=2.0; mimic joint=b_bot_finger_joint multiplier=-1 offset=0 -> joint=b_bot_finger_joint multiplier=1 offset=0; origin xyz=0 0.030601 0.054905 rpy=2.29579632679 0 3.14159265359 -> xyz=0 0.0306011 0.054904 rpy=0 0 0
- joint b_bot_robotiq_85_screw_tool_m3_tip_joint: origin xyz=.121 0 .0055  rpy=0 0 0 -> xyz=.14 0 .015  rpy=0 0 0
- joint b_bot_robotiq_85_set_screw_tool_tip_joint: origin xyz=0.058 0 0.006 rpy=0 0 0 -> xyz=0.068 0 0.0014 rpy=0 0 0
- joint b_bot_robotiq_85_tip_link_joint: origin xyz=0.246 0.0 0.0 rpy=0.0 0.0 0.0 -> xyz=.163 0 0 rpy=0 0 0; parent b_bot_robotiq_140_base_link -> b_bot_robotiq_85_base_link
- joint b_bot_robotiq_arg2f_base_joint: parent b_bot_robotiq_140_base_link -> b_bot_robotiq_85_base_link
