Commit message: Change robotiq_85_tip_link to gripper_tip_link
This was an overdue change.

File: catkin_ws/src/o2ac_scene_description/urdf/a_bot.urdf (robot description, URDF)
Before this commit: robot o2ac_base_scene, 53 links, 52 joints
Links:
- removed link a_bot_robotiq_85_tip_link
- added link a_bot_gripper_tip_link
Joints:
- removed joint a_bot_robotiq_85_tip_link_joint
- added joint a_bot_gripper_tip_link_joint: type fixed, parent a_bot_robotiq_140_base_link, child a_bot_gripper_tip_link, origin xyz=0.246 0.0 0.0 rpy=0.0 0.0 0.0
- joint a_bot_tool_intermediate_joint: parent a_bot_robotiq_85_tip_link -> a_bot_gripper_tip_link

File: catkin_ws/src/o2ac_scene_description/urdf/b_bot.urdf (robot description, URDF)
Before this commit: robot o2ac_base_scene, 54 links, 54 joints
Links:
- removed link b_bot_robotiq_85_tip_link
- added link b_bot_gripper_tip_link
Joints:
- removed joint b_bot_robotiq_85_tip_link_joint
- added joint b_bot_gripper_tip_link_joint: type fixed, parent b_bot_robotiq_85_base_link, child b_bot_gripper_tip_link, origin xyz=.163 0 0 rpy=0 0 0
- joint b_bot_tool_intermediate_joint: parent b_bot_robotiq_85_tip_link -> b_bot_gripper_tip_link

File: catkin_ws/src/o2ac_scene_description/urdf/camera_calibration_scene.xacro (robot description, xacro)
@@ -4,5 +4,5 @@
   <xacro:include filename="$(find o2ac_gazebo)/urdf/ar_markers.urdf.xacro"/>
   <!-- <xacro:ar_marker_70_5 prefix="b_bot_" -->
-  <!-- 			parent="b_bot_robotiq_85_tip_link" -->
+  <!-- 			parent="b_bot_gripper_tip_link" -->
   <!-- 			marker_id="26" -->
   <!-- 			thickness="0.005"> -->

File: catkin_ws/src/o2ac_scene_description/urdf/components/o2ac_end_effector.urdf.xacro (robot description, xacro)
@@ -35,15 +35,15 @@
     </xacro:if>
     <!-- Add an additional link to plan with. Oriented like the UR ee_link frame. -->
-    <joint name="${prefix}robotiq_85_tip_link_joint" type="fixed">
+    <joint name="${prefix}gripper_tip_link_joint" type="fixed">
       <parent link="${prefix}robotiq_85_base_link"/>
-      <child link="${prefix}robotiq_85_tip_link"/>
+      <child link="${prefix}gripper_tip_link"/>
       <origin rpy="0 0 0" xyz=".163 0 0"/>
     </joint>
-    <link name="${prefix}robotiq_85_tip_link"/>
+    <link name="${prefix}gripper_tip_link"/>
     <!-- ========= -->
     <!-- Add screw tool tip frames. X-axis points along the screw into the hole. -->
     <!-- Offset of the gripper tooltips -->
     <joint name="${prefix}tool_intermediate_joint" type="fixed">
-      <parent link="${prefix}robotiq_85_tip_link"/>
+      <parent link="${prefix}gripper_tip_link"/>
       <child link="${prefix}tool_intermediate_link"/>
       <origin rpy="${pi} ${-pi/3} 0" xyz="-.03 0 0"/>
@@ -77,5 +77,5 @@
     <!-- Add helper frames, e.g. for rotating bearing. -->
     <joint name="${prefix}bearing_rotate_helper_joint" type="fixed">
-      <parent link="${prefix}robotiq_85_tip_link"/>
+      <parent link="${prefix}gripper_tip_link"/>
       <child link="${prefix}bearing_rotate_helper_link"/>
       <origin rpy="${radians(180)} ${radians(30)} 0" xyz="-.003 0 -0.011"/>

File: catkin_ws/src/o2ac_scene_description/urdf/components/o2ac_end_effector_2F-140.urdf.xacro (robot description, xacro)
@@ -13,15 +13,15 @@
     </xacro:if>
     <!-- Add an additional link to plan with. Oriented like the UR ee_link frame. -->
-    <joint name="${prefix}robotiq_85_tip_link_joint" type="fixed">
+    <joint name="${prefix}gripper_tip_link_joint" type="fixed">
       <parent link="${prefix}robotiq_140_base_link"/>
-      <child link="${prefix}robotiq_85_tip_link"/>
+      <child link="${prefix}gripper_tip_link"/>
       <origin rpy="0.0 0.0 0.0" xyz="${.163+.083} 0.0 0.0"/>
     </joint>
-    <link name="${prefix}robotiq_85_tip_link"/>
+    <link name="${prefix}gripper_tip_link"/>
     <!-- ========= -->
     <!-- Add screw tool tip frames. X-axis points along the screw into the hole. -->
     <!-- Offset of the gripper tooltips -->
     <joint name="${prefix}tool_intermediate_joint" type="fixed">
-      <parent link="${prefix}robotiq_85_tip_link"/>
+      <parent link="${prefix}gripper_tip_link"/>
       <child link="${prefix}tool_intermediate_link"/>
       <origin rpy="${pi} ${-pi/3} 0" xyz="-.03 0 0"/>

Commit message: Fix URDF models for KDL/Force control

File: catkin_ws/src/o2ac_scene_description/urdf/a_bot.urdf (robot description, URDF)
Before this commit: robot o2ac_base_scene, 53 links, 52 joints
Links:
- removed link a_bot_left_inner_finger
- removed link a_bot_left_inner_finger_pad
- removed link a_bot_left_inner_knuckle
- removed link a_bot_left_outer_finger
- removed link a_bot_left_outer_knuckle
- removed link a_bot_right_inner_finger
- removed link a_bot_right_inner_finger_pad
- removed link a_bot_right_inner_knuckle
- removed link a_bot_right_outer_finger
- removed link a_bot_right_outer_knuckle
- added link a_bot_nut_tool_m4_hole_link
Joints:
- removed joint a_bot_finger_joint
- removed joint world_joint
- added joint a_bot__nut_tool_m4_joint: type fixed, parent a_bot_gripper_tip_link, child a_bot_nut_tool_m4_hole_link, origin xyz=0.002 0.0 .017 rpy=0.923 1.571 0.923
- added joint world_a_bot_joint: type fixed, parent world, child a_bot_base_link, origin xyz=-0.004 -0.525 0.75 rpy=0.0 0.0 0.0
- added joint world_o2ac_joint: type fixed, parent world, child o2ac_ground, origin xyz=0.0 0.0 0.0 rpy=0.0 0.0 0.0
- joint a_bot_robotiq_140_base_joint: parent a_bot_tool0 -> a_bot_ee_link

File: catkin_ws/src/o2ac_scene_description/urdf/ur5e_gripper.xacro (robot description, xacro)
@@ -13,5 +13,5 @@
   <!-- robots -->
   <xacro:include filename="$(find ur_e_description)/urdf/ur5e.urdf.xacro" />
-  <xacro:ur5e_robot prefix="b_bot_" joint_limited="true"
+  <xacro:ur5e_robot prefix="a_bot_" joint_limited="true"
     shoulder_pan_lower_limit="${-pi}" shoulder_pan_upper_limit="${pi}"
     shoulder_lift_lower_limit="${-pi}" shoulder_lift_upper_limit="${pi}"
@@ -23,13 +23,15 @@
     safety_limits="false" safety_pos_margin="0.15"
     safety_k_position="20"
-    kinematics_file="${load_yaml('$(find o2ac_scene_description)/config/b_bot_calibration.yaml')}"
+    kinematics_file="${load_yaml('$(find o2ac_scene_description)/config/a_bot_calibration.yaml')}"
   />
-  <joint name="world_b_bot_joint" type="fixed">
+  <joint name="world_a_bot_joint" type="fixed">
     <parent link="world" />
-    <child link = "b_bot_base_link" />
-    <origin xyz="${b_bot_x} ${b_bot_y} ${bots_z}" rpy="0.0 0.0 ${b_bot_theta}" />
+    <child link = "a_bot_base_link" />
+    <origin xyz="${a_bot_x} ${a_bot_y} ${bots_z}" rpy="0.0 0.0 ${a_bot_theta}" />
   </joint>
-  <xacro:include filename="$(find o2ac_scene_description)/urdf/components/o2ac_end_effector.urdf.xacro" />
-  <xacro:o2ac_end_effector prefix="b_bot_" use_soft_wrist="false" use_cameras="true" parent = "b_bot_ee_link" />
+  <xacro:include filename="$(find o2ac_scene_description)/urdf/components/o2ac_end_effector_2F-140.urdf.xacro" />
+  <xacro:o2ac_end_effector prefix="a_bot_" use_soft_wrist="false" use_cameras="true" parent = "a_bot_ee_link" />
+  <!-- <xacro:include filename="$(find o2ac_scene_description)/urdf/components/o2ac_end_effector.urdf.xacro" />
+  <xacro:o2ac_end_effector prefix="a_bot_" use_soft_wrist="false" use_cameras="true" parent = "a_bot_ee_link" /> -->
   <!-- The "world" link definition should be removed, but apparently it is necessary for Gazebo -->
   <link name="world" />
