Commit message: Add example, clean up

File: catkin_ws/src/o2ac_scene_description/urdf/o2ac_environment.xacro (robot description, xacro)
@@ -43,5 +43,5 @@
   <xacro:include filename="$(find o2ac_scene_description)/urdf/components/tray.xacro" />
   <xacro:tray trayname="tray" parent="workspace_center">
-    <origin xyz="0.2 -0.2 0" rpy="0 0 0" />
+    <origin xyz="0.05 -0.2 0" rpy="0 0 0" />
   </xacro:tray>
 </robot>

Commit message: Fix feeder screw picking

File: catkin_ws/src/o2ac_scene_description/urdf/o2ac_environment.xacro (robot description, xacro)
@@ -21,14 +21,10 @@
   <!-- Add screw feeders -->
   <xacro:include filename="$(find o2ac_scene_description)/urdf/components/screw_feeder.xacro" />
+  <xacro:screw_feeder feedername="m3_feeder" parent="workspace_center">
+    <origin xyz="-.511 -.13 -0.023" rpy="0 0 0" />
+  </xacro:screw_feeder>
   <xacro:screw_feeder feedername="m4_feeder" parent="workspace_center">
-    <origin xyz="-.511 -.13 -0.043" rpy="0 0 0" />
-    <!-- <origin xyz="-.55 .05 -0.043" rpy="0 0 0" />    -->
+    <origin xyz="-.512 0 -0.023" rpy="0 0 0" />
   </xacro:screw_feeder>
-  <!-- -0.016241; 0.18032; -0.039283 -->
-  <xacro:screw_feeder feedername="m3_feeder" parent="workspace_center">
-    <origin xyz="-.512 0 -0.043" rpy="0 0 0" />
-    <!-- <origin xyz="-.55 -.15 -0.043" rpy="0 0 0" />    -->
-  </xacro:screw_feeder>
-  <!-- -0.018032; -0.15035; -0.038212 -->
   <!-- Base fixture -->
   <xacro:include filename="$(find o2ac_scene_description)/urdf/components/base_fixture.xacro" />

Commit message: Add TV to scene, remove nut holders

File: catkin_ws/src/o2ac_scene_description/urdf/o2ac_environment.xacro (robot description, xacro)
@@ -47,5 +47,5 @@
   </xacro:jig_v_slope>  -->
   <!-- ======== -->
-  <xacro:include filename="$(find o2ac_scene_description)/urdf/components/nut_holder.xacro" />
+  <!-- <xacro:include filename="$(find o2ac_scene_description)/urdf/components/nut_holder.xacro" />
   <xacro:nut_holder partname="nut_holder" parent="a_bot_base_smfl">
     <origin xyz="0 .6 0.02" rpy="0 0 0" />
@@ -57,4 +57,41 @@
   <xacro:nut_holder partname="calibration_cone" parent="workspace_center">
     <origin xyz="${-0.365+0.01} ${0.345+.03} ${0.022-0.0465}" rpy="0 0 0" />
-  </xacro:nut_holder>
+  </xacro:nut_holder>   -->
+  <!-- ======== -->
+  <!-- TV -->
+  <link name="tv">
+    <!-- This tv box origin is at the front bottom, so it can more easily be measured  -->
+    <xacro:property name="tv_length_x" value="0.06"/>
+    <xacro:property name="tv_length_y" value="0.96"/>
+    <xacro:property name="tv_length_z" value="0.56"/>
+    <visual>
+      <origin xyz="${-tv_length_x/2} 0.0 ${tv_length_z/2}" rpy="0 0 0"/>
+      <geometry>
+        <box size="${tv_length_x} ${tv_length_y} ${tv_length_z}"/>
+      </geometry>
+      <material name="Black">
+        <color rgba="0.1 0.1 0.1 1.0"/>
+      </material>
+    </visual>
+    <collision>
+      <origin xyz="${-tv_length_x/2} 0.0 ${tv_length_z/2}" rpy="0 0 0"/>
+      <geometry>
+        <!-- 7.5 cm on each side -->
+        <box size="${tv_length_x + 0.15} ${tv_length_y + 0.15} ${tv_length_z+0.1}"/>
+      </geometry>
+    </collision>
+    <!-- This is required for Gazebo. -->
+    <inertial>
+      <mass value="1.0" />
+      <inertia ixx="0.0" ixy="0.0" ixz="0.0" iyy="0.0" iyz="0.0" izz="0.0" />
+    </inertial>
+  </link>
+  <gazebo reference="tv">
+    <material>Gazebo/Black</material>
+  </gazebo>
+  <joint name="tv_joint" type="fixed">
+    <parent link="o2ac_ground" />
+    <child link = "tv" />
+    <origin xyz="-0.4 0.0 1.58" rpy="0 0 0" />
+  </joint>
 </robot>

Commit message: Fix screw feeder position

File: catkin_ws/src/o2ac_scene_description/urdf/o2ac_environment.xacro (robot description, xacro)
@@ -25,5 +25,5 @@
   </xacro:screw_feeder>
   <xacro:screw_feeder feedername="m4_feeder" parent="workspace_center">
-    <origin xyz="-.511 .005 -0.023" rpy="0 0 0" />
+    <origin xyz="-.513 .004 -0.023" rpy="0 0 0" />
   </xacro:screw_feeder>
   <!-- Base fixture -->

Commit message: Minor changes

File: catkin_ws/src/o2ac_scene_description/urdf/o2ac_environment.xacro (robot description, xacro)
@@ -22,8 +22,8 @@
   <xacro:include filename="$(find o2ac_scene_description)/urdf/components/screw_feeder.xacro" />
   <xacro:screw_feeder feedername="m3_feeder" parent="workspace_center">
-    <origin xyz="-.513 -.152 -0.023" rpy="0 0 0" />
+    <origin xyz="-.512 -.152 -0.023" rpy="0 0 0" />
   </xacro:screw_feeder>
   <xacro:screw_feeder feedername="m4_feeder" parent="workspace_center">
-    <origin xyz="-.513 .006 -0.023" rpy="0 0 0" />
+    <origin xyz="-.512 .006 -0.023" rpy="0 0 0" />
   </xacro:screw_feeder>
   <!-- Base fixture -->

Commit message: Clean up

File: catkin_ws/src/o2ac_scene_description/urdf/o2ac_environment.xacro (robot description, xacro)
@@ -22,5 +22,5 @@
   <xacro:include filename="$(find o2ac_scene_description)/urdf/components/screw_feeder.xacro" />
   <xacro:screw_feeder feedername="m3_feeder" parent="workspace_center">
-    <origin xyz="-.514 -.151 -0.023" rpy="0 0 0" />
+    <origin xyz="-.512 -.1525 -0.023" rpy="0 0 0" />
   </xacro:screw_feeder>
   <xacro:screw_feeder feedername="m4_feeder" parent="workspace_center">

Commit message: Add simple holder to scene

File: catkin_ws/src/o2ac_scene_description/urdf/o2ac_environment.xacro (robot description, xacro)
@@ -46,4 +46,8 @@
     <origin xyz="-0.2927 0.17214 0.0" rpy="0 0 0" />
   </xacro:vgroove_aid>
+  <xacro:include filename="$(find o2ac_scene_description)/urdf/components/simple_holder.xacro" />
+  <xacro:simple_holder partname="simple_holder" parent="workspace_center">
+    <origin xyz="0.27 -0.6 -0.0149" rpy="0 0 0" />
+  </xacro:simple_holder>
   <!-- ======== -->
   <!-- <xacro:include filename="$(find o2ac_scene_description)/urdf/components/nut_holder.xacro" />

Commit message: WIP: Add orientation of shaft's end cap sequence

File: catkin_ws/src/o2ac_scene_description/urdf/o2ac_environment.xacro (robot description, xacro)
@@ -48,5 +48,5 @@
   <xacro:include filename="$(find o2ac_scene_description)/urdf/components/simple_holder.xacro" />
   <xacro:simple_holder partname="simple_holder" parent="workspace_center">
-    <origin xyz="0.27 -0.6 -0.0149" rpy="0 0 0" />
+    <origin xyz="0.257 -0.607 -0.0149" rpy="0 0 0" />
   </xacro:simple_holder>
   <!-- ======== -->

Commit message: Add frame for centering

File: catkin_ws/src/o2ac_scene_description/urdf/o2ac_environment.xacro (robot description, xacro)
@@ -50,4 +50,10 @@
     <origin xyz="0.257 -0.607 -0.0149" rpy="0 0 0" />
   </xacro:simple_holder>
+  <joint name="right_centering_joint" type="fixed">
+    <parent link="workspace_center"/>
+    <child link="right_centering_link"/>
+    <origin xyz="0.20 0.30 -0.0149" rpy="0 ${pi/2} -${pi/2}" />
+  </joint>
+  <link name="right_centering_link"/>
   <!-- ======== -->
   <!-- <xacro:include filename="$(find o2ac_scene_description)/urdf/components/nut_holder.xacro" />

Commit message: WIP: Add subtask e

File: catkin_ws/src/o2ac_scene_description/urdf/o2ac_environment.xacro (robot description, xacro)
@@ -56,4 +56,10 @@
   </joint>
   <link name="right_centering_link"/>
+  <joint name="left_centering_joint" type="fixed">
+    <parent link="workspace_center"/>
+    <child link="left_centering_link"/>
+    <origin xyz="0.20 -0.30 -0.0149" rpy="0 ${pi/2} -${pi/2}" />
+  </joint>
+  <link name="left_centering_link"/>
   <!-- ======== -->
   <!-- <xacro:include filename="$(find o2ac_scene_description)/urdf/components/nut_holder.xacro" />

Commit message: Cleanup, add test log

File: catkin_ws/src/o2ac_scene_description/urdf/o2ac_environment.xacro (robot description, xacro)
@@ -49,4 +49,8 @@
   <xacro:vgroove_aid jigname="vgroove_aid" parent="b_bot_base_link">
     <origin xyz="-0.2927 0.17214 0.0" rpy="0 0 0" />
+  </xacro:vgroove_aid>
+  <!-- The second vgroove at the back (for the motor)-->
+  <xacro:vgroove_aid jigname="vgroove_aid_motor" parent="b_bot_base_link">
+    <origin xyz="-0.225 -0.210 0.0" rpy="0 0 0" />
   </xacro:vgroove_aid>
   <xacro:include filename="$(find o2ac_scene_description)/urdf/components/simple_holder.xacro" />

Commit message: Add saved plans to taskboard tasks

File: catkin_ws/src/o2ac_scene_description/urdf/o2ac_environment.xacro (robot description, xacro)
@@ -52,5 +52,5 @@
   <!-- The second vgroove at the back (for the motor)-->
   <xacro:vgroove_aid jigname="vgroove_aid_motor" parent="b_bot_base_link">
-    <origin xyz="-0.225 -0.210 0.0" rpy="0 0 0" />
+    <origin xyz="-0.225 -0.210 0.001" rpy="0 0 0" />
   </xacro:vgroove_aid>
   <xacro:include filename="$(find o2ac_scene_description)/urdf/components/simple_holder.xacro" />

Commit message: Update pose of vgroove aid

File: catkin_ws/src/o2ac_scene_description/urdf/o2ac_environment.xacro (robot description, xacro)
@@ -48,5 +48,5 @@
   <xacro:include filename="$(find o2ac_scene_description)/urdf/components/vgroove_aid.xacro" />
   <xacro:vgroove_aid jigname="vgroove_aid" parent="b_bot_base_link">
-    <origin xyz="-0.2927 0.17214 0.0" rpy="0 0 ${pi/2}" />
+    <origin xyz="-0.2957 0.169 0.0" rpy="0 0 ${pi/2}" />
   </xacro:vgroove_aid>
   <!-- The second vgroove at the back (for the motor)-->

Commit message: Update tools and screw feeder

File: catkin_ws/src/o2ac_scene_description/urdf/o2ac_environment.xacro (robot description, xacro)
@@ -39,8 +39,8 @@
   <xacro:include filename="$(find o2ac_scene_description)/urdf/components/screw_feeder.xacro" />
   <xacro:screw_feeder feedername="m3_feeder" parent="workspace_center" with_collision_geometry="false">
-    <origin xyz="-.512 -.1525 -0.023" rpy="0 0 0" />
+    <origin xyz="-.511 -.154 0.028" rpy="0 0 0" />
   </xacro:screw_feeder>
   <xacro:screw_feeder feedername="m4_feeder" parent="workspace_center" with_collision_geometry="false">
-    <origin xyz="-.514 .004 -0.023" rpy="0 0 0" />
+    <origin xyz="-.514 .0035 0.03" rpy="0 0 0" />
   </xacro:screw_feeder>
   <!-- Base fixture -->

Commit message: Add orchestrated assembly sequence

File: catkin_ws/src/o2ac_scene_description/urdf/o2ac_environment.xacro (robot description, xacro)
@@ -75,4 +75,10 @@
     <origin xyz="0.257 -0.607 -0.0149" rpy="0 0 0" />
   </xacro:simple_holder>
+  <joint name="right_storage_area_joint" type="fixed">
+    <parent link="workspace_center"/>
+    <child link="right_storage_area_link"/>
+    <origin xyz="0.25 0.50 -0.0149" rpy="0 ${pi/2} -${pi/2}" />
+  </joint>
+  <link name="right_storage_area_link"/>
   <joint name="right_centering_joint" type="fixed">
     <parent link="workspace_center"/>

Commit message: WIP: Add subtask e

File: catkin_ws/src/o2ac_scene_description/urdf/o2ac_environment.xacro (robot description, xacro)
@@ -93,4 +93,20 @@
   </joint>
   <link name="left_centering_link"/>
+  <xacro:include filename="$(find o2ac_scene_description)/urdf/components/washer_holder.xacro" />
+  <xacro:washer_holder partname="washer_holder1" parent="workspace_center">
+    <origin xyz="0 -0.14 0.001" rpy="0 0 0" />
+  </xacro:washer_holder>
+  <xacro:include filename="$(find o2ac_scene_description)/urdf/components/washer_holder.xacro" />
+  <xacro:washer_holder partname="washer_holder2" parent="workspace_center">
+    <origin xyz="0 -0.05 0.001" rpy="0 0 0" />
+  </xacro:washer_holder>
+  <xacro:include filename="$(find o2ac_scene_description)/urdf/components/washer_holder.xacro" />
+  <xacro:washer_holder partname="washer_holder3" parent="workspace_center">
+    <origin xyz="0.325 -0.6 -0.045" rpy="0 ${pi/2} 0" />
+  </xacro:washer_holder>
+  <xacro:include filename="$(find o2ac_scene_description)/urdf/components/washer_holder.xacro" />
+  <xacro:washer_holder partname="washer_holder4" parent="workspace_center">
+    <origin xyz="0.325 -0.5 -0.045" rpy="0 ${pi/2} 0" />
+  </xacro:washer_holder>
   <!-- ======== -->
   <!-- <xacro:include filename="$(find o2ac_scene_description)/urdf/components/nut_holder.xacro" />
@@ -98,8 +114,4 @@
     <origin xyz="0 .6 0.02" rpy="0 0 0" />
   </xacro:nut_holder>
-  <xacro:include filename="$(find o2ac_scene_description)/urdf/components/washer_holder.xacro" />
-  <xacro:washer_holder partname="washer_holder" parent="a_bot_base_smfl">
-    <origin xyz="0 .54 0.02" rpy="0 0 0" />
-  </xacro:washer_holder>
   <xacro:nut_holder partname="calibration_cone" parent="workspace_center">
     <origin xyz="${-0.365+0.01} ${0.345+.03} ${0.022-0.0465}" rpy="0 0 0" />

Commit message: More finetuning

File: catkin_ws/src/o2ac_scene_description/urdf/o2ac_environment.xacro (robot description, xacro)
@@ -39,5 +39,5 @@
   <xacro:include filename="$(find o2ac_scene_description)/urdf/components/screw_feeder.xacro" />
   <xacro:screw_feeder feedername="m3_feeder" parent="workspace_center" with_collision_geometry="false">
-    <origin xyz="-.512 -.155 0.015" rpy="0 0 0" />
+    <origin xyz="-.5115 -.156 0.015" rpy="0 0 0" />
   </xacro:screw_feeder>
   <xacro:screw_feeder feedername="m4_feeder" parent="workspace_center" with_collision_geometry="false">
