Commit message: Update vision actions, cameras, documentation

File: catkin_ws/src/o2ac_scene_description/urdf/base_scene.urdf.xacro (robot description, xacro)
@@ -5,6 +5,5 @@
   <!-- Calibration parameters -->
   <xacro:property name="a_bot_x" value="-0.0"/>
-  <xacro:property name="a_bot_y" value="-0.445"/>
-  <xacro:property name="a_bot_y_base_offset" value="-0.08"/>   <!-- Moves the robot around on its plate -->
+  <xacro:property name="a_bot_y" value="-0.525"/>
   <xacro:property name="a_bot_theta" value="0.0"/>
   <xacro:property name="b_bot_x" value="-0.0"/>
@@ -23,6 +22,6 @@
   <xacro:include filename="$(find o2ac_scene_description)/urdf/o2ac_environment.xacro" />
   <!-- <xacro:include filename="$(find flexwrist_experiment)/urdf/2020-01-experiment-scene.xacro" /> -->
-  <xacro:include filename="$(find o2ac_scene_description)/urdf/taskboard_scene.xacro" />
-  <!-- <xacro:include filename="$(find o2ac_scene_description)/urdf/assembly_scene.xacro" /> -->
+  <!-- <xacro:include filename="$(find o2ac_scene_description)/urdf/taskboard_scene.xacro" /> -->
+  <xacro:include filename="$(find o2ac_scene_description)/urdf/assembly_scene.xacro" />
   <!-- Robot bases -->
   <!-- Putting these at height 0.0 makes them intersect with the ground, so they are elevated. -->
@@ -30,5 +29,5 @@
   <xacro:include filename="$(find o2ac_scene_description)/urdf/components/o2ac_base.xacro" />
   <xacro:o2ac_base boxname="a_bot_base_smfl" parent="o2ac_ground">
-    <origin xyz="${a_bot_x-.65/2} ${a_bot_y+a_bot_y_base_offset-.65/2} ${bots_z-.05}" rpy="0 0 0" />
+    <origin xyz="${a_bot_x-.65/2} ${a_bot_y-.65/2} ${bots_z-.05}" rpy="0 0 0" />
   </xacro:o2ac_base>
   <xacro:o2ac_base boxname="b_bot_base_smfl" parent="o2ac_ground">
@@ -50,13 +49,4 @@
     <origin xyz="0.0 0.0 ${bots_z-robot_mount_plate+workplate_h}" rpy="0.0 0.0 0.0" />
   </joint>
-  <!-- robot arms -->
-  <!-- <xacro:panda_arm arm_id="panda" />
-  <xacro:hand ns="panda" rpy="0 0 ${-pi/4}" connected_to="panda_link8"/>
-  <joint name="panda_tip_joint" type="fixed">
-    <parent link="panda_link8"/>
-    <child link="panda_tip"/>
-    <origin rpy="0.0 -1.5708 -0.7854" xyz="0.0 0.0 .11 "/>
-  </joint>
-  <link name="panda_tip"/> -->
   <xacro:ur5e_robot prefix="a_bot_" joint_limited="true"
     shoulder_pan_lower_limit="${-pi}" shoulder_pan_upper_limit="${pi}"
@@ -94,6 +84,6 @@
   <xacro:include filename="$(find o2ac_scene_description)/urdf/components/o2ac_end_effector.urdf.xacro" />
   <xacro:o2ac_end_effector prefix="a_bot_" use_soft_wrist="false" use_cameras="true" parent = "a_bot_ee_link" />
-  <xacro:include filename="$(find o2ac_scene_description)/urdf/components/o2ac_end_effector.urdf.xacro" />
-  <xacro:o2ac_end_effector prefix="b_bot_" use_soft_wrist="false" use_cameras="true" parent = "b_bot_ee_link" />
+  <xacro:include filename="$(find o2ac_scene_description)/urdf/components/o2ac_end_effector_old.urdf.xacro" />
+  <xacro:o2ac_end_effector_old prefix="b_bot_" use_soft_wrist="false" use_cameras="true" parent = "b_bot_ee_link" />
   <!-- Add cameras -->
   <!-- <xacro:include filename="$(find o2ac_scene_description)/urdf/components/_d435.urdf.xacro" />

File: catkin_ws/src/o2ac_scene_description/urdf/components/o2ac_end_effector.urdf.xacro (robot description, xacro)
@@ -4,18 +4,22 @@
 <robot name="robotiq_85_gripper_o2ac" xmlns:xacro="http://www.ros.org/wiki/xacro">
   <xacro:macro name="o2ac_end_effector" params="prefix use_soft_wrist:=false use_cameras:=false parent">
-    <xacro:if value="${use_soft_wrist}">
-      <xacro:include filename="$(find o2ac_scene_description)/urdf/components/robotiq_85_gripper_with_soft_wrist.urdf.xacro" />
-      <xacro:robotiq_85_gripper_with_soft_wrist prefix="${prefix}" parent="${parent}"/>
-    </xacro:if>
-    <xacro:if value="${not use_soft_wrist}">
-      <xacro:include filename="$(find o2ac_scene_description)/urdf/components/robotiq_85_gripper_with_ft300.urdf.xacro" />
-      <xacro:robotiq_85_gripper_with_ft300 prefix="${prefix}" parent="${parent}"/>
-    </xacro:if>
+    <xacro:include filename="$(find robotiq_description)/urdf/robotiq_85_gripper.urdf.xacro"/>
+    <xacro:robotiq_85_gripper prefix="${prefix}" parent="${parent}">
+        <origin rpy="0.0 0.0 0.0" xyz="0 0 0"/>
+    </xacro:robotiq_85_gripper>
     <xacro:if value="${use_cameras}">
       <xacro:include filename="$(find o2ac_scene_description)/urdf/components/wrist_cameras.xacro" />
       <xacro:wrist_cameras prefix="${prefix}" parent="${prefix}robotiq_85_base_link"/>
     </xacro:if>
+    <!-- Add an additional link to plan with. Oriented like the UR ee_link frame. -->
+    <joint name="${prefix}robotiq_85_tip_link_joint" type="fixed">
+      <parent link="${prefix}robotiq_85_base_link"/>
+      <child link="${prefix}robotiq_85_tip_link"/>
+      <!-- <origin rpy="0.0 0.0 0.0" xyz=".163 0.0 0.0"/> -->
+      <origin rpy="0.0 0.0 0.0" xyz="${.163+.083} 0.0 0.0"/>
+    </joint>
+    <link name="${prefix}robotiq_85_tip_link"/>
     <!-- ========= -->
-    <!-- Screw tool tip frames. X-axis points along the screw into the hole. -->
+    <!-- Add screw tool tip frames. X-axis points along the screw into the hole. -->
     <!-- Offset of the gripper tooltips -->
     <joint name="${prefix}tool_intermediate_joint" type="fixed">

File: catkin_ws/src/o2ac_scene_description/urdf/components/wrist_cameras.xacro (robot description, xacro)
@@ -34,20 +34,20 @@
       <origin xyz="0.035 0.0 0.025" rpy="0 0 0"/>
     </joint>
-    <link name="${prefix}cam_1_link" />
-    <joint name="${prefix}cam_1_joint" type="fixed">
+    <link name="${prefix}inside_cam_link" />
+    <joint name="${prefix}inside_cam_joint" type="fixed">
       <parent link="${parent}" />
-      <child link="${prefix}cam_1_link" />
+      <child link="${prefix}inside_cam_link" />
       <origin xyz="0.026 0 0.0595" rpy="0 ${20.0*pi/180.0} 0" />
     </joint>
-    <xacro:sensor_sr305 prefix="${prefix}_cam_1_" parent="${prefix}cam_1_link">
+    <xacro:sensor_sr305 prefix="${prefix}inside_cam_" parent="${prefix}inside_cam_link">
       <origin xyz="0 0 0" rpy="0 0 0"/>
     </xacro:sensor_sr305>
-    <link name="${prefix}cam_2_link" />
-    <joint name="${prefix}cam_2_joint" type="fixed">
+    <link name="${prefix}outside_cam_link" />
+    <joint name="${prefix}outside_cam_joint" type="fixed">
       <parent link="${parent}" />
-      <child link="${prefix}cam_2_link" />
+      <child link="${prefix}outside_cam_link" />
       <origin xyz="0.026 0 ${0.0595+.024}" rpy="0 ${-15.0*pi/180.0} 0" />
     </joint>
-    <xacro:sensor_sr305 prefix="${prefix}_cam_2_" parent="${prefix}cam_2_link">
+    <xacro:sensor_sr305 prefix="${prefix}outside_cam_" parent="${prefix}outside_cam_link">
       <origin xyz="0 0 0" rpy="0 0 0"/>
     </xacro:sensor_sr305>

File: catkin_ws/src/o2ac_scene_description/urdf/o2ac_environment.xacro (robot description, xacro)
@@ -41,3 +41,14 @@
     <origin xyz="0.05 -0.2 0" rpy="0 0 0" />
   </xacro:tray>
+  <!-- <link name="scene_cam_holder_link" />
+  <joint name="scene_cam_holder_joint" type="fixed">
+    <parent link="workspace_center" />
+    <child link="scene_cam_holder_link" />
+    <origin xyz="-0.265 0.03 0.115" rpy="0 0 ${pi/2}" />
+  </joint>
+  <xacro:include filename="$(find realsense2_description)/urdf/_d435.urdf.xacro" />
+  <xacro:arg name="use_nominal_extrinsics" default="True" />
+  <xacro:sensor_d435 parent="scene_cam_holder_link" name="scene_cam">
+    <origin xyz="0 0 0" rpy="0 0 0"/>
+  </xacro:sensor_d435> -->
 </robot>
