Commit message: Add holders, update tools, models etc.

File: catkin_ws/src/o2ac_scene_description/urdf/base_scene.urdf.xacro (robot description, xacro)
@@ -15,8 +15,5 @@
   <xacro:include filename="$(find o2ac_gazebo)/urdf/o2ac_base_scene.gazebo" />
   <!-- robots -->
-  <xacro:include filename="$(find ur_description)/urdf/ur5.urdf.xacro" />
   <xacro:include filename="$(find ur_e_description)/urdf/ur5e.urdf.xacro" />
-  <!-- <xacro:include filename="$(find franka_description)/robots/panda_arm.xacro"/>
-  <xacro:include filename="$(find franka_description)/robots/hand.xacro"/> -->
   <!-- Scene items (trays, columns, tools, jigs, feeders...) -->
   <xacro:include filename="$(find o2ac_scene_description)/urdf/o2ac_environment.xacro" />
@@ -54,5 +51,5 @@
     elbow_joint_lower_limit="0.0" elbow_joint_upper_limit="${pi}"
     wrist_1_lower_limit="${-pi}" wrist_1_upper_limit="${pi}"
-    wrist_2_lower_limit="${-pi}" wrist_2_upper_limit="${pi}"
+    wrist_2_lower_limit="${-pi*1.5}" wrist_2_upper_limit="${pi*1.5}"
     wrist_3_lower_limit="${-pi}" wrist_3_upper_limit="${pi}"
     transmission_hw_interface="hardware_interface/PositionJointInterface"
@@ -61,11 +58,14 @@
     kinematics_file="${load_yaml('$(find o2ac_scene_description)/config/a_bot_calibration.yaml')}"
   />
-  <xacro:ur5_robot prefix="b_bot_" joint_limited="true"
+  <xacro:ur5e_robot prefix="b_bot_" joint_limited="true"
     shoulder_pan_lower_limit="${-pi}" shoulder_pan_upper_limit="${pi}"
     shoulder_lift_lower_limit="${-pi}" shoulder_lift_upper_limit="${pi}"
     elbow_joint_lower_limit="0.0" elbow_joint_upper_limit="${pi}"
     wrist_1_lower_limit="${-pi}" wrist_1_upper_limit="${pi}"
-    wrist_2_lower_limit="${-pi}" wrist_2_upper_limit="${pi}"
+    wrist_2_lower_limit="${-pi*1.5}" wrist_2_upper_limit="${pi*1.5}"
     wrist_3_lower_limit="${-pi}" wrist_3_upper_limit="${pi}"
+    transmission_hw_interface="hardware_interface/PositionJointInterface"
+    safety_limits="false" safety_pos_margin="0.15"
+    safety_k_position="20"
     kinematics_file="${load_yaml('$(find o2ac_scene_description)/config/b_bot_calibration.yaml')}"
   />
@@ -81,20 +81,9 @@
     <origin xyz="${b_bot_x} ${b_bot_y} ${bots_z}" rpy="0.0 0.0 ${b_bot_theta}" />
   </joint>
-  <!-- spawn and attach robotiq 85 gripper (+ FT300 sensor, soft wrist...) -->
+  <!-- Spawn and attach robotiq 85 gripper (+ cameras) -->
+  <xacro:include filename="$(find o2ac_scene_description)/urdf/components/o2ac_end_effector_2F-140.urdf.xacro" />
+  <xacro:o2ac_end_effector prefix="a_bot_" use_soft_wrist="false" use_cameras="true" parent = "a_bot_ee_link" />
   <xacro:include filename="$(find o2ac_scene_description)/urdf/components/o2ac_end_effector.urdf.xacro" />
-  <xacro:o2ac_end_effector prefix="a_bot_" use_soft_wrist="false" use_cameras="true" parent = "a_bot_ee_link" />
-  <xacro:include filename="$(find o2ac_scene_description)/urdf/components/o2ac_end_effector_old.urdf.xacro" />
-  <xacro:o2ac_end_effector_old prefix="b_bot_" use_soft_wrist="false" use_cameras="true" parent = "b_bot_ee_link" />
-  <!-- Add cameras -->
-  <!-- <xacro:include filename="$(find o2ac_scene_description)/urdf/components/_d435.urdf.xacro" />
-  <link name="scene_cam_holder_link" />
-  <joint name="scene_cam_holder_joint" type="fixed">
-    <parent link="workspace_center" />
-    <child  link="scene_cam_holder_link" />
-    <origin xyz="-0.0179662 -0.155013 0.101615" rpy="0.0281409 -0.137996 -0.0954644" />
-  </joint>
-  <xacro:sensor_d435 prefix="scene_" parent="scene_cam_holder_link">
-    <origin xyz="0 0 0" rpy="0 0 0"/>
-  </xacro:sensor_d435> -->
+  <xacro:o2ac_end_effector prefix="b_bot_" use_soft_wrist="false" use_cameras="true" parent = "b_bot_ee_link" />
   <!-- The "world" link definition should be removed, but apparently it is necessary for Gazebo -->
   <link name="world" />

File: catkin_ws/src/o2ac_scene_description/urdf/components/base_fixture.xacro (robot description, xacro)
@@ -6,5 +6,5 @@
   <xacro:property name="long_bar_mesh" value="package://o2ac_scene_description/meshes/HFSP5-2080-320.stl" />
   <xacro:property name="length" value=".32" />
-  <xacro:property name="width" value=".2" />
+  <xacro:property name="width" value=".24" />
   <link name="base_fixture_top">
     <visual>
@@ -18,8 +18,21 @@
     </visual>
     <collision>
-      <origin rpy="0 0 0" xyz="${width/2} ${length/2} 0.095"/>
+      <origin rpy="0 0 0" xyz="${width/2} ${length/2} ${.08+.005/2}"/>
       <geometry>
-        <box size="${width} ${length} 0.03"/>
-        <!-- <mesh filename="${top_mesh}" scale=".001 .001 .001"/> -->
+        <box size="${width} ${length} 0.005"/>
+      </geometry>
+    </collision>
+    <!-- The long stopper bar -->
+    <collision>
+      <origin rpy="0 0 0" xyz="${width-.02/2} ${length-.20/2} ${.08+.03/2}"/>
+      <geometry>
+        <box size="${.02} ${.20} 0.03"/>
+      </geometry>
+    </collision>
+    <!-- The short stopper bar -->
+    <collision>
+      <origin rpy="0 0 0" xyz="${width-.16/2} ${length-.02/2} ${.08+.03/2}"/>
+      <geometry>
+        <box size="${.16} ${.02} 0.03"/>
       </geometry>
     </collision>
@@ -35,5 +48,4 @@
       <geometry>
         <box size=".02 ${length} .08"/>
-        <!-- <mesh filename="${long_bar_mesh}" scale=".001 .001 .001"/> -->
       </geometry>
       <material name="grey">

File: catkin_ws/src/o2ac_scene_description/urdf/components/o2ac_end_effector.urdf.xacro (robot description, xacro)
@@ -6,6 +6,28 @@
     <xacro:include filename="$(find robotiq_description)/urdf/robotiq_85_gripper.urdf.xacro"/>
     <xacro:robotiq_85_gripper prefix="${prefix}" parent="${parent}">
-        <origin rpy="0.0 0.0 0.0" xyz="0 0 0"/>
+        <origin rpy="0.0 0.0 0.0" xyz="0.01 0 0"/> <!-- This 0.01 offset is the Robotiq/UR coupling -->
     </xacro:robotiq_85_gripper>
+    <link name="${prefix}_coupling">
+      <visual>
+        <origin rpy="0 ${pi/2} 0" xyz=".005 0 0"/>
+        <geometry>
+          <cylinder length="0.01" radius="0.0375"/>
+        </geometry>
+        <material name="black">
+        <color rgba=".1 .1 .1 1"/>
+      </material>
+      </visual>
+      <collision>
+        <origin rpy="0 ${pi/2} 0" xyz=".005 0 0"/>
+        <geometry>
+          <cylinder length="0.01" radius="0.0375"/>
+        </geometry>
+      </collision>
+    </link>
+    <joint name="${prefix}_coupling_joint" type="fixed">
+      <parent link="${parent}" />
+      <child link = "${prefix}_coupling" />
+      <origin rpy="0 0 0" xyz="0 0 0"/>
+    </joint>
     <xacro:if value="${use_cameras}">
       <xacro:include filename="$(find o2ac_scene_description)/urdf/components/wrist_cameras.xacro" />
@@ -16,6 +38,5 @@
       <parent link="${prefix}robotiq_85_base_link"/>
       <child link="${prefix}robotiq_85_tip_link"/>
-      <!-- <origin rpy="0.0 0.0 0.0" xyz=".163 0.0 0.0"/> -->
-      <origin rpy="0.0 0.0 0.0" xyz="${.163+.083} 0.0 0.0"/>
+      <origin rpy="0.0 0.0 0.0" xyz=".163 0.0 0.0"/>
     </joint>
     <link name="${prefix}robotiq_85_tip_link"/>
@@ -29,10 +50,4 @@
     </joint>
     <link name="${prefix}tool_intermediate_link"/>
-    <joint name="${prefix}robotiq_85_screw_tool_m6_tip_joint" type="fixed">
-      <parent link="${prefix}tool_intermediate_link"/>
-      <child link="${prefix}screw_tool_m6_tip_link"/>
-      <origin rpy="0.0 ${pi/2} 0.0" xyz="0.0 0.0 -0.135 "/>
-    </joint>
-    <link name="${prefix}screw_tool_m6_tip_link"/>
     <joint name="${prefix}robotiq_85_nut_tool_m6_tip_joint" type="fixed">
       <parent link="${prefix}tool_intermediate_link"/>
@@ -54,15 +69,9 @@
     <link name="${prefix}screw_tool_m3_tip_link"/>
     <joint name="${prefix}robotiq_85_set_screw_tool_tip_joint" type="fixed">
-      <parent link="${prefix}tool_intermediate_link"/>
+      <parent link="${prefix}robotiq_85_tip_link"/>
       <child link="${prefix}set_screw_tool_tip_link"/>
-      <origin rpy="0.0 ${pi/2} 0.0" xyz=".01 0.0 -0.085 "/>
+      <origin rpy="0.0 ${-pi/6} 0.0" xyz=".0045 0.0 0.047 "/>
     </joint>
     <link name="${prefix}set_screw_tool_tip_link"/>
-    <joint name="${prefix}robotiq_85_suction_tool_tip_joint" type="fixed">
-      <parent link="${prefix}tool_intermediate_link"/>
-      <child link="${prefix}suction_tool_tip_link"/>
-      <origin rpy="0.0 ${pi/2} 0.0" xyz=".02 0.0 -0.131 "/>
-    </joint>
-    <link name="${prefix}suction_tool_tip_link"/>
     <joint name="${prefix}dual_suction_gripper_pad_joint" type="fixed">
       <parent link="${prefix}tool_intermediate_link"/>

File: catkin_ws/src/o2ac_scene_description/urdf/components/tools.xacro (robot description, xacro)
@@ -1,65 +1,16 @@
+<?xml version="1.0"?>
+<robot xmlns:xacro="http://www.ros.org/wiki/xacro">
 <!-- This holder has a size of about 155 mm x 40 mm x 26 mm -->
 <!-- The Bit cushion has a height of 30.5 mm, starts about 24 mm from the top-->
 <!-- The gripper center would be about 44 mm from the top, so the tip might be 111 mm further down -->
 <!-- The tip\axis seems to be 11.5 mm from the "front" side. The front side looks into the gripper -->
-<robot xmlns:xacro="http://www.ros.org/wiki/xacro">
-  <!-- Tools at the front of the robot -->
-  <joint name="belt_holder_to_environment_joint" type="fixed">
-    <parent link="b_bot_base" />
-    <child link="belt_tool_holder" />
-    <origin xyz=".325 -.2 .0" rpy="0 0 0" />
-  </joint>
-  <link name="belt_tool_holder">
-    <visual>
-      <origin rpy="${pi/2} 0 ${pi/2}" xyz="0 -.025 -.005"/>
-      <geometry>
-        <mesh filename="package://o2ac_scene_description/meshes/gravity_tool_holder.stl" scale="0.001 0.001 0.001"/>
-      </geometry>
-      <material name="grey">
-        <color rgba=".5 .5 .5 1"/>
-      </material>
-    </visual>
-    <collision>
-      <origin rpy="0 0 0" xyz="0 0 0"/>
-      <geometry>
-        <box size=".001 .001 .001"/>
-      </geometry>
-    </collision>
-  </link>
-  <link name="belt_tool_link">
-    <inertial>
-      <origin rpy="0 0 0" xyz="0 0 0"/>
-      <mass value="1.0"/>
-      <inertia ixx="1" ixy="0" ixz="0" iyy="1" iyz="0" izz="1"/>
-    </inertial>
-    <visual>
-      <origin rpy="0 0 ${-pi/2}" xyz="0.02 0 -0.017"/>
-      <geometry>
-        <mesh filename="package://o2ac_scene_description/meshes/belt_hook_tool.stl" scale="0.001 0.001 0.001"/>
-      </geometry>
-      <material name="white">
-        <color rgba=".9 .9 .9 1"/>
-      </material>
-    </visual>
-    <collision>
-      <origin rpy="0 0 0" xyz="0 0 0"/>
-      <geometry>
-        <box size=".026 .04 .055"/>
-      </geometry>
-    </collision>
-  </link>
-  <joint name="belt_tool_to_holder" type="fixed">
-    <parent link="belt_tool_holder" />
-    <child link="belt_tool_link" />
-    <origin xyz="0 0 0" rpy="0 0 0" />
-  </joint>
-  <!-- +++++++++++++++++++ -->
-  <!-- Tools at the back of the robot system -->
-  <joint name="screw_holder_to_environment_joint" type="fixed">
+  <!-- Tool holders at the back of the robot system -->
+  <!-- The long tool holder with 3 tools -->
+  <joint name="screw_tool_holder_long_to_environment_joint" type="fixed">
     <parent link="horizontal_column_for_tools" />
-    <child link="screw_tool_holder" />
+    <child link="screw_tool_holder_long" />
     <origin xyz=".04 .0 .04" rpy="0.0 0.0 ${-pi/2}" />
   </joint>
-  <link name="screw_tool_holder">
+  <link name="screw_tool_holder_long">
     <inertial>
       <origin rpy="0 0 0" xyz="0 0 0"/>
@@ -100,7 +51,55 @@
     </collision>
   </link>
+  <!-- ==== -->
+  <!-- The short tool holder with a single tool -->
+  <joint name="screw_holder_short_to_environment_joint" type="fixed">
+    <parent link="horizontal_column_for_tools" />
+    <child link="screw_tool_holder_short" />
+    <origin xyz=".04 .3 .04" rpy="0.0 0.0 ${-pi/2}" />
+  </joint>
+  <link name="screw_tool_holder_short">
+    <inertial>
+      <origin rpy="0 0 0" xyz="0 0 0"/>
+      <mass value="1.0"/>
+      <inertia ixx="1" ixy="0" ixz="0" iyy="1" iyz="0" izz="1"/>
+    </inertial>
+    <!-- The horizontal plate -->
+    <visual>
+      <origin rpy="0 0 0" xyz="-0.05 .0013 0.002"/>
+      <geometry>
+        <box size=".1 .066 .004"/>
+      </geometry>
+      <material name="whitish">
+        <color rgba=".7 .7 .7 1"/>
+      </material>
+    </visual>
+    <collision>
+      <origin rpy="0 0 0" xyz="-0.05 .0013 0.002"/>
+      <geometry>
+        <box size=".1 .066 .004"/>
+      </geometry>
+    </collision>
+    <!-- The vertical plate -->
+    <visual>
+      <origin rpy="0 0 0" xyz="-0.05 -.014 0.0179"/>
+      <geometry>
+        <box size=".1 .004 .035"/>
+      </geometry>
+      <material name="grey">
+        <color rgba=".5 .5 .5 1"/>
+      </material>
+    </visual>
+    <collision>
+      <origin rpy="0 0 0" xyz="-0.05 -.014 0.0179"/>
+      <geometry>
+        <box size=".1 .004 .035"/>
+      </geometry>
+    </collision>
+  </link>
   <!-- ++++++++++++++++++++++++++++ -->
-  <!-- Screw tools -->
+  <!-- Screw tools on the holders in the back of the system -->
   <xacro:property name="bit_cushion_to_axis" value="0.0285"/>
+  <xacro:property name="back_plate_offset_long" value=".009"/>
+  <xacro:property name="back_plate_offset_short" value=".01"/>
   <xacro:property name="tool_offset" value="${-.005 + bit_cushion_to_axis}" />
   <!-- The collision boxes of the tools only include the top part (not what is hanging underneath the holder) -->
@@ -111,8 +110,63 @@
       <inertia ixx="1" ixy="0" ixz="0" iyy="1" iyz="0" izz="1"/>
     </inertial>
-    <!-- <visual>
-      <origin rpy="0 0 0" xyz="0 0 0"/>
-      <geometry>
-        <mesh filename="package://o2ac_scene_description/meshes/nut_tool_m6_BC5-XL320-LG20-R_v2.stl" scale="0.001 0.001 0.001"/>
+    <visual>
+      <origin rpy="0 0 0" xyz="0 0 ${.052/2}"/>
+      <geometry>
+        <box size=".026 .059 .052"/>
+      </geometry>
+      <material name="yellowish">
+        <color rgba=".9 .9 .7 1"/>
+      </material>
+    </visual>
+    <collision>
+      <origin rpy="0 0 0" xyz="0 0 ${.052/2}"/>
+      <geometry>
+        <box size=".026 .059 .052"/>
+      </geometry>
+    </collision>
+  </link>
+  <joint name="nut_tool_m6_to_holder" type="fixed">
+    <parent link="screw_tool_holder_long" />
+    <child link="nut_tool_m6_link" />
+    <origin xyz="-0.05 ${-back_plate_offset_long + .059/2 + .0155} 0.004" rpy="0.0 0.0 0.0" />
+    <!-- .0155 is the distance from the center of the box to the axis of the tool -->
+  </joint>
+  <link name="set_screw_tool_link">
+    <inertial>
+      <origin rpy="0 0 0" xyz="0 0 0"/>`
+      <mass value="1.0"/>
+      <inertia ixx="1" ixy="0" ixz="0" iyy="1" iyz="0" izz="1"/>
+    </inertial>
+    <visual>
+      <origin rpy="0 0 0" xyz="0 0 ${.052/2}"/>
+      <geometry>
+        <box size=".026 .059 .052"/>
+      </geometry>
+      <material name="yellowish">
+        <color rgba=".9 .9 .7 1"/>
+      </material>
+    </visual>
+    <collision>
+      <origin rpy="0 0 0" xyz="0 0 ${.052/2}"/>
+      <geometry>
+        <box size=".026 .059 .052"/>
+      </geometry>
+    </collision>
+  </link>
+  <joint name="set_screw_tool_to_holder" type="fixed">
+    <parent link="screw_tool_holder_short" />
+    <child link="set_screw_tool_link" />
+    <origin xyz="-0.05 ${-back_plate_offset_short + .059/2 + .0155} 0.004" rpy="0.0 0.0 0.0" />
+  </joint>
+  <link name="screw_tool_m4_link">
+    <inertial>
+      <origin rpy="0 0 0" xyz="0 0 0"/>
+      <mass value="1.0"/>
+      <inertia ixx="1" ixy="0" ixz="0" iyy="1" iyz="0" izz="1"/>
+    </inertial>
+    <visual>
+      <origin rpy="0 0 0" xyz="0 0 0"/>
+      <geometry>
+        <mesh filename="package://o2ac_scene_description/meshes/screw_tool_m4_BC5-XL320-AY3.5-EH3R4.stl" scale="0.001 0.001 0.001"/>
       </geometry>
       <material name="white">
@@ -121,37 +175,31 @@
     </visual>
     <collision>
-      <origin rpy="0 0 0" xyz="0 ${bit_cushion_to_axis - .02} .0275"/>
+      <origin rpy="0 0 0" xyz="0 ${-bit_cushion_to_axis + .02} .0275"/>
       <geometry>
         <box size=".026 .04 .055"/>
       </geometry>
-    </collision> -->
-  </link>
-  <joint name="nut_tool_m6_to_holder" type="fixed">
-    <parent link="screw_tool_holder" />
-    <child link="nut_tool_m6_link" />
-    <origin xyz="-0.35 ${tool_offset} 0.004" rpy="0.0 0.0 0.0" />
-  </joint>
-  <link name="set_screw_tool_link">
-    <inertial>
-      <origin rpy="0 0 0" xyz="0 0 0"/>
-      <mass value="1.0"/>
-      <inertia ixx="1" ixy="0" ixz="0" iyy="1" iyz="0" izz="1"/>
-    </inertial>
-  </link>
-  <joint name="set_screw_tool_to_holder" type="fixed">
-    <parent link="screw_tool_holder" />
-    <child link="set_screw_tool_link" />
-    <origin xyz="-0.355 ${tool_offset- .015} 0.004" rpy="0.0 0.0 0.0" />
-  </joint>
-  <link name="screw_tool_m4_link">
-    <inertial>
-      <origin rpy="0 0 0" xyz="0 0 0"/>
-      <mass value="1.0"/>
-      <inertia ixx="1" ixy="0" ixz="0" iyy="1" iyz="0" izz="1"/>
-    </inertial>
-    <visual>
-      <origin rpy="0 0 0" xyz="0 0 0"/>
-      <geometry>
-        <mesh filename="package://o2ac_scene_description/meshes/screw_tool_m4_BC5-XL320-AY3.5-EH3R4.stl" scale="0.001 0.001 0.001"/>
+    </collision>
+    <collision>
+      <origin rpy="0 0 0" xyz="0 0 ${-.12/2}"/>
+      <geometry>
+        <cylinder length=".12" radius=".01"/>
+      </geometry>
+    </collision>
+  </link>
+  <joint name="screw_tool_m4_to_holder" type="fixed">
+    <parent link="screw_tool_holder_long" />
+    <child link="screw_tool_m4_link" />
+    <origin xyz="-0.15 ${tool_offset} 0.004" rpy="0.0 0.0 0.0" />
+  </joint>
+  <link name="screw_tool_m3_link">
+    <inertial>
+      <origin rpy="0 0 0" xyz="0 0 0"/>
+      <mass value="1.0"/>
+      <inertia ixx="1" ixy="0" ixz="0" iyy="1" iyz="0" izz="1"/>
+    </inertial>
+    <visual>
+      <origin rpy="0 0 0" xyz="0 0 0"/>
+      <geometry>
+        <mesh filename="package://o2ac_scene_description/meshes/screw_tool_m3_BC5-XL320-R-AY2.6-EH2.stl" scale="0.001 0.001 0.001"/>
       </geometry>
       <material name="white">
@@ -160,39 +208,18 @@
     </visual>
     <collision>
-      <origin rpy="0 0 0" xyz="0 ${bit_cushion_to_axis - .02} .0275"/>
+      <origin rpy="0 0 0" xyz="0 ${-bit_cushion_to_axis + .02} .0275"/>
       <geometry>
         <box size=".026 .04 .055"/>
       </geometry>
     </collision>
-  </link>
-  <joint name="screw_tool_m4_to_holder" type="fixed">
-    <parent link="screw_tool_holder" />
-    <child link="screw_tool_m4_link" />
-    <origin xyz="-0.15 ${tool_offset} 0.004" rpy="0.0 0.0 0.0" />
-  </joint>
-  <link name="screw_tool_m3_link">
-    <inertial>
-      <origin rpy="0 0 0" xyz="0 0 0"/>
-      <mass value="1.0"/>
-      <inertia ixx="1" ixy="0" ixz="0" iyy="1" iyz="0" izz="1"/>
-    </inertial>
-    <visual>
-      <origin rpy="0 0 0" xyz="0 0 0"/>
-      <geometry>
-        <mesh filename="package://o2ac_scene_description/meshes/screw_tool_m3_BC5-XL320-R-AY2.6-EH2.stl" scale="0.001 0.001 0.001"/>
-      </geometry>
-      <material name="white">
-        <color rgba=".9 .9 .9 1"/>
-      </material>
-    </visual>
-    <collision>
-      <origin rpy="0 0 0" xyz="0 ${bit_cushion_to_axis - .02} .0275"/>
-      <geometry>
-        <box size=".026 .04 .055"/>
+    <collision>
+      <origin rpy="0 0 0" xyz="0 0 ${-.1/2}"/>
+      <geometry>
+        <cylinder length=".1" radius=".01"/>
       </geometry>
     </collision>
   </link>
   <joint name="screw_tool_m3_to_holder" type="fixed">
-    <parent link="screw_tool_holder" />
+    <parent link="screw_tool_holder_long" />
     <child link="screw_tool_m3_link" />
     <origin xyz="-0.25 ${tool_offset} 0.004" rpy="0.0 0.0 0.0" />
@@ -203,5 +230,5 @@
     <parent link="screw_tool_m3_link" />
     <child link="screw_tool_m3_pickup_link" />
-    <origin xyz="0.0 0.0 0.0" rpy="0.0 0.0 ${-pi/2}" />
+    <origin xyz="0.0 0.0 0.0" rpy="0.0 ${pi} ${pi/2}" />
   </joint>
   <link name="screw_tool_m4_pickup_link"/>
@@ -209,11 +236,5 @@
     <parent link="screw_tool_m4_link" />
     <child link="screw_tool_m4_pickup_link" />
-    <origin xyz="0.0 0.0 0.0" rpy="0.0 0.0 ${-pi/2}" />
-  </joint>
-  <link name="belt_tool_pickup_link"/>
-  <joint name="belt_tool_pickup_joint" type="fixed">
-    <parent link="belt_tool_link" />
-    <child link="belt_tool_pickup_link" />
-    <origin xyz="0.0 0.0 0.0" rpy="0.0 0.0 ${-pi/2}" />
+    <origin xyz="0.0 0.0 0.0" rpy="0.0 ${pi} ${pi/2}" />
   </joint>
   <link name="nut_tool_m6_pickup_link"/>
@@ -221,5 +242,5 @@
     <parent link="nut_tool_m6_link" />
     <child link="nut_tool_m6_pickup_link" />
-    <origin xyz="0.0 0.0 0.0" rpy="0.0 0.0 ${-pi/2}" />
+    <origin xyz="0.0 0.0 0.0" rpy="0.0 ${pi} ${pi/2}" />
   </joint>
   <link name="set_screw_tool_pickup_link"/>
@@ -227,5 +248,133 @@
     <parent link="set_screw_tool_link" />
     <child link="set_screw_tool_pickup_link" />
-    <origin xyz="0.0 0.0 0.0" rpy="0.0 0.0 ${-pi/2}" />
+    <origin xyz="0.0 0.0 0.0" rpy="0.0 ${pi} ${pi/2}" />
+  </joint>
+<!-- ================ -->
+<!-- Tools at the front of b_bot base -->
+<!-- Belt hook tool -->
+  <link name="belt_tool_holder">
+    <visual>
+      <origin rpy="${pi/2} 0 ${pi/2}" xyz="0 -.025 -.005"/>
+      <geometry>
+        <mesh filename="package://o2ac_scene_description/meshes/gravity_tool_holder.stl" scale="0.001 0.001 0.001"/>
+      </geometry>
+      <material name="grey">
+        <color rgba=".5 .5 .5 1"/>
+      </material>
+    </visual>
+    <collision>
+      <origin rpy="0 0 0" xyz="${.05/2} 0 ${-.045/2}"/>
+      <geometry>
+        <box size=".05 .05 .045"/>
+      </geometry>
+    </collision>
+  </link>
+  <joint name="belt_holder_to_environment_joint" type="fixed">
+    <parent link="b_bot_base" />
+    <child link="belt_tool_holder" />
+    <origin xyz=".325 -.2 .0" rpy="0 0 0" />
+  </joint>
+  <link name="belt_tool_link">
+    <inertial>
+      <origin rpy="0 0 0" xyz="0 0 0"/>
+      <mass value="1.0"/>
+      <inertia ixx="1" ixy="0" ixz="0" iyy="1" iyz="0" izz="1"/>
+    </inertial>
+    <visual>
+      <origin rpy="0 0 ${-pi/2}" xyz="0.02 0 -0.017"/>
+      <geometry>
+        <mesh filename="package://o2ac_scene_description/meshes/belt_hook_tool.stl" scale="0.001 0.001 0.001"/>
+      </geometry>
+      <material name="white">
+        <color rgba=".9 .9 .9 1"/>
+      </material>
+    </visual>
+    <!-- The graspable part -->
+    <collision>
+      <origin rpy="0 0 0" xyz="${.04/2} 0 ${-.01}"/>
+      <geometry>
+        <box size=".04 .03 .055"/>
+      </geometry>
+    </collision>
+    <!-- The bottom part -->
+    <collision>
+      <origin rpy="0 0 0" xyz="${.02} 0 ${-.03-.1/2}"/>
+      <geometry>
+        <box size=".01 .035 .1"/>
+      </geometry>
+    </collision>
+  </link>
+  <joint name="belt_tool_to_holder_joint" type="fixed">
+    <parent link="belt_tool_holder" />
+    <child link="belt_tool_link" />
+    <origin xyz="0 0 0" rpy="0 0 0" />
+  </joint>
+  <link name="belt_tool_pickup_link"/>
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