Commit message: Add holders, update tools, models etc.

File: catkin_ws/src/o2ac_scene_description/urdf/o2ac_environment.xacro (robot description, xacro)
@@ -15,5 +15,5 @@
   </xacro:o2ac_box>
   <xacro:o2ac_box boxname="horizontal_column_for_tools" box_w=".04" box_l=".4" box_h=".04" parent="o2ac_ground">
-    <origin xyz="${vert_column_x_back} -.2 1.05" rpy="0 0 0" />
+    <origin xyz="${vert_column_x_back} -.2 1.058" rpy="0 0 0" />
   </xacro:o2ac_box>
   <!-- Screw holder & screw tool visual -->
@@ -42,18 +42,19 @@
     <origin xyz="0.04 0.15 0" rpy="0 0 0" />
   </xacro:jig_flat_slope>  -->
-  <xacro:include filename="$(find o2ac_scene_description)/urdf/components/jig_v_slope.xacro" />
+  <!-- <xacro:include filename="$(find o2ac_scene_description)/urdf/components/jig_v_slope.xacro" /> -->
   <!-- <xacro:jig_v_slope jigname="jig_v_slope" parent="horizontal_column_1">
     <origin xyz="0 0 0" rpy="0 0 0" />
   </xacro:jig_v_slope>  -->
-  <!-- <link name="scene_cam_holder_link" />
-  <joint name="scene_cam_holder_joint" type="fixed">
-    <parent link="workspace_center" />
-    <child link="scene_cam_holder_link" />
-    <origin xyz="-0.265 0.03 0.115" rpy="0 0 ${pi/2}" />
-  </joint>
-  <xacro:include filename="$(find realsense2_description)/urdf/_d435.urdf.xacro" />
-  <xacro:arg name="use_nominal_extrinsics" default="True" />
-  <xacro:sensor_d435 parent="scene_cam_holder_link" name="scene_cam">
-    <origin xyz="0 0 0" rpy="0 0 0"/>
-  </xacro:sensor_d435> -->
+  <!-- ======== -->
+  <xacro:include filename="$(find o2ac_scene_description)/urdf/components/nut_holder.xacro" />
+  <xacro:nut_holder partname="nut_holder" parent="a_bot_base_smfl">
+    <origin xyz="0 .6 0.02" rpy="0 0 0" />
+  </xacro:nut_holder>
+  <xacro:include filename="$(find o2ac_scene_description)/urdf/components/washer_holder.xacro" />
+  <xacro:washer_holder partname="washer_holder" parent="a_bot_base_smfl">
+    <origin xyz="0 .54 0.02" rpy="0 0 0" />
+  </xacro:washer_holder>
+  <xacro:nut_holder partname="calibration_cone" parent="workspace_center">
+    <origin xyz="${-0.365+0.01} ${0.345+.03} ${0.022-0.0465}" rpy="0 0 0" />
+  </xacro:nut_holder>
 </robot>

Commit message: WIP: Update scene

File: catkin_ws/src/o2ac_scene_description/urdf/base_scene.urdf.xacro (robot description, xacro)
@@ -15,8 +15,5 @@
   <xacro:include filename="$(find o2ac_gazebo)/urdf/o2ac_base_scene.gazebo" />
   <!-- robots -->
-  <xacro:include filename="$(find ur_description)/urdf/ur5.urdf.xacro" />
   <xacro:include filename="$(find ur_e_description)/urdf/ur5e.urdf.xacro" />
-  <!-- <xacro:include filename="$(find franka_description)/robots/panda_arm.xacro"/>
-  <xacro:include filename="$(find franka_description)/robots/hand.xacro"/> -->
   <!-- Scene items (trays, columns, tools, jigs, feeders...) -->
   <xacro:include filename="$(find o2ac_scene_description)/urdf/o2ac_environment.xacro" />
@@ -61,5 +58,5 @@
     kinematics_file="${load_yaml('$(find o2ac_scene_description)/config/a_bot_calibration.yaml')}"
   />
-  <xacro:ur5_robot prefix="b_bot_" joint_limited="true"
+  <xacro:ur5e_robot prefix="b_bot_" joint_limited="true"
     shoulder_pan_lower_limit="${-pi}" shoulder_pan_upper_limit="${pi}"
     shoulder_lift_lower_limit="${-pi}" shoulder_lift_upper_limit="${pi}"
@@ -68,4 +65,7 @@
     wrist_2_lower_limit="${-pi}" wrist_2_upper_limit="${pi}"
     wrist_3_lower_limit="${-pi}" wrist_3_upper_limit="${pi}"
+    transmission_hw_interface="hardware_interface/PositionJointInterface"
+    safety_limits="false" safety_pos_margin="0.15"
+    safety_k_position="20"
     kinematics_file="${load_yaml('$(find o2ac_scene_description)/config/b_bot_calibration.yaml')}"
   />
@@ -82,8 +82,8 @@
   </joint>
   <!-- spawn and attach robotiq 85 gripper (+ FT300 sensor, soft wrist...) -->
+  <xacro:include filename="$(find o2ac_scene_description)/urdf/components/o2ac_end_effector_2F-140.urdf.xacro" />
+  <xacro:o2ac_end_effector prefix="a_bot_" use_soft_wrist="false" use_cameras="true" parent = "a_bot_ee_link" />
   <xacro:include filename="$(find o2ac_scene_description)/urdf/components/o2ac_end_effector.urdf.xacro" />
-  <xacro:o2ac_end_effector prefix="a_bot_" use_soft_wrist="false" use_cameras="true" parent = "a_bot_ee_link" />
-  <xacro:include filename="$(find o2ac_scene_description)/urdf/components/o2ac_end_effector_old.urdf.xacro" />
-  <xacro:o2ac_end_effector_old prefix="b_bot_" use_soft_wrist="false" use_cameras="true" parent = "b_bot_ee_link" />
+  <xacro:o2ac_end_effector prefix="b_bot_" use_soft_wrist="false" use_cameras="true" parent = "b_bot_ee_link" />
   <!-- Add cameras -->
   <!-- <xacro:include filename="$(find o2ac_scene_description)/urdf/components/_d435.urdf.xacro" />

File: catkin_ws/src/o2ac_scene_description/urdf/components/o2ac_end_effector_2F-140.urdf.xacro (robot description, xacro)
@@ -1,5 +1,5 @@
 <?xml version="1.0"?>
-<!-- This macro adds a convenient TF frame at the tip of the closed gripper. -->
-<!-- The position of the TF frame has not been measured at all and needs to be calibrated. -->
+<!-- This file is a safety measure because a_bot is temporarily using a 2F-140 gripper
+     instead of a 2F-85 gripper. The tip link is set to the . -->
 <robot name="robotiq_85_gripper_o2ac" xmlns:xacro="http://www.ros.org/wiki/xacro">
   <xacro:macro name="o2ac_end_effector" params="prefix use_soft_wrist:=false use_cameras:=false parent">
@@ -16,5 +16,5 @@
       <parent link="${prefix}robotiq_85_base_link"/>
       <child link="${prefix}robotiq_85_tip_link"/>
-      <origin rpy="0.0 0.0 0.0" xyz=".163 0.0 0.0"/>
+      <origin rpy="0.0 0.0 0.0" xyz="${.163+.083} 0.0 0.0"/>
     </joint>
     <link name="${prefix}robotiq_85_tip_link"/>

File: catkin_ws/src/o2ac_scene_description/urdf/components/tools.xacro (robot description, xacro)
@@ -1,8 +1,26 @@
+<?xml version="1.0"?>
+<robot xmlns:xacro="http://www.ros.org/wiki/xacro">
 <!-- This holder has a size of about 155 mm x 40 mm x 26 mm -->
 <!-- The Bit cushion has a height of 30.5 mm, starts about 24 mm from the top-->
 <!-- The gripper center would be about 44 mm from the top, so the tip might be 111 mm further down -->
 <!-- The tip\axis seems to be 11.5 mm from the "front" side. The front side looks into the gripper -->
-<robot xmlns:xacro="http://www.ros.org/wiki/xacro">
-  <!-- Tools at the front of the robot -->
+  <!-- Belt hook tool -->
+  <link name="belt_tool_holder">
+    <visual>
+      <origin rpy="${pi/2} 0 ${pi/2}" xyz="0 -.025 -.005"/>
+      <geometry>
+        <mesh filename="package://o2ac_scene_description/meshes/gravity_tool_holder.stl" scale="0.001 0.001 0.001"/>
+      </geometry>
+      <material name="grey">
+        <color rgba=".5 .5 .5 1"/>
+      </material>
+    </visual>
+    <collision>
+      <origin rpy="0 0 0" xyz="0 0 0"/>
+      <geometry>
+        <box size=".001 .001 .001"/>
+      </geometry>
+    </collision>
+  </link>
   <joint name="belt_holder_to_environment_joint" type="fixed">
     <parent link="b_bot_base" />
@@ -10,21 +28,4 @@
     <origin xyz=".325 -.2 .0" rpy="0 0 0" />
   </joint>
-  <link name="belt_tool_holder">
-    <visual>
-      <origin rpy="${pi/2} 0 ${pi/2}" xyz="0 -.025 -.005"/>
-      <geometry>
-        <mesh filename="package://o2ac_scene_description/meshes/gravity_tool_holder.stl" scale="0.001 0.001 0.001"/>
-      </geometry>
-      <material name="grey">
-        <color rgba=".5 .5 .5 1"/>
-      </material>
-    </visual>
-    <collision>
-      <origin rpy="0 0 0" xyz="0 0 0"/>
-      <geometry>
-        <box size=".001 .001 .001"/>
-      </geometry>
-    </collision>
-  </link>
   <link name="belt_tool_link">
     <inertial>
@@ -52,4 +53,54 @@
     <parent link="belt_tool_holder" />
     <child link="belt_tool_link" />
+    <origin xyz="0 0 0" rpy="0 0 0" />
+  </joint>
+  <!-- Plunger tool -->
+  <link name="plunger_tool_holder">
+    <visual>
+      <origin rpy="${pi/2} 0 ${pi/2}" xyz="0 -.025 -.005"/>
+      <geometry>
+        <mesh filename="package://o2ac_scene_description/meshes/gravity_tool_holder.stl" scale="0.001 0.001 0.001"/>
+      </geometry>
+      <material name="grey">
+        <color rgba=".5 .5 .5 1"/>
+      </material>
+    </visual>
+    <collision>
+      <origin rpy="0 0 0" xyz="0 0 0"/>
+      <geometry>
+        <box size=".001 .001 .001"/>
+      </geometry>
+    </collision>
+  </link>
+  <joint name="plunger_holder_to_environment_joint" type="fixed">
+    <parent link="b_bot_base" />
+    <child link="plunger_tool_holder" />
+    <origin xyz=".325 -.1 .0" rpy="0 0 0" />
+  </joint>
+  <link name="plunger_tool_link">
+    <inertial>
+      <origin rpy="0 0 0" xyz="0 0 0"/>
+      <mass value="1.0"/>
+      <inertia ixx="1" ixy="0" ixz="0" iyy="1" iyz="0" izz="1"/>
+    </inertial>
+    <visual>
+      <origin rpy="0 ${pi/2} ${pi/2}" xyz="0.02 0 -0.017"/>
+      <geometry>
+        <mesh filename="package://o2ac_scene_description/meshes/plunger_tool.stl" scale="0.001 0.001 0.001"/>
+      </geometry>
+      <material name="white">
+        <color rgba=".9 .9 .9 1"/>
+      </material>
+    </visual>
+    <collision>
+      <origin rpy="0 0 0" xyz="0 0 0"/>
+      <geometry>
+        <box size=".026 .04 .055"/>
+      </geometry>
+    </collision>
+  </link>
+  <joint name="plunger_tool_to_holder" type="fixed">
+    <parent link="plunger_tool_holder" />
+    <child link="plunger_tool_link" />
     <origin xyz="0 0 0" rpy="0 0 0" />
   </joint>

File: catkin_ws/src/o2ac_scene_description/urdf/o2ac_environment.xacro (robot description, xacro)
@@ -42,5 +42,5 @@
     <origin xyz="0.04 0.15 0" rpy="0 0 0" />
   </xacro:jig_flat_slope>  -->
-  <xacro:include filename="$(find o2ac_scene_description)/urdf/components/jig_v_slope.xacro" />
+  <!-- <xacro:include filename="$(find o2ac_scene_description)/urdf/components/jig_v_slope.xacro" /> -->
   <!-- <xacro:jig_v_slope jigname="jig_v_slope" parent="horizontal_column_1">
     <origin xyz="0 0 0" rpy="0 0 0" />
@@ -57,3 +57,14 @@
     <origin xyz="0 0 0" rpy="0 0 0"/>
   </xacro:sensor_d435> -->
+  <!-- ======== -->
+  <xacro:include filename="$(find o2ac_scene_description)/urdf/components/nut_holder.xacro" />
+  <xacro:nut_holder partname="nut_holder" parent="a_bot_base_smfl">
+    <origin xyz="0 .6 0.02" rpy="0 0 0" />
+  </xacro:nut_holder>
+  <xacro:include filename="$(find o2ac_scene_description)/urdf/components/washer_holder.xacro" />
+  <xacro:washer_holder partname="washer_holder" parent="a_bot_base_smfl">
+    <origin xyz="0 .54 0.02" rpy="0 0 0" />
+  </xacro:washer_holder>
+  <!-- Robotiq tip link at the tip of the nut holder  -->
+  <!-- -0.33429; -0.23224; 0.76964 -->
 </robot>

Commit message: Update cameras

File: catkin_ws/src/o2ac_scene_description/urdf/base_scene.urdf.xacro (robot description, xacro)
@@ -81,20 +81,9 @@
     <origin xyz="${b_bot_x} ${b_bot_y} ${bots_z}" rpy="0.0 0.0 ${b_bot_theta}" />
   </joint>
-  <!-- spawn and attach robotiq 85 gripper (+ FT300 sensor, soft wrist...) -->
+  <!-- Spawn and attach robotiq 85 gripper (+ cameras) -->
   <xacro:include filename="$(find o2ac_scene_description)/urdf/components/o2ac_end_effector_2F-140.urdf.xacro" />
   <xacro:o2ac_end_effector prefix="a_bot_" use_soft_wrist="false" use_cameras="true" parent = "a_bot_ee_link" />
   <xacro:include filename="$(find o2ac_scene_description)/urdf/components/o2ac_end_effector.urdf.xacro" />
   <xacro:o2ac_end_effector prefix="b_bot_" use_soft_wrist="false" use_cameras="true" parent = "b_bot_ee_link" />
-  <!-- Add cameras -->
-  <!-- <xacro:include filename="$(find o2ac_scene_description)/urdf/components/_d435.urdf.xacro" />
-  <link name="scene_cam_holder_link" />
-  <joint name="scene_cam_holder_joint" type="fixed">
-    <parent link="workspace_center" />
-    <child  link="scene_cam_holder_link" />
-    <origin xyz="-0.0179662 -0.155013 0.101615" rpy="0.0281409 -0.137996 -0.0954644" />
-  </joint>
-  <xacro:sensor_d435 prefix="scene_" parent="scene_cam_holder_link">
-    <origin xyz="0 0 0" rpy="0 0 0"/>
-  </xacro:sensor_d435> -->
   <!-- The "world" link definition should be removed, but apparently it is necessary for Gazebo -->
   <link name="world" />

File: catkin_ws/src/o2ac_scene_description/urdf/components/_d435.urdf.xacro (robot description, xacro)
@@ -2,7 +2,8 @@
 <!-- This macro adds a rotated frame at the depth camera, for use with the OMRON cad matching library. -->
 <robot name="o2ac_sensor_d435" xmlns:xacro="http://wiki.ros.org/xacro">
-  <xacro:include filename="$(find realsense2_camera)/urdf/_d435.urdf.xacro" />
+  <xacro:include filename="$(find realsense2_description)/urdf/_d435.urdf.xacro" />
+  <!-- <xacro:include filename="$(find o2ac_scene_description)/urdf/components/_d435_internal.urdf.xacro" /> -->
   <xacro:macro name="o2ac_sensor_d435" params="prefix parent *origin">
-    <xacro:sensor_d435 prefix="${prefix}" parent="${parent}">
+    <xacro:sensor_d435 name="${prefix}camera" parent="${parent}">
       <xacro:insert_block name="origin" />
     </xacro:sensor_d435>

File: catkin_ws/src/o2ac_scene_description/urdf/o2ac_environment.xacro (robot description, xacro)
@@ -46,15 +46,4 @@
     <origin xyz="0 0 0" rpy="0 0 0" />
   </xacro:jig_v_slope>  -->
-  <!-- <link name="scene_cam_holder_link" />
-  <joint name="scene_cam_holder_joint" type="fixed">
-    <parent link="workspace_center" />
-    <child link="scene_cam_holder_link" />
-    <origin xyz="-0.265 0.03 0.115" rpy="0 0 ${pi/2}" />
-  </joint>
-  <xacro:include filename="$(find realsense2_description)/urdf/_d435.urdf.xacro" />
-  <xacro:arg name="use_nominal_extrinsics" default="True" />
-  <xacro:sensor_d435 parent="scene_cam_holder_link" name="scene_cam">
-    <origin xyz="0 0 0" rpy="0 0 0"/>
-  </xacro:sensor_d435> -->
   <!-- ======== -->
   <xacro:include filename="$(find o2ac_scene_description)/urdf/components/nut_holder.xacro" />

Commit message: Temporary scene changes

File: catkin_ws/src/o2ac_scene_description/urdf/base_scene.urdf.xacro (robot description, xacro)
@@ -19,5 +19,5 @@
   <xacro:include filename="$(find o2ac_scene_description)/urdf/o2ac_environment.xacro" />
   <!-- <xacro:include filename="$(find flexwrist_experiment)/urdf/2020-01-experiment-scene.xacro" /> -->
-  <xacro:include filename="$(find o2ac_scene_description)/urdf/taskboard_scene.xacro" />
+  <!-- <xacro:include filename="$(find o2ac_scene_description)/urdf/taskboard_scene.xacro" /> -->
   <!-- <xacro:include filename="$(find o2ac_scene_description)/urdf/assembly_scene.xacro" /> -->
   <!-- Robot bases -->
@@ -47,6 +47,6 @@
   </joint>
   <xacro:ur5e_robot prefix="a_bot_" joint_limited="true"
-    shoulder_pan_lower_limit="${-pi}" shoulder_pan_upper_limit="${pi}"
-    shoulder_lift_lower_limit="${-pi}" shoulder_lift_upper_limit="${pi}"
+    shoulder_pan_lower_limit="${-pi/1.5}" shoulder_pan_upper_limit="${pi/1.5}"
+    shoulder_lift_lower_limit="${-pi/1.5}" shoulder_lift_upper_limit="${pi/1.5}"
     elbow_joint_lower_limit="0.0" elbow_joint_upper_limit="${pi}"
     wrist_1_lower_limit="${-pi}" wrist_1_upper_limit="${pi}"
@@ -59,6 +59,6 @@
   />
   <xacro:ur5e_robot prefix="b_bot_" joint_limited="true"
-    shoulder_pan_lower_limit="${-pi}" shoulder_pan_upper_limit="${pi}"
-    shoulder_lift_lower_limit="${-pi}" shoulder_lift_upper_limit="${pi}"
+    shoulder_pan_lower_limit="${-pi/1.5}" shoulder_pan_upper_limit="${pi/1.5}"
+    shoulder_lift_lower_limit="${-pi/1.5}" shoulder_lift_upper_limit="${pi/1.5}"
     elbow_joint_lower_limit="0.0" elbow_joint_upper_limit="${pi}"
     wrist_1_lower_limit="${-pi}" wrist_1_upper_limit="${pi}"
@@ -82,5 +82,6 @@
   </joint>
   <!-- Spawn and attach robotiq 85 gripper (+ cameras) -->
-  <xacro:include filename="$(find o2ac_scene_description)/urdf/components/o2ac_end_effector_2F-140.urdf.xacro" />
+  <!-- <xacro:include filename="$(find o2ac_scene_description)/urdf/components/o2ac_end_effector_2F-140.urdf.xacro" /> -->
+  <xacro:include filename="$(find o2ac_scene_description)/urdf/components/o2ac_end_effector.urdf.xacro" />
   <xacro:o2ac_end_effector prefix="a_bot_" use_soft_wrist="false" use_cameras="true" parent = "a_bot_ee_link" />
   <xacro:include filename="$(find o2ac_scene_description)/urdf/components/o2ac_end_effector.urdf.xacro" />

File: catkin_ws/src/o2ac_scene_description/urdf/components/tools.xacro (robot description, xacro)
@@ -74,10 +74,10 @@
       </material>
     </visual>
-    <collision>
+    <!-- <collision>
       <origin rpy="0 0 0" xyz="-0.05 .0013 0.002"/>
       <geometry>
         <box size=".1 .066 .004"/>
       </geometry>
-    </collision>
+    </collision> -->
     <!-- The vertical plate -->
     <visual>
@@ -90,10 +90,10 @@
       </material>
     </visual>
-    <collision>
+    <!-- <collision>
       <origin rpy="0 0 0" xyz="-0.05 -.014 0.0179"/>
       <geometry>
         <box size=".1 .004 .035"/>
       </geometry>
-    </collision>
+    </collision> -->
   </link>
   <!-- ++++++++++++++++++++++++++++ -->
@@ -174,10 +174,10 @@
       </material>
     </visual>
-    <collision>
+    <!-- <collision>
       <origin rpy="0 0 0" xyz="0 ${-bit_cushion_to_axis + .02} .0275"/>
       <geometry>
         <box size=".026 .04 .055"/>
       </geometry>
-    </collision>
+    </collision> -->
     <collision>
       <origin rpy="0 0 0" xyz="0 0 ${-.12/2}"/>
@@ -207,10 +207,10 @@
       </material>
     </visual>
-    <collision>
+    <!-- <collision>
       <origin rpy="0 0 0" xyz="0 ${-bit_cushion_to_axis + .02} .0275"/>
       <geometry>
         <box size=".026 .04 .055"/>
       </geometry>
-    </collision>
+    </collision> -->
     <collision>
       <origin rpy="0 0 0" xyz="0 0 ${-.1/2}"/>

Commit message: Add missing script select_realsense_camera.py

File: catkin_ws/src/o2ac_scene_description/urdf/base_scene.urdf.xacro (robot description, xacro)
@@ -84,7 +84,8 @@
   <!-- spawn and attach robotiq 85 gripper (+ FT300 sensor, soft wrist...) -->
   <xacro:include filename="$(find o2ac_scene_description)/urdf/components/o2ac_end_effector_new.urdf.xacro" />
-  <xacro:o2ac_end_effector prefix="a_bot_" use_soft_wrist="false" use_cameras="true" parent = "a_bot_ee_link" />
-  <xacro:include filename="$(find o2ac_scene_description)/urdf/components/o2ac_end_effector_old.urdf.xacro" />
-  <xacro:o2ac_end_effector_old prefix="b_bot_" use_soft_wrist="false" use_cameras="true" parent = "b_bot_ee_link" />
+  <xacro:o2ac_end_effector_new prefix="a_bot_" use_soft_wrist="false" use_cameras="true" parent = "a_bot_ee_link" />
+  <xacro:include filename="$(find o2ac_scene_description
+			   )/urdf/components/o2ac_end_effector.urdf.xacro" />
+  <xacro:o2ac_end_effector prefix="b_bot_" use_soft_wrist="false" use_cameras="true" parent = "b_bot_ee_link" />
   <!-- Add cameras -->
   <!-- <xacro:include filename="$(find o2ac_scene_description)/urdf/components/_d435.urdf.xacro" />

File: catkin_ws/src/o2ac_scene_description/urdf/components/o2ac_end_effector_new.urdf.xacro (robot description, xacro)
@@ -3,5 +3,5 @@
 <!-- The position of the TF frame has not been measured at all and needs to be calibrated. -->
 <robot name="robotiq_140_gripper_o2ac" xmlns:xacro="http://www.ros.org/wiki/xacro">
-  <xacro:macro name="o2ac_end_effector" params="prefix use_soft_wrist:=false use_cameras:=false parent">
+  <xacro:macro name="o2ac_end_effector_new" params="prefix use_soft_wrist:=false use_cameras:=false parent">
     <xacro:include filename="$(find robotiq_description)/urdf/robotiq_140_gripper.urdf.xacro"/>
     <xacro:robotiq_140_gripper prefix="${prefix}" parent="${parent}">

Commit message: WIP: squash redundant commits

File: catkin_ws/src/o2ac_scene_description/urdf/base_scene.urdf.xacro (robot description, xacro)
@@ -62,5 +62,5 @@
     kinematics_file="${load_yaml('$(find o2ac_scene_description)/config/a_bot_calibration.yaml')}"
   />
-  <xacro:ur5_robot prefix="b_bot_" joint_limited="true"
+  <xacro:ur5e_robot prefix="b_bot_" joint_limited="true"
     shoulder_pan_lower_limit="${-pi}" shoulder_pan_upper_limit="${pi}"
     shoulder_lift_lower_limit="${-pi}" shoulder_lift_upper_limit="${pi}"
@@ -83,20 +83,9 @@
   </joint>
   <!-- spawn and attach robotiq 85 gripper (+ FT300 sensor, soft wrist...) -->
-  <xacro:include filename="$(find o2ac_scene_description)/urdf/components/o2ac_end_effector_new.urdf.xacro" />
-  <xacro:o2ac_end_effector_new prefix="a_bot_" use_soft_wrist="false" use_cameras="true" parent = "a_bot_ee_link" />
+  <xacro:include filename="$(find o2ac_scene_description)/urdf/components/o2ac_end_effector_2F-140.urdf.xacro" />
+  <xacro:o2ac_end_effector prefix="a_bot_" use_soft_wrist="false" use_cameras="true" parent = "a_bot_ee_link" />
   <xacro:include filename="$(find o2ac_scene_description
 			   )/urdf/components/o2ac_end_effector.urdf.xacro" />
   <xacro:o2ac_end_effector prefix="b_bot_" use_soft_wrist="false" use_cameras="true" parent = "b_bot_ee_link" />
-  <!-- Add cameras -->
-  <!-- <xacro:include filename="$(find o2ac_scene_description)/urdf/components/_d435.urdf.xacro" />
-  <link name="scene_cam_holder_link" />
-  <joint name="scene_cam_holder_joint" type="fixed">
-    <parent link="workspace_center" />
-    <child  link="scene_cam_holder_link" />
-    <origin xyz="-0.0179662 -0.155013 0.101615" rpy="0.0281409 -0.137996 -0.0954644" />
-  </joint>
-  <xacro:sensor_d435 prefix="scene_" parent="scene_cam_holder_link">
-    <origin xyz="0 0 0" rpy="0 0 0"/>
-  </xacro:sensor_d435> -->
   <!-- The "world" link definition should be removed, but apparently it is necessary for Gazebo -->
   <link name="world" />

File: catkin_ws/src/o2ac_scene_description/urdf/calibration_scene.xacro (robot description, xacro)
@@ -9,9 +9,9 @@
   <!--   <origin xyz="0.0 0.0 0.0185" rpy="0 0 0"/> -->
   <!-- </xacro:ar_marker_70_5> -->
-  <xacro:ar_marker_80_10 prefix="base_"
+  <xacro:ar_marker_70_5 prefix="base_"
 			parent="attached_base_origin_link"
-			marker_id="17"
+			marker_id="32"
 			thickness="0.001">
     <origin xyz="0.06 0.06 0.0005" rpy="0 0 0"/>
-  </xacro:ar_marker_80_10>
+  </xacro:ar_marker_70_5>
 </robot>

Commit message: Update scene for screw picking

File: catkin_ws/src/o2ac_scene_description/urdf/base_scene.urdf.xacro (robot description, xacro)
@@ -4,5 +4,5 @@
   <!-- This is the main file defining our robot arrangement and physical environment. -->
   <!-- Calibration parameters -->
-  <xacro:property name="a_bot_x" value="-0.0"/>
+  <xacro:property name="a_bot_x" value="-0.004"/>
   <xacro:property name="a_bot_y" value="-0.525"/>
   <xacro:property name="a_bot_theta" value="0.0"/>

File: catkin_ws/src/o2ac_scene_description/urdf/o2ac_environment.xacro (robot description, xacro)
@@ -25,5 +25,5 @@
   </xacro:screw_feeder>
   <xacro:screw_feeder feedername="m4_feeder" parent="workspace_center">
-    <origin xyz="-.512 0 -0.023" rpy="0 0 0" />
+    <origin xyz="-.513 -0.002 -0.023" rpy="0 0 0" />
   </xacro:screw_feeder>
   <!-- Base fixture -->
