Commit message: Scene updates

File: catkin_ws/src/o2ac_scene_description/urdf/base_scene.urdf.xacro (robot description, xacro)
@@ -51,5 +51,5 @@
     shoulder_lift_lower_limit="${-pi}" shoulder_lift_upper_limit="${pi}"
     elbow_joint_lower_limit="0.0" elbow_joint_upper_limit="${pi}"
-    wrist_1_lower_limit="${-pi}" wrist_1_upper_limit="${pi}"
+    wrist_1_lower_limit="${-pi*1.5}" wrist_1_upper_limit="${pi}"
     wrist_2_lower_limit="${-pi*1.5}" wrist_2_upper_limit="${pi*1.5}"
     wrist_3_lower_limit="${-2*pi}" wrist_3_upper_limit="${2*pi}"
@@ -63,5 +63,5 @@
     shoulder_lift_lower_limit="${-pi}" shoulder_lift_upper_limit="${pi}"
     elbow_joint_lower_limit="0.0" elbow_joint_upper_limit="${pi}"
-    wrist_1_lower_limit="${-pi}" wrist_1_upper_limit="${pi}"
+    wrist_1_lower_limit="${-pi*1.5}" wrist_1_upper_limit="${pi}"
     wrist_2_lower_limit="${-pi*1.5}" wrist_2_upper_limit="${pi*1.5}"
     wrist_3_lower_limit="${-2*pi}" wrist_3_upper_limit="${2*pi}"

File: catkin_ws/src/o2ac_scene_description/urdf/components/o2ac_end_effector_2F-140.urdf.xacro (robot description, xacro)
@@ -43,5 +43,5 @@
       <parent link="${prefix}tool_intermediate_link"/>
       <child link="${prefix}screw_tool_m3_tip_link"/>
-      <origin rpy="0 0 0" xyz=".14 0 .015 "/>
+      <origin rpy="0 0 0" xyz=".121 0 .003 "/>
     </joint>
     <link name="${prefix}screw_tool_m3_tip_link"/>

File: catkin_ws/src/o2ac_scene_description/urdf/components/taskboard.xacro (robot description, xacro)
@@ -79,5 +79,5 @@
   <xacro:include filename="$(find o2ac_parts_description)/urdf/generated/07_SBARB6200ZZ_30_macro.urdf.xacro" />
   <xacro:assy_part_07 prefix="${boardname}_" parent="${boardname}_plate" spawn_attached="true">
-    <origin rpy="0 0 0" xyz="${0.025+.008} 0.165 0.12"/>
+    <origin rpy="${pi} 0 0" xyz="${0.025+.008} 0.165 0.12"/>
   </xacro:assy_part_07>
   <!-- The large pulley -->
@@ -137,5 +137,5 @@
     <parent link="${boardname}_plate"/>
     <child link="${boardname}_set_screw_link"/>
-    <origin rpy="0 0 ${pi}" xyz=".025 0.054 0.075"/>
+    <origin rpy="${pi} 0 ${pi}" xyz=".025 0.054 0.075"/>
   </joint>
   <link name="${boardname}_set_screw_link"/>
@@ -143,5 +143,5 @@
     <parent link="${boardname}_plate"/>
     <child link="${boardname}_m3_screw_link"/>
-    <origin rpy="0 0 ${pi}" xyz=".025 0.072 0.035"/>
+    <origin rpy="${pi} 0 ${pi}" xyz=".025 0.072 0.035"/>
   </joint>
   <link name="${boardname}_m3_screw_link"/>
@@ -149,5 +149,5 @@
     <parent link="${boardname}_plate"/>
     <child link="${boardname}_m4_screw_link"/>
-    <origin rpy="0 0 ${pi}" xyz=".025 0.105 0.036"/>
+    <origin rpy="${pi} 0 ${pi}" xyz=".025 0.105 0.036"/>
   </joint>
   <link name="${boardname}_m4_screw_link"/>
@@ -155,5 +155,5 @@
     <parent link="${boardname}_plate"/>
     <child link="${boardname}_long_hole_middle_link"/>
-    <origin rpy="0 0 ${pi}" xyz=".025 0.1 0.125"/>
+    <origin rpy="${pi} 0 ${pi}" xyz=".025 0.1 0.125"/>
   </joint>
   <link name="${boardname}_long_hole_middle_link"/>

File: catkin_ws/src/o2ac_scene_description/urdf/o2ac_environment.xacro (robot description, xacro)
@@ -22,5 +22,5 @@
   <xacro:include filename="$(find o2ac_scene_description)/urdf/components/screw_feeder.xacro" />
   <xacro:screw_feeder feedername="m3_feeder" parent="workspace_center">
-    <origin xyz="-.511 -.13 -0.023" rpy="0 0 0" />
+    <origin xyz="-.511 -.132 -0.023" rpy="0 0 0" />
   </xacro:screw_feeder>
   <xacro:screw_feeder feedername="m4_feeder" parent="workspace_center">

Commit message: Add vgroove aid to scene

File: catkin_ws/src/o2ac_scene_description/urdf/base_scene.urdf.xacro (robot description, xacro)
@@ -13,5 +13,5 @@
   <!-- common stuff -->
   <xacro:include filename="$(find ur_description)/urdf/common.gazebo.xacro" />
-  <xacro:include filename="$(find o2ac_gazebo)/urdf/o2ac_base_scene.gazebo" />
+  <!-- <xacro:include filename="$(find o2ac_gazebo)/urdf/o2ac_base_scene.gazebo" /> -->
   <!-- robots -->
   <xacro:include filename="$(find ur_e_description)/urdf/ur5e.urdf.xacro" />

File: catkin_ws/src/o2ac_scene_description/urdf/o2ac_environment.xacro (robot description, xacro)
@@ -42,8 +42,8 @@
     <origin xyz="0.04 0.15 0" rpy="0 0 0" />
   </xacro:jig_flat_slope>  -->
-  <!-- <xacro:include filename="$(find o2ac_scene_description)/urdf/components/jig_v_slope.xacro" /> -->
-  <!-- <xacro:jig_v_slope jigname="jig_v_slope" parent="horizontal_column_1">
-    <origin xyz="0 0 0" rpy="0 0 0" />
-  </xacro:jig_v_slope>  -->
+  <xacro:include filename="$(find o2ac_scene_description)/urdf/components/vgroove_aid.xacro" />
+  <xacro:vgroove_aid jigname="vgroove_aid" parent="b_bot_base_link">
+    <origin xyz="-0.2927 0.17214 0.0" rpy="0 0 0" />
+  </xacro:vgroove_aid>
   <!-- ======== -->
   <!-- <xacro:include filename="$(find o2ac_scene_description)/urdf/components/nut_holder.xacro" />

Commit message: Adjust feeders & M3 screw tool position

File: catkin_ws/src/o2ac_scene_description/urdf/base_scene.urdf.xacro (robot description, xacro)
@@ -21,5 +21,5 @@
   <xacro:include filename="$(find o2ac_scene_description)/urdf/taskboard_scene.xacro" />
   <!-- <xacro:include filename="$(find o2ac_scene_description)/urdf/assembly_scene.xacro" /> -->
-  <!-- <xacro:include filename="$(find o2ac_scene_description)/urdf/calibration_scene.xacro" /> -->
+  <!-- <xacro:include filename="$(find o2ac_scene_description)/urdf/camera_calibration_scene.xacro" /> -->
   <!-- Robot bases -->
   <!-- Putting these at height 0.0 makes them intersect with the ground, so they are elevated. -->

File: catkin_ws/src/o2ac_scene_description/urdf/components/o2ac_end_effector_2F-140.urdf.xacro (robot description, xacro)
@@ -43,5 +43,5 @@
       <parent link="${prefix}tool_intermediate_link"/>
       <child link="${prefix}screw_tool_m3_tip_link"/>
-      <origin rpy="0 0 0" xyz=".121 0 .003 "/>
+      <origin rpy="0 0 0" xyz=".121 0 .0055 "/>
     </joint>
     <link name="${prefix}screw_tool_m3_tip_link"/>

File: catkin_ws/src/o2ac_scene_description/urdf/o2ac_environment.xacro (robot description, xacro)
@@ -22,8 +22,8 @@
   <xacro:include filename="$(find o2ac_scene_description)/urdf/components/screw_feeder.xacro" />
   <xacro:screw_feeder feedername="m3_feeder" parent="workspace_center">
-    <origin xyz="-.511 -.132 -0.023" rpy="0 0 0" />
+    <origin xyz="-.513 -.152 -0.023" rpy="0 0 0" />
   </xacro:screw_feeder>
   <xacro:screw_feeder feedername="m4_feeder" parent="workspace_center">
-    <origin xyz="-.513 -0.002 -0.023" rpy="0 0 0" />
+    <origin xyz="-.511 .005 -0.023" rpy="0 0 0" />
   </xacro:screw_feeder>
   <!-- Base fixture -->

Commit message: Fix minor issues

File: catkin_ws/src/o2ac_scene_description/urdf/base_scene.urdf.xacro (robot description, xacro)
@@ -19,6 +19,6 @@
   <xacro:include filename="$(find o2ac_scene_description)/urdf/o2ac_environment.xacro" />
   <!-- <xacro:include filename="$(find flexwrist_experiment)/urdf/2020-01-experiment-scene.xacro" /> -->
-  <!-- <xacro:include filename="$(find o2ac_scene_description)/urdf/taskboard_scene.xacro" /> -->
-  <xacro:include filename="$(find o2ac_scene_description)/urdf/assembly_scene.xacro" />
+  <xacro:include filename="$(find o2ac_scene_description)/urdf/taskboard_scene.xacro" />
+  <!-- <xacro:include filename="$(find o2ac_scene_description)/urdf/assembly_scene.xacro" /> -->
   <!-- <xacro:include filename="$(find o2ac_scene_description)/urdf/camera_calibration_scene.xacro" /> -->
   <!-- Robot bases -->

File: catkin_ws/src/o2ac_scene_description/urdf/o2ac_environment.xacro (robot description, xacro)
@@ -25,5 +25,5 @@
   </xacro:screw_feeder>
   <xacro:screw_feeder feedername="m4_feeder" parent="workspace_center">
-    <origin xyz="-.513 .004 -0.023" rpy="0 0 0" />
+    <origin xyz="-.513 .006 -0.023" rpy="0 0 0" />
   </xacro:screw_feeder>
   <!-- Base fixture -->

Commit message: Adjust magic numbers

File: catkin_ws/src/o2ac_scene_description/urdf/base_scene.urdf.xacro (robot description, xacro)
@@ -19,6 +19,6 @@
   <xacro:include filename="$(find o2ac_scene_description)/urdf/o2ac_environment.xacro" />
   <!-- <xacro:include filename="$(find flexwrist_experiment)/urdf/2020-01-experiment-scene.xacro" /> -->
-  <!-- <xacro:include filename="$(find o2ac_scene_description)/urdf/taskboard_scene.xacro" /> -->
-  <xacro:include filename="$(find o2ac_scene_description)/urdf/assembly_scene.xacro" />
+  <xacro:include filename="$(find o2ac_scene_description)/urdf/taskboard_scene.xacro" />
+  <!-- <xacro:include filename="$(find o2ac_scene_description)/urdf/assembly_scene.xacro" /> -->
   <!-- <xacro:include filename="$(find o2ac_scene_description)/urdf/camera_calibration_scene.xacro" /> -->
   <!-- Robot bases -->

File: catkin_ws/src/o2ac_scene_description/urdf/o2ac_environment.xacro (robot description, xacro)
@@ -22,8 +22,8 @@
   <xacro:include filename="$(find o2ac_scene_description)/urdf/components/screw_feeder.xacro" />
   <xacro:screw_feeder feedername="m3_feeder" parent="workspace_center">
-    <origin xyz="-.512 -.152 -0.023" rpy="0 0 0" />
+    <origin xyz="-.514 -.151 -0.023" rpy="0 0 0" />
   </xacro:screw_feeder>
   <xacro:screw_feeder feedername="m4_feeder" parent="workspace_center">
-    <origin xyz="-.512 .006 -0.023" rpy="0 0 0" />
+    <origin xyz="-.514 .004 -0.023" rpy="0 0 0" />
   </xacro:screw_feeder>
   <!-- Base fixture -->

Commit message: Add invisible walls for plan safety

File: catkin_ws/src/o2ac_scene_description/urdf/base_scene.urdf.xacro (robot description, xacro)
@@ -20,4 +20,5 @@
   <xacro:include filename="$(find o2ac_scene_description)/urdf/o2ac_environment.xacro" />
   <!-- <xacro:include filename="$(find flexwrist_experiment)/urdf/2020-01-experiment-scene.xacro" /> -->
+  <!-- This argument can be set in base_scene_upload.launch -->
   <xacro:if value="$(arg taskboard)">
     <xacro:include filename="$(find o2ac_scene_description)/urdf/taskboard_scene.xacro" />

File: catkin_ws/src/o2ac_scene_description/urdf/components/o2ac_box_2.xacro (robot description, xacro)
@@ -1,11 +1,11 @@
 <?xml version="1.0"?>
 <robot xmlns:xacro="http://www.ros.org/wiki/xacro">
-  <xacro:macro name="o2ac_box" params="boxname box_w box_l box_h parent invisible:=false *origin">
-    <!-- This creates a box with the origin in the bottom corner. -->
+  <xacro:macro name="o2ac_box_2" params="boxname box_w box_l box_h parent invisible:=false *origin">
+    <!-- A simple macro for a box that can have its visual geometry hidden. -->
     <link name="${boxname}">
       <!-- w is in x, l is in y, h is in z -->
       <xacro:if value="${not invisible}">
         <visual>
-          <origin xyz="${box_w/2} ${box_l/2} ${box_h/2}" rpy="0 0 0"/>
+          <origin xyz="0 0 0" rpy="0 0 0"/>
           <geometry>
             <box size="${box_w} ${box_l} ${box_h}"/>
@@ -17,5 +17,5 @@
       </xacro:if>
       <collision>
-        <origin xyz="${box_w/2} ${box_l/2} ${box_h/2}" rpy="0 0 0"/>
+        <origin xyz="0 0 0" rpy="0 0 0"/>
         <geometry>
           <box size="${box_w} ${box_l} ${box_h}"/>

File: catkin_ws/src/o2ac_scene_description/urdf/o2ac_environment.xacro (robot description, xacro)
@@ -3,4 +3,5 @@
        name="o2ac_environment" >
   <xacro:include filename="$(find o2ac_scene_description)/urdf/components/o2ac_box.xacro" />
+  <xacro:include filename="$(find o2ac_scene_description)/urdf/components/o2ac_box_2.xacro" />
   <!-- This file defines the frames surrounding the robots, used to fix the tools, multi-jig etc. -->
   <xacro:property name="vert_column_x_back" value="${-.325-.15-.04}"/>
@@ -17,4 +18,20 @@
     <origin xyz="${vert_column_x_back} -.2 1.058" rpy="0 0 0" />
   </xacro:o2ac_box>
+  <!-- Invisible walls to avoid OMPL creating crazy plans (sanity limits) -->
+  <xacro:o2ac_box_2 boxname="agv_table" box_w=".6" box_l=".5" box_h=".05" invisible="true" parent="workspace_center">
+    <origin xyz=".65 0 -.04" rpy="0 0 0" />
+  </xacro:o2ac_box_2>
+  <xacro:o2ac_box_2 boxname="back_limit_a" box_w=".05" box_l=".5" box_h=".5" invisible="true" parent="workspace_center">
+    <origin xyz="${vert_column_x_back} -.5 .3" rpy="0 0 0" />
+  </xacro:o2ac_box_2>
+  <xacro:o2ac_box_2 boxname="back_limit_b" box_w=".05" box_l=".5" box_h=".5" invisible="true" parent="workspace_center">
+    <origin xyz="${vert_column_x_back} .5 .3" rpy="0 0 0" />
+  </xacro:o2ac_box_2>
+  <xacro:o2ac_box_2 boxname="side_limit_a" box_w="1.0" box_l=".05" box_h="1.0" invisible="true" parent="workspace_center">
+    <origin xyz=".0 1.1 .5" rpy="0 0 0" />
+  </xacro:o2ac_box_2>
+  <xacro:o2ac_box_2 boxname="side_limit_b" box_w="1.0" box_l=".05" box_h="1.0" invisible="true" parent="workspace_center">
+    <origin xyz=".0 -1.1 .5" rpy="0 0 0" />
+  </xacro:o2ac_box_2>
   <!-- Screw holder & screw tool visual -->
   <xacro:include filename="$(find o2ac_scene_description)/urdf/components/tools.xacro" />

Commit message: WIP: Tons of offsets and calibration additions
Not finished, but screw picking works and the tool heights seem roughly correct

File: catkin_ws/src/o2ac_scene_description/urdf/base_scene.urdf.xacro (robot description, xacro)
@@ -6,9 +6,12 @@
   <!-- Calibration parameters -->
   <xacro:property name="a_bot_x" value="-0.004"/>
-  <xacro:property name="a_bot_y" value="-0.525"/>
-  <xacro:property name="a_bot_theta" value="0.0"/>
-  <xacro:property name="b_bot_x" value="-0.0"/>
-  <xacro:property name="b_bot_y" value="0.525"/>
-  <xacro:property name="b_bot_theta" value="-3.141"/>
+  <xacro:property name="a_bot_y" value="-0.531"/>     <!-- Positive moves to the left -->
+  <!-- Original: -0.525 -->
+  <xacro:property name="a_bot_z_angle" value="0.0"/>
+  <xacro:property name="a_bot_y_angle" value="0.0"/>
+  <xacro:property name="b_bot_x" value="-0.001"/>
+  <xacro:property name="b_bot_y" value="0.531"/>
+  <xacro:property name="b_bot_z_angle" value="-3.141"/>
+  <xacro:property name="b_bot_y_angle" value="0"/>
   <xacro:property name="bots_z" value="0.75"/>
   <!-- common stuff -->
@@ -76,13 +79,25 @@
   />
   <link name="o2ac_ground" />
+  <link name="a_bot_intermediate_link" />
+  <joint name="world_a_bot_intermediate_joint" type="fixed">
+    <parent link="o2ac_ground" />
+    <child link="a_bot_intermediate_link" />
+    <origin xyz="${a_bot_x} ${a_bot_y} ${bots_z}" rpy="0.0 0.0 ${a_bot_z_angle}" />
+  </joint>
   <joint name="world_a_bot_joint" type="fixed">
+    <parent link="a_bot_intermediate_link" />
+    <child link="a_bot_base_link" />
+    <origin xyz="0 0 0" rpy="${a_bot_y_angle} 0.0 0.0" />
+  </joint>
+  <link name="b_bot_intermediate_link" />
+  <joint name="world_b_bot_intermediate_joint" type="fixed">
     <parent link="o2ac_ground" />
-    <child link="a_bot_base_link" />
-    <origin xyz="${a_bot_x} ${a_bot_y} ${bots_z}" rpy="0.0 0.0 ${a_bot_theta}" />
+    <child link="b_bot_intermediate_link" />
+    <origin xyz="${b_bot_x} ${b_bot_y} ${bots_z}" rpy="0.0 0.0 ${b_bot_z_angle}" />
   </joint>
   <joint name="world_b_bot_joint" type="fixed">
-    <parent link="o2ac_ground" />
-    <child link = "b_bot_base_link" />
-    <origin xyz="${b_bot_x} ${b_bot_y} ${bots_z}" rpy="0.0 0.0 ${b_bot_theta}" />
+    <parent link="b_bot_intermediate_link" />
+    <child link="b_bot_base_link" />
+    <origin xyz="0 0 0" rpy="${-b_bot_y_angle} 0.0 0.0" />
   </joint>
   <!-- Spawn and attach robotiq 85 gripper (+ cameras) -->

File: catkin_ws/src/o2ac_scene_description/urdf/components/o2ac_end_effector.urdf.xacro (robot description, xacro)
@@ -77,5 +77,5 @@
       <parent link="${prefix}tool_intermediate_link"/>
       <child link="${prefix}screw_tool_m4_tip_link"/>
-      <origin rpy="0 0 0" xyz=".14689 0.0 0.003 "/>
+      <origin rpy="0 0 0" xyz=".148 0.0 0.005 "/>
     </joint>
     <link name="${prefix}screw_tool_m4_tip_link"/>

File: catkin_ws/src/o2ac_scene_description/urdf/components/o2ac_end_effector_2F-140.urdf.xacro (robot description, xacro)
@@ -63,5 +63,5 @@
       <parent link="${prefix}tool_intermediate_link"/>
       <child link="${prefix}screw_tool_m4_tip_link"/>
-      <origin rpy="0 0 0" xyz=".146 -.001 -0.005 "/>
+      <origin rpy="0 0 0" xyz=".145 -.001 -0.005 "/>
     </joint>
     <link name="${prefix}screw_tool_m4_tip_link"/>
@@ -69,5 +69,5 @@
       <parent link="${prefix}tool_intermediate_link"/>
       <child link="${prefix}screw_tool_m3_tip_link"/>
-      <origin rpy="0 0 0" xyz=".128 -.001 -.0045 "/>
+      <origin rpy="0 0 0" xyz=".1265 -.001 -.0045 "/>
     </joint>
     <link name="${prefix}screw_tool_m3_tip_link"/>

File: catkin_ws/src/o2ac_scene_description/urdf/components/tools.xacro (robot description, xacro)
@@ -5,4 +5,6 @@
 <!-- The gripper center would be about 44 mm from the top, so the tip might be 111 mm further down -->
 <!-- The tip\axis seems to be 11.5 mm from the "front" side. The front side looks into the gripper -->
+  <xacro:property name="tool_offset_global_y" value="-.004" />
+  <xacro:property name="set_screw_tool_extra_offset_global_y" value="-.004" />
   <!-- Tool holders at the back of the robot system -->
   <!-- The long tool holder with 3 tools -->
@@ -10,5 +12,5 @@
     <parent link="horizontal_column_for_tools" />
     <child link="screw_tool_holder_long" />
-    <origin xyz=".04 .0 .04" rpy="0.0 0.0 ${-pi/2}" />
+    <origin xyz=".04 ${tool_offset_global_y} .04" rpy="0.0 0.0 ${-pi/2}" />
   </joint>
   <link name="screw_tool_holder_long">
@@ -56,5 +58,5 @@
     <parent link="horizontal_column_for_tools" />
     <child link="screw_tool_holder_short" />
-    <origin xyz=".04 .3 .04" rpy="0.0 0.0 ${-pi/2}" />
+    <origin xyz=".04 ${.3+set_screw_tool_extra_offset_global_y} .04" rpy="0.0 0.0 ${-pi/2}" />
   </joint>
   <link name="screw_tool_holder_short">
@@ -103,4 +105,5 @@
   <xacro:property name="back_plate_offset_short" value=".01"/>
   <xacro:property name="tool_offset" value="${-.005 + bit_cushion_to_axis}" />
+  <!--  -->
   <!-- The collision boxes of the tools only include the top part (not what is hanging underneath the holder) -->
   <link name="set_screw_tool_link">

File: catkin_ws/src/o2ac_scene_description/urdf/o2ac_environment.xacro (robot description, xacro)
@@ -16,5 +16,5 @@
   </xacro:o2ac_box>
   <xacro:o2ac_box boxname="horizontal_column_for_tools" box_w=".04" box_l=".4" box_h=".04" parent="o2ac_ground">
-    <origin xyz="${vert_column_x_back} -.2 1.058" rpy="0 0 0" />
+    <origin xyz="${vert_column_x_back} -.2 1.046" rpy="0 0 0" />
   </xacro:o2ac_box>
   <!-- Invisible walls to avoid OMPL creating crazy plans (sanity limits) -->
@@ -39,8 +39,8 @@
   <xacro:include filename="$(find o2ac_scene_description)/urdf/components/screw_feeder.xacro" />
   <xacro:screw_feeder feedername="m3_feeder" parent="workspace_center" with_collision_geometry="false">
-    <origin xyz="-.5115 -.156 0.015" rpy="0 0 0" />
+    <origin xyz="-.5115 -.155 0.005" rpy="0 0 0" />
   </xacro:screw_feeder>
   <xacro:screw_feeder feedername="m4_feeder" parent="workspace_center" with_collision_geometry="false">
-    <origin xyz="-.512 .0037 0.018" rpy="0 0 0" />
+    <origin xyz="-.513 -.002 0.008" rpy="0 0 0" />
   </xacro:screw_feeder>
   <!-- Base fixture -->
@@ -152,5 +152,5 @@
     <parent link="o2ac_ground" />
     <child link = "tv" />
-    <origin xyz="-0.4 0.0 1.58" rpy="0 0 0" />
+    <origin xyz="-0.4 0.0 1.55" rpy="0 0 0" />
   </joint>
 </robot>

Commit message: Mechanical calibration (office version)

File: catkin_ws/src/o2ac_scene_description/urdf/base_scene.urdf.xacro (robot description, xacro)
@@ -5,11 +5,13 @@
   <xacro:arg name="taskboard" default="false"/>
   <!-- Calibration parameters -->
-  <xacro:property name="a_bot_x" value="-0.004"/>
-  <xacro:property name="a_bot_y" value="-0.531"/>     <!-- Positive moves to the left -->
+  <xacro:property name="a_bot_x" value="-0.004"/>     <!-- Positive moves back -->
+  <xacro:property name="a_bot_y" value="-0.529"/>     <!-- Positive moves left -->
+  <xacro:property name="a_bot_z" value="0.0005"/>     <!-- Positive moves down -->
   <!-- Original: -0.525 -->
   <xacro:property name="a_bot_z_angle" value="0.0"/>
   <xacro:property name="a_bot_y_angle" value="0.0"/>
-  <xacro:property name="b_bot_x" value="-0.001"/>
-  <xacro:property name="b_bot_y" value="0.531"/>
+  <xacro:property name="b_bot_x" value="-0.0025"/>
+  <xacro:property name="b_bot_y" value="0.527"/>
+  <xacro:property name="b_bot_z" value="-0.005"/>
   <xacro:property name="b_bot_z_angle" value="-3.141"/>
   <xacro:property name="b_bot_y_angle" value="0"/>
@@ -83,5 +85,5 @@
     <parent link="o2ac_ground" />
     <child link="a_bot_intermediate_link" />
-    <origin xyz="${a_bot_x} ${a_bot_y} ${bots_z}" rpy="0.0 0.0 ${a_bot_z_angle}" />
+    <origin xyz="${a_bot_x} ${a_bot_y} ${bots_z+a_bot_z}" rpy="0.0 0.0 ${a_bot_z_angle}" />
   </joint>
   <joint name="world_a_bot_joint" type="fixed">
@@ -94,5 +96,5 @@
     <parent link="o2ac_ground" />
     <child link="b_bot_intermediate_link" />
-    <origin xyz="${b_bot_x} ${b_bot_y} ${bots_z}" rpy="0.0 0.0 ${b_bot_z_angle}" />
+    <origin xyz="${b_bot_x} ${b_bot_y} ${bots_z+b_bot_z}" rpy="0.0 0.0 ${b_bot_z_angle}" />
   </joint>
   <joint name="world_b_bot_joint" type="fixed">

File: catkin_ws/src/o2ac_scene_description/urdf/components/tools.xacro (robot description, xacro)
@@ -5,6 +5,6 @@
 <!-- The gripper center would be about 44 mm from the top, so the tip might be 111 mm further down -->
 <!-- The tip\axis seems to be 11.5 mm from the "front" side. The front side looks into the gripper -->
-  <xacro:property name="tool_offset_global_y" value="-.004" />
-  <xacro:property name="set_screw_tool_extra_offset_global_y" value="-.004" />
+  <xacro:property name="tool_offset_global_y" value="-0.004" />
+  <xacro:property name="set_screw_tool_extra_offset_global_y" value="-.002" />
   <!-- Tool holders at the back of the robot system -->
   <!-- The long tool holder with 3 tools -->

File: catkin_ws/src/o2ac_scene_description/urdf/o2ac_environment.xacro (robot description, xacro)
@@ -16,5 +16,5 @@
   </xacro:o2ac_box>
   <xacro:o2ac_box boxname="horizontal_column_for_tools" box_w=".04" box_l=".4" box_h=".04" parent="o2ac_ground">
-    <origin xyz="${vert_column_x_back} -.2 1.046" rpy="0 0 0" />
+    <origin xyz="${vert_column_x_back} -.2 1.058" rpy="0 0 0" />
   </xacro:o2ac_box>
   <!-- Invisible walls to avoid OMPL creating crazy plans (sanity limits) -->
@@ -39,8 +39,8 @@
   <xacro:include filename="$(find o2ac_scene_description)/urdf/components/screw_feeder.xacro" />
   <xacro:screw_feeder feedername="m3_feeder" parent="workspace_center" with_collision_geometry="false">
-    <origin xyz="-.5115 -.155 0.005" rpy="0 0 0" />
+    <origin xyz="-.5115 -.1555 0.015" rpy="0 0 0" />
   </xacro:screw_feeder>
   <xacro:screw_feeder feedername="m4_feeder" parent="workspace_center" with_collision_geometry="false">
-    <origin xyz="-.513 -.002 0.008" rpy="0 0 0" />
+    <origin xyz="-.514 0.009 0.018" rpy="0 0 0" />
   </xacro:screw_feeder>
   <!-- Base fixture -->
