Commit message: More calibrations and documentations

File: catkin_ws/src/o2ac_scene_description/urdf/base_scene.urdf.xacro (robot description, xacro)
@@ -5,14 +5,13 @@
   <xacro:arg name="taskboard" default="false"/>
   <!-- Calibration parameters -->
-  <xacro:property name="a_bot_x" value="-0.004"/>     <!-- Positive moves back -->
-  <xacro:property name="a_bot_y" value="-0.529"/>     <!-- Positive moves left -->
+  <xacro:property name="a_bot_x" value="-0.005"/>     <!-- Positive moves back -->
+  <xacro:property name="a_bot_y" value="-0.527"/>     <!-- Positive moves left -->
   <xacro:property name="a_bot_z" value="0.0005"/>     <!-- Positive moves down -->
-  <!-- Original: -0.525 -->
   <xacro:property name="a_bot_z_angle" value="0.0"/>
   <xacro:property name="a_bot_y_angle" value="0.0"/>
-  <xacro:property name="b_bot_x" value="-0.0025"/>
-  <xacro:property name="b_bot_y" value="0.527"/>
-  <xacro:property name="b_bot_z" value="-0.005"/>
-  <xacro:property name="b_bot_z_angle" value="-3.141"/>
+  <xacro:property name="b_bot_x" value="-0.002"/>
+  <xacro:property name="b_bot_y" value="0.529"/>
+  <xacro:property name="b_bot_z" value="-0.001"/>
+  <xacro:property name="b_bot_z_angle" value="${-3.1415926 + -0.001}"/> <!-- Mirror a_bot + calibration offset -->
   <xacro:property name="b_bot_y_angle" value="0"/>
   <xacro:property name="bots_z" value="0.75"/>

File: catkin_ws/src/o2ac_scene_description/urdf/components/o2ac_end_effector.urdf.xacro (robot description, xacro)
@@ -77,5 +77,7 @@
       <parent link="${prefix}tool_intermediate_link"/>
       <child link="${prefix}screw_tool_m4_tip_link"/>
-      <origin rpy="0 0 0" xyz=".148 -0.002 0.003 "/>
+      <!-- y: points towards back -->
+      <!-- z: points towards right -->
+      <origin rpy="0 0 0" xyz=".145 -0.001 0.007 "/>
     </joint>
     <link name="${prefix}screw_tool_m4_tip_link"/>

File: catkin_ws/src/o2ac_scene_description/urdf/components/o2ac_end_effector_2F-140.urdf.xacro (robot description, xacro)
@@ -63,5 +63,7 @@
       <parent link="${prefix}tool_intermediate_link"/>
       <child link="${prefix}screw_tool_m4_tip_link"/>
-      <origin rpy="0 0 0" xyz=".145 -.001 -0.005 "/>
+      <!-- y: points towards back -->
+      <!-- z: points towards left -->
+      <origin rpy="0 0 0" xyz=".145 -.001 0.0 "/>
     </joint>
     <link name="${prefix}screw_tool_m4_tip_link"/>

File: catkin_ws/src/o2ac_scene_description/urdf/components/tools.xacro (robot description, xacro)
@@ -5,5 +5,5 @@
 <!-- The gripper center would be about 44 mm from the top, so the tip might be 111 mm further down -->
 <!-- The tip\axis seems to be 11.5 mm from the "front" side. The front side looks into the gripper -->
-  <xacro:property name="tool_offset_global_y" value="-0.004" />
+  <xacro:property name="tool_offset_global_y" value="0.003" />
   <xacro:property name="set_screw_tool_extra_offset_global_y" value="-.002" />
   <!-- Tool holders at the back of the robot system -->

Commit message: Update base_scene with new universal_robot descriptions

File: catkin_ws/src/o2ac_scene_description/urdf/base_scene.urdf.xacro (robot description, xacro)
@@ -4,4 +4,5 @@
   <!-- This is the main file defining our robot arrangement and physical environment. -->
   <xacro:arg name="taskboard" default="false"/>
+  <xacro:arg name="gazebo" default="false"/>
   <!-- Calibration parameters -->
   <xacro:property name="a_bot_x" value="-0.005"/>     <!-- Positive moves back -->
@@ -17,8 +18,14 @@
   <xacro:property name="bots_z" value="0.75"/>
   <!-- common stuff -->
-  <xacro:include filename="$(find ur_description)/urdf/common.gazebo.xacro" />
+  <!-- <xacro:include filename="$(find ur_description)/urdf/common.gazebo.xacro" />
+  <xacro:include filename="$(find ur_e_description)/urdf/ur5e.urdf.xacro" /> -->
+  <xacro:if value="$(arg gazebo)">
+    <xacro:include filename="$(find o2ac_scene_description)/urdf/ur_gazebo.xacro"/>
+  </xacro:if>
+  <xacro:unless value="$(arg gazebo)">
+    <xacro:include filename="$(find ur_description)/urdf/inc/ur_macro.xacro"/>
+  </xacro:unless>
   <!-- <xacro:include filename="$(find o2ac_gazebo)/urdf/o2ac_base_scene.gazebo" /> -->
   <!-- robots -->
-  <xacro:include filename="$(find ur_e_description)/urdf/ur5e.urdf.xacro" />
   <!-- Scene items (trays, columns, tools, jigs, feeders...) -->
   <xacro:include filename="$(find o2ac_scene_description)/urdf/o2ac_environment.xacro" />
@@ -55,28 +62,52 @@
     <origin xyz="0.0 0.0 ${bots_z-robot_mount_plate+workplate_h}" rpy="0.0 0.0 0.0" />
   </joint>
-  <xacro:ur5e_robot prefix="a_bot_" joint_limited="true"
-    shoulder_pan_lower_limit="${-pi}" shoulder_pan_upper_limit="${pi}"
-    shoulder_lift_lower_limit="${-pi}" shoulder_lift_upper_limit="${pi}"
-    elbow_joint_lower_limit="0.0" elbow_joint_upper_limit="${pi}"
-    wrist_1_lower_limit="${-pi*1.5}" wrist_1_upper_limit="${pi}"
-    wrist_2_lower_limit="${-pi*1.5}" wrist_2_upper_limit="${pi*1.5}"
-    wrist_3_lower_limit="${-2*pi}" wrist_3_upper_limit="${2*pi}"
-    transmission_hw_interface="hardware_interface/PositionJointInterface"
-    safety_limits="false" safety_pos_margin="0.15"
+  <xacro:ur_robot
+    prefix="a_bot_"
+    joint_limits_parameters_file='$(find o2ac_scene_description)/config/a_bot_joint_limits.yaml'
+    kinematics_parameters_file='$(find o2ac_scene_description)/config/a_bot_calibration.yaml'
+    physical_parameters_file='$(find ur_description)/config/ur5e/physical_parameters.yaml'
+    visual_parameters_file='$(find ur_description)/config/ur5e/visual_parameters.yaml'
+    transmission_hw_interface='hardware_interface/PositionJointInterface'
+    safety_limits="false"
+    safety_pos_margin="0.15"
     safety_k_position="20"
-    kinematics_file="${load_yaml('$(find o2ac_scene_description)/config/a_bot_calibration.yaml')}"
   />
-  <xacro:ur5e_robot prefix="b_bot_" joint_limited="true"
-    shoulder_pan_lower_limit="${-pi}" shoulder_pan_upper_limit="${pi}"
-    shoulder_lift_lower_limit="${-pi}" shoulder_lift_upper_limit="${pi}"
-    elbow_joint_lower_limit="0.0" elbow_joint_upper_limit="${pi}"
-    wrist_1_lower_limit="${-pi*1.5}" wrist_1_upper_limit="${pi}"
-    wrist_2_lower_limit="${-pi*1.5}" wrist_2_upper_limit="${pi*1.5}"
-    wrist_3_lower_limit="${-2*pi}" wrist_3_upper_limit="${2*pi}"
-    transmission_hw_interface="hardware_interface/PositionJointInterface"
-    safety_limits="false" safety_pos_margin="0.15"
+  <link name="a_bot_ee_link">
+    <collision>
+      <geometry>
+        <box size="0.01 0.01 0.01"/>
+      </geometry>
+      <origin rpy="0 0 0" xyz="-0.01 0 0"/>
+    </collision>
+  </link>
+  <joint name="a_bot_ee_fixed_joint" type="fixed">
+    <parent link="a_bot_wrist_3_link"/>
+    <child link="a_bot_ee_link"/>
+    <origin rpy="0.0 -1.57079632679 1.57079632679" xyz="0.0 0.0 0.0"/>
+  </joint>
+  <xacro:ur_robot
+    prefix="b_bot_"
+    joint_limits_parameters_file='$(find o2ac_scene_description)/config/b_bot_joint_limits.yaml'
+    kinematics_parameters_file='$(find o2ac_scene_description)/config/b_bot_calibration.yaml'
+    physical_parameters_file='$(find ur_description)/config/ur5e/physical_parameters.yaml'
+    visual_parameters_file='$(find ur_description)/config/ur5e/visual_parameters.yaml'
+    transmission_hw_interface='hardware_interface/PositionJointInterface'
+    safety_limits="false"
+    safety_pos_margin="0.15"
     safety_k_position="20"
-    kinematics_file="${load_yaml('$(find o2ac_scene_description)/config/b_bot_calibration.yaml')}"
   />
+  <link name="b_bot_ee_link">
+    <collision>
+      <geometry>
+        <box size="0.01 0.01 0.01"/>
+      </geometry>
+      <origin rpy="0 0 0" xyz="-0.01 0 0"/>
+    </collision>
+  </link>
+  <joint name="b_bot_ee_fixed_joint" type="fixed">
+    <parent link="b_bot_wrist_3_link"/>
+    <child link="b_bot_ee_link"/>
+    <origin rpy="0.0 -1.57079632679 1.57079632679" xyz="0.0 0.0 0.0"/>
+  </joint>
   <link name="o2ac_ground" />
   <link name="a_bot_intermediate_link" />
