Commit message: Update cooking env

File: catkin_ws/src/o2ac_scene_description/urdf/cooking_environment.xacro (robot description, xacro)
@@ -115,5 +115,11 @@
     <origin rpy="0 0 0" xyz="-0.15 0 0.10"/>
   </joint>
-  <link name="bowl">
+  <link name="cooking_board_surface"/>
+  <joint name="cooking_board_surface_joint" type="fixed">
+    <parent link="cooking_board" />
+    <child link = "cooking_board_surface" />
+    <origin rpy="0 0 0" xyz="0.0 0 0.01"/>
+  </joint>
+  <!-- <link name="bowl">
     <visual>
       <origin rpy="0 0 0" xyz="0 0 0"/>
@@ -136,5 +142,5 @@
     <child link = "bowl" />
     <origin rpy="0 0 0" xyz="0.05 0 0.0"/>
-  </joint>
+  </joint> -->
   <link name="plate">
     <visual>
