Commit message: Confirmed that calibration works for cameras fixed to the environment

File: catkin_ws/src/aist_modules/aist_scene_description/urdf/base_scene.urdf.xacro (robot description, xacro)
@@ -62,10 +62,14 @@
   </joint>
   <!-- Spawn and attach gripper (+ FT300 sensor) -->
-  <xacro:include filename="$(find aist_scene_description
-			   )/urdf/components/aist_end_effector.urdf.xacro"/>
-  <xacro:aist_end_effector prefix="a_bot_" use_soft_wrist="false"
-			   use_cameras="true" parent="a_bot_ee_link"/>
-  <xacro:include filename="$(find aist_scene_description
+  <xacro:include filename="$(find o2ac_scene_description
 			   )/urdf/components/ft300.urdf.xacro"/>
+  <xacro:ft300 prefix="a_bot_" parent="a_bot_ee_link">
+    <origin xyz="0 0 0" rpy="0 0 0"/>
+  </xacro:ft300>
+  <xacro:include filename="$(find o2ac_scene_description
+			   )/urdf/components/o2ac_end_effector.urdf.xacro" />
+  <xacro:o2ac_end_effector prefix="a_bot_" use_soft_wrist="false"
+			   use_cameras="true"
+			   parent = "a_bot_ft300_flange_link" />
   <xacro:ft300 prefix="b_bot_" parent="b_bot_ee_link">
     <origin xyz="0 0 0" rpy="0 0 0"/>

File: catkin_ws/src/aist_modules/aist_scene_description/urdf/calibration.urdf.xacro (robot description, xacro)
@@ -15,9 +15,9 @@
     <origin xyz="0.063 0.0 0.0215" rpy="0 0 0"/>
   </xacro:ar_marker_70_5>
-  <xacro:ar_marker_160_10 prefix="workspace_"
-			  parent="workspace_center"
-			  marker_id="32"
-			  thickness="0.001">
+  <xacro:ar_marker_70_5 prefix="workspace_"
+			parent="workspace_center"
+			marker_id="32"
+			thickness="0.001">
     <origin xyz="0.0 0.0 0.0005" rpy="0 0 0"/>
-  </xacro:ar_marker_160_10>
+  </xacro:ar_marker_70_5>
 </robot>

Commit message: Squashed changes from localizer branch (ueshiba)

File: catkin_ws/src/aist_modules/aist_scene_description/urdf/base_scene.urdf.xacro (robot description, xacro)
@@ -3,11 +3,10 @@
   <xacro:arg name="scene" default=""/>
   <!-- Calibration help: If the robot is not moving far enough to the calibration point, increase these distances -->
-  <xacro:property name="a_bot_x" value="0"/>
-  <xacro:property name="a_bot_y" value="-0.4875"/>
-  <!-- <xacro:property name="a_bot_theta" value="${pi}"/> -->
-  <xacro:property name="b_bot_x" value="0"/>
-  <xacro:property name="b_bot_y" value="0.4875"/>
-  <xacro:property name="b_bot_theta" value="${pi}"/>
-  <xacro:property name="bots_z" value="0.77"/>
+  <xacro:property name="a_bot_x"	value="0"/>
+  <xacro:property name="a_bot_y"	value="-0.4875"/>
+  <xacro:property name="b_bot_x"	value="0"/>
+  <xacro:property name="b_bot_y"	value="0.4875"/>
+  <xacro:property name="b_bot_theta"	value="${pi}"/>
+  <xacro:property name="bots_z"		value="0.77"/>
   <!-- This is the main file defining our robot arrangement and physical environment. -->
   <!-- Main workspace -->
@@ -42,5 +41,6 @@
     wrist_2_lower_limit="${-pi}" wrist_2_upper_limit="${pi}"
     wrist_3_lower_limit="${-pi}" wrist_3_upper_limit="${pi}"
-    kinematics_file="${load_yaml('$(find aist_scene_description)/config/a_bot_calibration.yaml')}"/>
+    kinematics_file="${load_yaml('$(find aist_scene_description
+		     )/config/a_bot_calibration.yaml')}"/>
   <xacro:ur5_robot prefix="b_bot_" joint_limited="false"
     shoulder_pan_lower_limit="${-pi}" shoulder_pan_upper_limit="${pi}"
@@ -50,5 +50,6 @@
     wrist_2_lower_limit="${-pi}" wrist_2_upper_limit="${pi}"
     wrist_3_lower_limit="${-pi}" wrist_3_upper_limit="${pi}"
-    kinematics_file="${load_yaml('$(find aist_scene_description)/config/b_bot_calibration.yaml')}"/>
+    kinematics_file="${load_yaml('$(find aist_scene_description
+		     )/config/b_bot_calibration.yaml')}"/>
   <joint name="ground_a_bot_joint" type="fixed">
     <parent link="ground"/>
@@ -70,6 +71,6 @@
 			   )/urdf/components/o2ac_end_effector.urdf.xacro" />
   <xacro:o2ac_end_effector prefix="a_bot_" use_soft_wrist="false"
-			   use_cameras="true"
-			   parent = "a_bot_ft300_flange_link" />
+  			   use_cameras="true"
+  			   parent = "a_bot_ft300_flange_link" />
   <xacro:ft300 prefix="b_bot_" parent="b_bot_ee_link">
     <origin xyz="0 0 0" rpy="0 0 0"/>
@@ -87,14 +88,14 @@
   <!-- </xacro:o2ac_box> -->
   <!-- Add PhoXi 3D scanner -->
-  <xacro:include filename="$(find
-			   aist_phoxi_camera)/urdf/phoxi_m_camera.urdf.xacro"/>
-  <xacro:phoxi_m_camera prefix="a_phoxi_m_" parent="workspace_center">
-    <origin xyz="0.483543436025
-		 -0.0149511700982
-		 0.633792706454"
-	    rpy="${-152.286950706*pi/180}
-		 ${-2.00315281361*pi/180}
-		 ${86.7522427304*pi/180}"/>
-  </xacro:phoxi_m_camera>
+  <!-- <xacro:include filename="$(find -->
+  <!-- 			   aist_phoxi_camera)/urdf/phoxi_m_camera.urdf.xacro"/> -->
+  <!-- <xacro:phoxi_m_camera prefix="a_phoxi_m_" parent="workspace_center"> -->
+  <!--   <origin xyz="0.483543436025 -->
+  <!-- 		 -0.0149511700982 -->
+  <!-- 		 0.633792706454" -->
+  <!-- 	    rpy="${-152.286950706*pi/180} -->
+  <!-- 		 ${-2.00315281361*pi/180} -->
+  <!-- 		 ${86.7522427304*pi/180}"/> -->
+  <!-- </xacro:phoxi_m_camera> -->
   <!-- I would like to remove the "world" link definition, but apparently it is necessary for Gazebo -->
   <link name="world"/>
@@ -107,6 +108,6 @@
   <xacro:property name="scene_name" value="$(arg scene)"/>
   <xacro:if value="${scene_name != ''}">
-    <xacro:include filename="$(find aist_scene_description)/urdf/$(arg
-			     scene).urdf.xacro"/>
+    <xacro:include filename="$(find aist_scene_description
+			     )/urdf/$(arg scene).urdf.xacro"/>
   </xacro:if>
 </robot>

Commit message: Confirmed that calibration works with 'aist' configuration

File: catkin_ws/src/aist_modules/aist_scene_description/urdf/base_scene.urdf.xacro (robot description, xacro)
@@ -77,25 +77,32 @@
   </xacro:ft300>
   <xacro:include filename="$(find aist_scene_description
-			   )/urdf/components/single_suction_gripper.urdf.xacro"/>
+  			   )/urdf/components/single_suction_gripper.urdf.xacro"/>
   <xacro:single_suction_gripper prefix="b_bot_"
   				parent="b_bot_ft300_flange_link">
     <origin xyz="0 0 0" rpy="0 ${0.4*pi/180} ${0.1*pi/180}"/>
   </xacro:single_suction_gripper>
-  <!-- Add virtual wall to avoid collisions-->
-  <!-- <xacro:o2ac_box boxname="vwall1" box_w="0.01" box_l="0.3" box_h="0.5" -->
-  <!-- 		  parent="ground"> -->
-  <!--   <origin xyz="0.45 -0.15 ${bots_z}" rpy="0 0 0"/> -->
-  <!-- </xacro:o2ac_box> -->
-  <!-- Add PhoXi 3D scanner -->
-  <!-- <xacro:include filename="$(find -->
-  <!-- 			   aist_phoxi_camera)/urdf/phoxi_m_camera.urdf.xacro"/> -->
-  <!-- <xacro:phoxi_m_camera prefix="a_phoxi_m_" parent="workspace_center"> -->
-  <!--   <origin xyz="0.483543436025 -->
-  <!-- 		 -0.0149511700982 -->
-  <!-- 		 0.633792706454" -->
-  <!-- 	    rpy="${-152.286950706*pi/180} -->
-  <!-- 		 ${-2.00315281361*pi/180} -->
-  <!-- 		 ${86.7522427304*pi/180}"/> -->
-  <!-- </xacro:phoxi_m_camera> -->
+  <!-- Provide force feedback -->
+  <gazebo reference="a_bot_wrist_3_joint">
+    <provideFeedback>true</provideFeedback>
+  </gazebo>
+  <gazebo>
+    <plugin name="ft_sensor" filename="libgazebo_ros_ft_sensor.so">
+      <updateRate>500.0</updateRate>
+      <topicName>a_bot/wrench</topicName>
+      <gaussianNoise>1.0</gaussianNoise>
+      <jointName>a_bot_wrist_3_joint</jointName>
+    </plugin>
+  </gazebo>
+  <gazebo reference="b_bot_wrist_3_joint">
+    <provideFeedback>true</provideFeedback>
+  </gazebo>
+  <gazebo>
+    <plugin name="ft_sensor" filename="libgazebo_ros_ft_sensor.so">
+      <updateRate>500.0</updateRate>
+      <topicName>b_bot/wrench</topicName>
+      <gaussianNoise>1.0</gaussianNoise>
+      <jointName>b_bot_wrist_3_joint</jointName>
+    </plugin>
+  </gazebo>
   <!-- I would like to remove the "world" link definition, but apparently it is necessary for Gazebo -->
   <link name="world"/>

File: catkin_ws/src/aist_modules/aist_scene_description/urdf/camera_calibration.urdf.xacro (robot description, xacro)
@@ -9,10 +9,10 @@
   <!--   <origin xyz="0.0 0.0 0.0185" rpy="0 0 0"/> -->
   <!-- </xacro:ar_marker_70_5> -->
-  <xacro:ar_marker_70_5 prefix="b_bot_"
-  			parent="b_bot_single_suction_gripper_base_link"
-  			marker_id="26"
-			thickness="0.005">
-    <origin xyz="0.063 0.0 0.0215" rpy="0 0 0"/>
-  </xacro:ar_marker_70_5>
+  <!-- <xacro:ar_marker_70_5 prefix="b_bot_" -->
+  <!-- 			parent="b_bot_single_suction_gripper_base_link" -->
+  <!-- 			marker_id="26" -->
+  <!-- 			thickness="0.005"> -->
+  <!--   <origin xyz="0.063 0.0 0.0215" rpy="0 0 0"/> -->
+  <!-- </xacro:ar_marker_70_5> -->
   <xacro:ar_marker_70_5 prefix="workspace_"
 			parent="workspace_center"
