Commit message: WIP: Fix localizer mesh orientation

File: catkin_ws/src/o2ac_parts_description/urdf/templates/macro_template.urdf.xacro (robot description, xacro)
@@ -3,5 +3,5 @@
     <link name="${prefix}MACRONAME_INTERNAL">
       <visual>
-        <origin rpy="1.5707 0 0" xyz="0 0 0"/>
+        <origin rpy="0 0 0" xyz="0 0 0"/>
         <geometry>
           <mesh filename="package://o2ac_parts_description/meshes/PARTNAME.dae" scale="0.001 0.001 0.001"/>
@@ -12,5 +12,5 @@
       </visual>
       <collision>
-        <origin rpy="1.5707 0 0" xyz="0 0 0"/>
+        <origin rpy="0 0 0" xyz="0 0 0"/>
         <geometry>
           <mesh filename="package://o2ac_parts_description/meshes/PARTNAME.vhacd.dae" scale="0.001 0.001 0.001"/>

Commit message: Improve checking whether the registered model is involved within bounding box

File: catkin_ws/src/o2ac_parts_description/urdf/templates/macro_template.urdf.xacro (robot description, xacro)
@@ -18,9 +18,15 @@
       </collision>
     </link>
+    <link name="${prefix}MACRONAME_INTERNAL_origin"/>
+    <joint name="${prefix}MACRONAME_INTERNAL_origin_joint" type="fixed">
+      <parent link="${prefix}MACRONAME_INTERNAL"/>
+      <child link="${prefix}MACRONAME_INTERNAL_origin"/>
+      <origin rpy="${-pi/2} 0 0" xyz="0 0 0"/>
+    </joint>
     <xacro:if value="${spawn_attached}">
       <joint name="${prefix}MACRONAME_INTERNAL_joint" type="fixed">
         <parent link="${parent}"/>
         <child link="${prefix}MACRONAME_INTERNAL"/>
-        <xacro:insert_block name="origin"/>
+	<xacro:insert_block name="origin"/>
       </joint>
     </xacro:if>
